File: ecad/Front_Panel_sch.kicad_sch (KiCad schematic)
At the start: 0 parts

Commit message: To add front panel
Parts:
- added SW2, SW3, SW4, SW5, SW6, SW7: SW_MEC_5E, symbol Switch:SW_MEC_5E
Other:
- title: (none) -> Buck Converter
