File: ecad/Card_3.kicad_sch (KiCad schematic)
At the start: 61 parts, among them J3 Conn_01x03_Pin, J4 USB_C_Receptacle_USB2.0_14P, SW16 SW_Push, SW17 SW_Push, U10 MCP23017_SO, U11 NCP1117-3.3_SOT223, U12 MCP23017_SO, U8 W25Q128JVS, U9 RP2350_80QFN, X2 ABM8-272-T3

Commit message: Front Panel Schematic Done
Finished Part of the Schematic, need to check for ERC.
Parts:
- renumbered C29 to C5, C30 to C53, C31 to C54, C32 to C55, C33 to C56, C34 to C57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

Commit message: New Project Layout
Other:
- moved on the sheet: C73, C74, U7
