File: ecad/Card_3.kicad_sch (KiCad schematic)
At the start: 61 parts, among them J1 Conn_01x03_Pin, J2 USB_C_Receptacle_USB2.0_14P, SW14 SW_Push, SW18 SW_Push, U13 MCP23017_SO, U3 W25Q128JVS, U4 RP2350_80QFN, U5 MCP23017_SO, U7 NCP1117-3.3_SOT223, X1 ABM8-272-T3

Commit message: PCB Update
Changed lines of the file:
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@@
 (kicad_sch
-	(version 20231120)
+	(version 20250114)
 	(generator "eeschema")
-	(generator_version "8.0")
+	(generator_version "9.0")
 	(paper "A3")
 	(title_block
@@
 		(comment 4 "Seth Deegan")
 	)
+	(text "Bulk"
+		(exclude_from_sim no)
+		(at 221.488 57.404 0)
+		(effects
+			(font
+				(size 1.27 1.27)
+			)
+		)
+	)
+	(text "Keep Close"
+		(exclude_from_sim no)
+		(at 162.56 77.216 0)
+		(effects
+			(font
+				(size 1.27 1.27)
+			)
+		)
+	)
+	(text "Pin 53 & 54, and 68 & 69, shared"
+		(exclude_from_sim no)
+		(at 119.126 54.356 0)
+		(effects
+			(font
+				(size 1.27 1.27)
+			)
+		)
+	)
 	(junction
 		(at 44.45 74.93)
@@
 		)
 	)
-	(text "Bulk"
-		(exclude_from_sim no)
-		(at 221.488 57.404 0)
-		(effects
-			(font
-				(size 1.27 1.27)
-			)
-		)
-	)
-	(text "Keep Close"
-		(exclude_from_sim no)
-		(at 162.56 77.216 0)
-		(effects
-			(font
-				(size 1.27 1.27)
-			)
-		)
-	)
-	(text "Pin 53 & 54, and 68 & 69, shared"
-		(exclude_from_sim no)
-		(at 119.126 54.356 0)
-		(effects
-			(font
-				(size 1.27 1.27)
-			)
-		)
-	)

Commit message: New labels
Other:
- note added: "This is a STRETCH PDSR"
Changed lines of the file:
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@@
+		)
+	)
+	(text "This is a STRETCH PDSR\n"
+		(exclude_from_sim no)
+		(at 34.544 22.86 0)
+		(effects
+			(font
+				(size 1.27 1.27)
+				(thickness 0.254)
+				(bold yes)
+			)
 		)
 	)

Commit message: Testing Resets Placed
Other:
- company: (none) -> ECE 477: Digital Systems Design
Changed lines of the file:
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@@
 	(paper "A3")
 	(title_block
+		(date "2025-02-26")
+		(company "ECE 477: Digital Systems Design")
 		(comment 1 "Brian Lu")
 		(comment 2 "Nathan Huang")

Commit message: Push
Parts:
- renumbered C57 to C5, C60 to C54, C61 to C55, C62 to C56, C63 to C57, C64 to C58, C65 to C59, C59 to C6, C66 to C60, C67 to C61, C68 to C62, C69 to C63, C71 to C64, C72 to C65, C58 to C66, C53 to C67, C56 to C68, C54 to C69, C73 to C70, C74 to C71, C5 to C72, C55 to C73, C70 to C74, J1 to J5, JP41 to JP33, JP38 to JP34, JP1 to JP36, JP46 to JP37, JP44 to JP38, JP42 to JP39, JP39 to JP40, JP36 to JP41, JP33 to JP42, JP47 to JP43, JP45 to JP44, JP43 to JP45, JP40 to JP46, JP37 to JP47, JP34 to JP48, L1 to L4, R33 to R31, R34 to R32, R37 to R33, R38 to R34, R31 to R35, R32 to R36, R10 to R37, R35 to R38, R36 to R42, SW14 to SW26, SW18 to SW27, U4 to U13, U7 to U14, U5 to U15, U13 to U16, U3 to U7, X1 to X5
Other:
- moved on the sheet: C5, C54, C6
