File: ecad/Front_Panel.kicad_sch (KiCad schematic)
At the start: 69 parts, among them SW23 SW_SPST, SW24 SW_SPST, SW25 SW_SPST, SW26 SW_SPST, SW27 SW_SPST, SW28 SW_SPST, SW29 SW_SPST, SW30 SW_SPST, SW31 SW_SPST, SW32 SW_SPST, SW33 SW_SPST, SW34 SW_SPST, SW35 SW_SPST, SW36 SW_SPST, SW37 SW_SPST, SW38 SW_SPST, U18 TLC5916, U19 MCP23008-xSO, U20 MCP23017_SO, U21 TLC5916, U22 TLC5916

Commit message: Front Panel Schematic Done
Finished Part of the Schematic, need to check for ERC.
Parts:
- removed D25, D40, D48: A7, symbol Device:LED
- removed D26, D39, D47: A6, symbol Device:LED
- removed D27, D38, D46: A5, symbol Device:LED
- removed D28, D37, D45: A4, symbol Device:LED
- removed D29, D36, D44: A3, symbol Device:LED
- removed D30, D35, D43: A2, symbol Device:LED
- removed D31, D34, D42: A1, symbol Device:LED
- removed D32, D33, D41: A0, symbol Device:LED
- removed R42, R43, R44, R45, R54, R55, R56, R57, R58, R59, R60, R61, R62, R63, R64, R65, R66, R67, R68, R69, R70, R71, R72, R73: 220, symbol Device:R_US
- removed SW23, SW24, SW25, SW26, SW27, SW28, SW29, SW30, SW31, SW32, SW33, SW34, SW35, SW36, SW37, SW38: SW_SPST, symbol Switch:SW_SPST
- removed U18, U21, U22: TLC5916, symbol Driver_LED:TLC5916
- removed U19: MCP23008-xSO, Package_SO:SOIC-18W_7.5x11.6mm_P1.27mm, symbol Interface_Expansion:MCP23008-xSO
- removed U20: MCP23017_SO, Package_SO:SOIC-28W_7.5x17.9mm_P1.27mm, symbol Interface_Expansion:MCP23017_SO
- added D1, D17, D9: A0, symbol Device:LED
- added D10, D18, D2: A1, symbol Device:LED
- added D11, D19, D3: A2, symbol Device:LED
- added D12, D20, D4: A3, symbol Device:LED
- added D13, D21, D5: A4, symbol Device:LED
- added D14, D22, D6: A5, symbol Device:LED
- added D15, D23, D7: A6, symbol Device:LED
- added D16, D24, D8: A7, symbol Device:LED
- added R1, R10, R11, R12, R13, R14, R15, R16, R2, R3, R4, R46, R47, R48, R49, R5, R50, R51, R52, R53, R6, R7, R8, R9: 220, symbol Device:R_US
- added SW1, SW10, SW11, SW12, SW13, SW19, SW2, SW20, SW21, SW3, SW4, SW5, SW6, SW7, SW8, SW9: SW_SPST, symbol Switch:SW_SPST
- added U14, U17, U2: TLC5916, symbol Driver_LED:TLC5916
- added U15: MCP23017_SO, Package_SO:SOIC-28W_7.5x17.9mm_P1.27mm, symbol Interface_Expansion:MCP23017_SO
- added U16: MCP23008-xSO, Package_SO:SOIC-18W_7.5x11.6mm_P1.27mm, symbol Interface_Expansion:MCP23008-xSO
Connections:
- net +3.3V: now also R1.2, R10.2, R11.2, R12.2, R13.2, R14.2, R15.2, R16.2, R2.2, R3.2, R4.2, R46.2, R47.2, R48.2, R49.2, R5.2, R50.2, R51.2, R52.2, R53.2, R6.2, R7.2, R8.2, R9.2, U14.16 (VDD), U15.10 (VSS), U15.9 (VDD), U16.18 (VDD), U16.9 (VSS), U17.16 (VDD), U2.16 (VDD)
- net A0: now also SW1.1 (A)
- net A1: now also SW2.1 (A)
- net A10: now also SW11.1 (A)
- net A11: now also SW12.1 (A)
- net A12: now also SW13.1 (A)
- net A13: now also SW19.1 (A)
- net A14: now also SW20.1 (A)
- net A15: now also SW21.1 (A)
- net A2: now also SW3.1 (A)
- net A3: now also SW4.1 (A)
- net A4: now also SW5.1 (A)
- net A5: now also SW6.1 (A)
- net A6: now also SW7.1 (A)
- net A7: now also SW8.1 (A)
- net A8: now also SW9.1 (A)
- net A9: now also SW10.1 (A)
- net Earth: now also U14.1 (GND), U17.1 (GND), U2.1 (GND)
- new net: D12.2 (A), R12.1
- new net: D1.1 (K), U15.1 (GPB0), U2.5 (~{OUT0})
- new net: D1.2 (A), R1.1
- new net: D13.1 (K), U14.9 (~{OUT4}), U15.25 (GPA4)
- new net: D13.2 (A), R13.1
- new net: D9.1 (K), U14.5 (~{OUT0}), U15.21 (GPA0)
- new net: D9.2 (A), R9.1
- new net: D17.2 (A), R46.1
- new net: D6.1 (K), U15.6 (GPB5), U2.10 (~{OUT5})
- new net: D7.1 (K), U15.7 (GPB6), U2.11 (~{OUT6})
- new net: D8.1 (K), U15.8 (GPB7), U2.12 (~{OUT7})
- new net: D2.1 (K), U15.2 (GPB1), U2.6 (~{OUT1})
- new net: D3.1 (K), U15.3 (GPB2), U2.7 (~{OUT2})
- new net: D4.1 (K), U15.4 (GPB3), U2.8 (~{OUT3})
- new net: D5.1 (K), U15.5 (GPB4), U2.9 (~{OUT4})
- new net: D14.2 (A), R14.1
- new net: D7.2 (A), R7.1
- new net: D22.1 (K), U16.15 (GP5), U17.10 (~{OUT5})
- new net: D23.1 (K), U16.16 (GP6), U17.11 (~{OUT6})
- new net: D24.1 (K), U16.17 (GP7), U17.12 (~{OUT7})
- new net: D17.1 (K), U16.10 (GP0), U17.5 (~{OUT0})
- new net: D18.1 (K), U16.11 (GP1), U17.6 (~{OUT1})
- new net: D19.1 (K), U16.12 (GP2), U17.7 (~{OUT2})
- new net: D20.1 (K), U16.13 (GP3), U17.8 (~{OUT3})
- new net: D21.1 (K), U16.14 (GP4), U17.9 (~{OUT4})
- new net: D4.2 (A), R4.1
- new net: D20.2 (A), R49.1
- new net: D23.2 (A), R52.1
- new net: D3.2 (A), R3.1
- new net: D5.2 (A), R5.1
- new net: D8.2 (A), R8.1
- new net: D6.2 (A), R6.1
- new net: D11.1 (K), U14.7 (~{OUT2}), U15.23 (GPA2)
- new net: D11.2 (A), R11.1
- new net: D18.2 (A), R47.1
- new net: D24.2 (A), R53.1
- new net: D21.2 (A), R50.1
- new net: D16.2 (A), R16.1
- new net: D12.1 (K), U14.8 (~{OUT3}), U15.24 (GPA3)
- new net: D10.1 (K), U14.6 (~{OUT1}), U15.22 (GPA1)
- new net: D10.2 (A), R10.1
- new net: D22.2 (A), R51.1
- new net: D2.2 (A), R2.1
- new net: D19.2 (A), R48.1
- new net: D15.1 (K), U14.11 (~{OUT6}), U15.27 (GPA6)
- new net: D15.2 (A), R15.1
- new net: D14.1 (K), U14.10 (~{OUT5}), U15.26 (GPA5)
- new net: D16.1 (K), U14.12 (~{OUT7}), U15.28 (GPA7)
Other:
- removed sheet Back_Plane
- removed sheet Card 1 (CPU)
- removed sheet Card 2 (RAM)
- removed sheet Card 3 (UART) - Stretch
- removed sheet Front_Panel (Clone)
- note removed: "Converted Size:"
- note removed: "FRONT PANEL"
- note removed: "Original Size: 17 inches (length of front panel) x 7 inches (height of front panel) x 18 inches (depth of machine)"
- title: ECE 477 Digital Systems Design -> (none)

Commit message: PCB Update
Parts:
- added A1: RaspberryPi_Pico, Module:RaspberryPi_Pico_Common_Unspecified, symbol MCU_Module:RaspberryPi_Pico
Connections:
- new net: A1.13 (GND), A1.18 (GND), A1.23 (GND), A1.28 (GND), A1.3 (GND), A1.38 (GND), A1.8 (GND)
Changed lines of the file:
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@@
 (kicad_sch
-	(version 20231120)
+	(version 20250114)
 	(generator "eeschema")
-	(generator_version "8.0")
+	(generator_version "9.0")
 	(paper "A3")
 	(title_block
@@
 		(comment 4 "Seth Deegan")
 	)
+	(text "Put Switch Array\n"
+		(exclude_from_sim no)
+		(at 137.922 160.274 0)
+		(effects
+			(font
+				(size 1.27 1.27)
+			)
+		)
+	)
+	(text "Replace with TLC59211IN Footprint\n"
+		(exclude_from_sim no)
+		(at 98.806 160.528 0)
+		(effects
+			(font
+				(size 1.27 1.27)
+			)
+		)
+	)
 	(junction
 		(at 339.09 217.17)
@@
 		)
 	)
-	(text "Put Switch Array\n"
-		(exclude_from_sim no)
-		(at 137.922 160.274 0)
-		(effects
-			(font
-				(size 1.27 1.27)
-			)
-		)
-	)
-	(text "Replace with TLC59211IN Footprint\n"
-		(exclude_from_sim no)
-		(at 98.806 160.528 0)
-		(effects
-			(font
-				(size 1.27 1.27)
-			)
-		)
-	)
 	(global_label "A6"
 		(shape input)
@@
 					(unit 1)
 				)
+			)
+		)
+	)
+	(symbol
+		(lib_id "MCU_Module:RaspberryPi_Pico")
+		(at 124.46 219.71 0)
+		(unit 1)
+		(exclude_from_sim no)
+		(in_bom yes)
+		(on_board yes)
+		(dnp no)
+		(fields_autoplaced yes)
+		(property "Reference" "A1"
+			(at 126.6033 254 0)
+			(effects
+				(font
+					(size 1.27 1.27)
+				)
+				(justify left)
+			)
+		)
+		(property "Value" "RaspberryPi_Pico"
+			(at 126.6033 256.54 0)
+			(effects
+				(font
+					(size 1.27 1.27)
+				)
+				(justify left)
+			)
+		)
+		(property "Footprint" "Module:RaspberryPi_Pico_Common_Unspecified"
+			(at 124.46 266.7 0)
+			(effects
+				(font
+					(size 1.27 1.27)
+				)
+				(hide yes)
+			)
+		)
+		(property "Datasheet" "https://datasheets.raspberrypi.com/pico/pico-datasheet.pdf"
+			(at 124.46 269.24 0)
+			(effects
+				(font
+					(size 1.27 1.27)
+				)
+				(hide yes)
+			)
+		)
+		(property "Description" "Versatile and inexpensive microcontroller module powered by RP2040 dual-core Arm Cortex-M0+ processor up to 133 MHz, 264kB SRAM, 2MB QSPI flash; also supports Raspberry Pi Pico 2"
+			(at 124.46 271.78 0)
+			(effects
+				(font
+					(size 1.27 1.27)
+				)
+				(hide yes)
+			)
+		)
+		(pin "40"
+		)
+		(pin "5"
+		)
+		(pin "13"
+		)
+		(pin "30"
+		)
+		(pin "6"
+		)
+		(pin "25"
+		)
+		(pin "4"
+		)
+		(pin "33"
+		)
+		(pin "8"
+		)
+		(pin "3"
+		)
+		(pin "7"
+		)
+		(pin "2"
+		)
+		(pin "9"
+		)
+		(pin "15"
+		)
+		(pin "20"
+		)
+		(pin "17"
+		)
+		(pin "39"
+		)
+		(pin "1"
+		)
+		(pin "12"
+		)
+		(pin "11"
+		)
+		(pin "14"
+		)
+		(pin "18"
+		)
+		(pin "28"
+		)
+		(pin "19"
+		)
+		(pin "38"
+		)
+		(pin "36"
+		)
+		(pin "21"
+		)
+		(pin "10"
+		)
+		(pin "26"
+		)
+		(pin "27"
+		)
+		(pin "37"
+		)
+		(pin "23"
+		)
+		(pin "29"
+		)
+		(pin "31"
+		)
+		(pin "34"
+		)
+		(pin "22"
+		)
+		(pin "32"
+		)
+		(pin "24"
+		)
+		(pin "16"
+		)
+		(pin "35"
+		)
+		(instances
+			(project ""
+				(path "/b682b302-8ca4-4b40-b0cb-fd99f4675538/2b76b2e1-4674-498d-877d-fd40f416b010"
+					(reference "A1")
+					(unit 1)
+				)
