File: ecad/Card_2.kicad_sch (KiCad schematic)
At the start: 61 parts, among them J3 Conn_01x03_Pin, J4 USB_C_Receptacle_USB2.0_14P, SW16 SW_Push, SW17 SW_Push, U10 MCP23017_SO, U11 NCP1117-3.3_SOT223, U12 MCP23017_SO, U8 W25Q128JVS, U9 RP2350_80QFN, X2 ABM8-272-T3

Commit message: Testing Resets Placed
Other:
- company: (none) -> ECE 477: Digital Systems Design
- title: (none) -> RAM Card for Miniaturized Altair 8800 
Changed lines of the file:
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@@
 	(paper "A3")
 	(title_block
+		(title "RAM Card for Miniaturized Altair 8800 ")
+		(date "2025-02-26")
+		(company "ECE 477: Digital Systems Design")
 		(comment 1 "Brian Lu")
 		(comment 2 "Nathan Huang")
