File: ecad/ecad.kicad_sch (KiCad schematic)
At the start: 69 parts, among them SW23 SW_SPST, SW24 SW_SPST, SW25 SW_SPST, SW26 SW_SPST, SW27 SW_SPST, SW28 SW_SPST, SW29 SW_SPST, SW30 SW_SPST, SW31 SW_SPST, SW32 SW_SPST, SW33 SW_SPST, SW34 SW_SPST, SW35 SW_SPST, SW36 SW_SPST, SW37 SW_SPST, SW38 SW_SPST, U18 TLC5916, U19 MCP23008-xSO, U20 MCP23017_SO, U21 TLC5916, U22 TLC5916

Commit message: New labels
Parts:
- removed SW31, SW32, SW33, SW34, SW35, SW36, SW37, SW38: SW_SPST, symbol Switch:SW_SPST
- removed U21: TLC5916, symbol Driver_LED:TLC5916
- added SW1, SW2, SW3, SW4, SW5, SW6, SW7, SW8: SW_SPST, symbol Switch:SW_SPST
- added U1, U2: TLC59211IN, N20, symbol 2025-02-26_04-26-50:TLC59211IN
Connections:
- net +3.3V: now also SW23.1 (A), SW24.1 (A), SW25.1 (A), SW26.1 (A), SW27.1 (A), SW28.1 (A), SW29.1 (A), SW30.1 (A), SW1.1 (A), SW2.1 (A), SW3.1 (A), SW4.1 (A), SW5.1 (A), SW6.1 (A), SW7.1 (A), SW8.1 (A)
- net A0: now also SW1.2 (B), U1.2 (D1); no longer SW23.1 (A)
- net A1: now also SW24.2 (B), SW2.2 (B), U1.3 (D2); no longer SW24.1 (A)
- net A10: now also U2.4 (D3)
- net A11: now also U2.5 (D4)
- net A12: now also U2.6 (D5)
- net A13: now also U2.7 (D6)
- net A14: now also U2.8 (D7)
- net A15: now also U2.9 (D8)
- net A2: now also SW25.2 (B), SW3.2 (B), U1.4 (D3); no longer SW25.1 (A)
- net A3: now also SW26.2 (B), SW4.2 (B), U1.5 (D4); no longer SW26.1 (A)
- net A4: now also SW27.2 (B), SW5.2 (B), U1.6 (D5); no longer SW27.1 (A)
- net A5: now also SW28.2 (B), SW6.2 (B), U1.7 (D6); no longer SW28.1 (A)
- net A6: now also SW29.2 (B), SW7.2 (B), U1.8 (D7); no longer SW29.1 (A)
- net A7: now also SW30.2 (B), SW8.2 (B), U1.9 (D8); no longer SW30.1 (A)
- net A8: now also SW23.2 (B), U2.2 (D1)
- net A9: now also U2.3 (D2)
- no-connect marks 0 -> 4
Other:
- sheet Card 3 (UART) - Stretch renamed Card 3 (UART)

Commit message: Testing Resets Placed
Parts:
- removed D25, D40, D48: A7, symbol Device:LED
- removed D26, D39, D47: A6, symbol Device:LED
- removed D27, D38, D46: A5, symbol Device:LED
- removed D28, D37, D45: A4, symbol Device:LED
- removed D29, D36, D44: A3, symbol Device:LED
- removed D30, D35, D43: A2, symbol Device:LED
- removed D31, D34, D42: A1, symbol Device:LED
- removed D32, D33, D41: A0, symbol Device:LED
- removed R42, R43, R44, R45, R54, R55, R56, R57, R58, R59, R60, R61, R62, R63, R64, R65, R66, R67, R68, R69, R70, R71, R72, R73: 220, symbol Device:R_US
- removed U18, U22: TLC5916, symbol Driver_LED:TLC5916
- removed U19: MCP23008-xSO, Package_SO:SOIC-18W_7.5x11.6mm_P1.27mm, symbol Interface_Expansion:MCP23008-xSO
- added D1, D10, D11, D12, D13, D14, D15, D16, D17, D18, D19, D2, D20, D21, D22, D23, D24, D3, D4, D5, D6, D7, D8, D9: LED, symbol Device:LED
- added R1, R10, R11, R12, R13, R14, R15, R16, R17, R18, R19, R2, R20, R21, R22, R23, R24, R3, R4, R5, R6, R7, R8, R9: 220, symbol Device:R_US
- added SW17, SW18, SW19, SW20, SW21, SW22, SW23, SW24, SW25: SW_SPST, symbol Switch:SW_SPST
- added U3: TLC59211IN, N20, symbol 2025-02-26_04-26-50:TLC59211IN
- added U4: MCP23008-xSO, Package_SO:SOIC-18W_7.5x11.6mm_P1.27mm, symbol Interface_Expansion:MCP23008-xSO
- added U6: RP2350_80QFN, RP2350_80QFN_minimal:RP2350-QFN-80-1EP_10x10_P0.4mm_EP3.4x3.4mm_ThermalVias, symbol MCU_RaspberryPi_RP2350:RP2350_80QFN
- renumbered SW24 to SW10, SW25 to SW11, SW26 to SW12, SW27 to SW13, SW28 to SW14, SW29 to SW15, SW30 to SW16, SW23 to SW9, U20 to U5
Connections:
- net A0: now also U5.1 (GPB0)
- net A1: now also U5.2 (GPB1); no longer SW10.2 (B)
- net A10: now also SW11.2 (B), U5.23 (GPA2)
- net A11: now also SW12.2 (B), U5.24 (GPA3)
- net A12: now also SW13.2 (B), U5.25 (GPA4)
- net A13: now also SW14.2 (B), U5.26 (GPA5)
- net A14: now also SW15.2 (B), U5.27 (GPA6)
- net A15: now also SW16.2 (B), U5.28 (GPA7)
- net A2: now also U5.3 (GPB2); no longer SW11.2 (B)
- net A3: now also U5.4 (GPB3); no longer SW12.2 (B)
- net A4: now also U5.5 (GPB4); no longer SW13.2 (B)
- net A5: now also U5.6 (GPB5); no longer SW14.2 (B)
- net A6: now also U5.7 (GPB6); no longer SW15.2 (B)
- net A7: now also U5.8 (GPB7); no longer SW16.2 (B)
- net A8: now also U5.21 (GPA0)
- net A9: now also SW10.2 (B), U5.22 (GPA1)
- net GND: now reaches U1.11 (GND)
- net GND: now also U2.11 (GND), U5.10 (VSS), U5.15 (A0), U5.16 (A1), U5.17 (A2), SW25.1 (A), U3.11 (GND), U4.4 (A1), U4.5 (A0), U4.9 (VSS)
- net A7_LED: now reaches U1.12 (*Y8)
- net A7_LED: now also D8.1 (K)
- net A6_LED: now reaches U1.13 (*Y7)
- net A6_LED: now also D7.1 (K)
- net A5_LED: now reaches U1.14 (*Y6)
- net A5_LED: now also D6.1 (K)
- net A4_LED: now reaches U1.15 (*Y5)
- net A4_LED: now also D5.1 (K)
- net A3_LED: now reaches U1.16 (*Y4)
- net A3_LED: now also D4.1 (K)
- net A2_LED: now reaches U1.17 (*Y3)
- net A2_LED: now also D3.1 (K)
- net A1_LED: now reaches U1.18 (*Y2)
- net A1_LED: now also D2.1 (K)
- net A0_LED: now reaches U1.19 (*Y1)
- net A0_LED: now also D1.1 (K)
- net 3.3V: now reaches U1.20 (VCC)
- net 3.3V: now also SW1.1 (A), SW10.1 (A), SW11.1 (A), SW12.1 (A), SW13.1 (A), SW14.1 (A), SW15.1 (A), SW16.1 (A), SW2.1 (A), SW3.1 (A), SW4.1 (A), SW5.1 (A), SW6.1 (A), SW7.1 (A), SW8.1 (A), SW9.1 (A), U2.20 (VCC), U5.18 (~{RESET}), U5.9 (VDD), R1.2, R10.2, R11.2, R12.2, R13.2, R14.2, R15.2, R16.2, R17.2, R18.2, R19.2, R2.2, R20.2, R21.2, R22.2, R23.2, R24.2, R3.2, R4.2, R5.2, R6.2, R7.2, R8.2, R9.2, SW17.1 (A), SW18.1 (A), SW19.1 (A), SW20.1 (A), SW21.1 (A), SW22.1 (A), SW23.1 (A), SW24.1 (A), SW25.2 (B), U3.20 (VCC), U4.18 (VDD), U4.3 (A2), U4.6 (~{RESET})
- net A15_LED: now reaches U2.12 (*Y8)
- net A15_LED: now also D16.1 (K)
- net A14_LED: now reaches U2.13 (*Y7)
- net A14_LED: now also D15.1 (K)
- net A13_LED: now reaches U2.14 (*Y6)
- net A13_LED: now also D14.1 (K)
- net A12_LED: now reaches U2.15 (*Y5)
- net A12_LED: now also D13.1 (K)
- net A11_LED: now reaches U2.16 (*Y4)
- net A11_LED: now also D12.1 (K)
- net A10_LED: now reaches U2.17 (*Y3)
- net A10_LED: now also D11.1 (K)
- net A9_LED: now reaches U2.18 (*Y2)
- net A9_LED: now also D10.1 (K)
- net A8_LED: now reaches U2.19 (*Y1)
- net A8_LED: now also D9.1 (K)
- net IQR_Handler_A1: now reaches U5.19 (INTB)
- net IQR_Handler_A2: now reaches U5.20 (INTA)
- removed net +3.3V: SW1.1 (A), SW10.1 (A), SW11.1 (A), SW12.1 (A), SW13.1 (A), SW14.1 (A), SW15.1 (A), SW16.1 (A), SW2.1 (A), SW3.1 (A), SW4.1 (A), SW5.1 (A), SW6.1 (A), SW7.1 (A), SW8.1 (A), SW9.1 (A), U5.10 (VSS), U5.9 (VDD)
- new net: D22.2 (A), R22.1
- new net: D13.2 (A), R13.1
- new net: D12.2 (A), R12.1
- new net: D15.2 (A), R15.1
- new net: D8.2 (A), R8.1
- new net: D19.2 (A), R19.1
- new net: D5.2 (A), R5.1
- new net: D17.2 (A), R17.1
- new net: D9.2 (A), R9.1
- new net: D11.2 (A), R11.1
- new net: D18.2 (A), R18.1
- new net: D6.2 (A), R6.1
- new net: D7.2 (A), R7.1
- new net: D14.2 (A), R14.1
- new net: D3.2 (A), R3.1
- new net: D23.2 (A), R23.1
- new net: D20.2 (A), R20.1
- new net: D2.2 (A), R2.1
- new net: D21.2 (A), R21.1
- new net: D16.2 (A), R16.1
- new net: D4.2 (A), R4.1
- new net: D24.2 (A), R24.1
- new net: D1.2 (A), R1.1
- new net: D10.2 (A), R10.1
- new net AUX1: SW23.2 (B)
- new net AUX2: SW24.2 (B)
- new net D0: U3.2 (D1), U4.10 (GP0)
- new net D0_LED: D17.1 (K), U3.19 (*Y1)
- new net D1: U3.3 (D2), U4.11 (GP1)
- new net D1_LED: D18.1 (K), U3.18 (*Y2)
- new net D2: U3.4 (D3), U4.12 (GP2)
- new net D2_LED: D19.1 (K), U3.17 (*Y3)
- new net D3: U3.5 (D4), U4.13 (GP3)
- new net D3_LED: D20.1 (K), U3.16 (*Y4)
- new net D4: U3.6 (D5), U4.14 (GP4)
- new net D4_LED: D21.1 (K), U3.15 (*Y5)
- new net D5: U3.7 (D6), U4.15 (GP5)
- new net D5_LED: D22.1 (K), U3.14 (*Y6)
- new net D6: U3.8 (D7), U4.16 (GP6)
- new net D6_LED: D23.1 (K), U3.13 (*Y7)
- new net D7: U3.9 (D8), U4.17 (GP7)
- new net D7_LED: D24.1 (K), U3.12 (*Y8)
- new net DEPOSIT: SW20.2 (B)
- new net EXAMINE: SW19.2 (B)
- new net IQR_Handler_DATA: U4.8 (INT)
- new net PROTECT: SW22.2 (B)
- new net RESET: SW21.2 (B)
- new net SINGLE: SW18.2 (B)
- new net STOP: SW17.2 (B)
- no-connect marks 4 -> 17
Other:
- removed sheet Front_Panel (Clone)
- note added: "*BOLD ON A LABEL MEANS IT IS NOT CURRENTLY BEING USED"
- note added: "ADDRESS I/O EXPANDER"
- note added: "ADDRESS LINE LEDs"
- note added: "DATA I/O EXPANDER"
- note added: "DATA LINE LEDs"
- note added: "FOOTNOTES"
- note added: "FRONT PANEL (NEW)"
- note added: "FRONT PANEL (OLD)"
- note added: "MICROCONTROLLER (1)"
- note added: "OFF (IMPORTANT)"
- note added: "OPTIONAL LABELS, MAY USE LATER"
- note added: "SINK DRIVERS"
- note added: "SWITCHES"
- note removed: "FRONT PANEL"
- note removed: "Put Switch Array"
- note removed: "Replace with TLC59211IN Footprint"
- company: (none) -> ECE 477: Digital Systems Design
- moved on the sheet: SW1, SW10, SW11, SW12, SW13, SW14, SW15, SW16, SW2, SW3, SW4, SW5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
