File: ecad/Power_Distribution.kicad_sch (KiCad schematic)
At the start: 10 parts, among them SW22 SW_SPST, U1 MCP16331x-xCH

Commit message: PCB Update
Changed lines of the file:
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@@
 (kicad_sch
-	(version 20231120)
+	(version 20250114)
 	(generator "eeschema")
-	(generator_version "8.0")
+	(generator_version "9.0")
 	(paper "A4")
 	(title_block

Commit message: Testing Resets Placed
Other:
- company: (none) -> ECE 477: Digital Systems Design
Changed lines of the file:
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@@
 	(paper "A4")
 	(title_block
+		(date "2025-02-26")
+		(company "ECE 477: Digital Systems Design")
 		(comment 1 "Brian Lu")
 		(comment 2 "Nathan Huang")

Commit message: Ready for Layout
Parts:
- removed SW22: SW_SPST, Button_Switch_SMD:SW_DIP_SPSTx01_Slide_6.7x4.1mm_W6.73mm_P2.54mm_LowProfile_JPin, symbol Switch:SW_SPST
- renumbered C3 to C49, C2 to C50, C1 to C51, C4 to C52, L2 to L3, R39 to R49, R40 to R50, R41 to R51, U1 to U20
Connections:
- net +5V: now also R49.1, U20.4 (EN)
Changed lines of the file:
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@@
-	)
-	(junction
-		(at 68.58 87.63)
-		(diameter 0)
-		(color 0 0 0 0)
 	)
 	(junction
@@
 	(wire
 		(pts
-			(xy 81.28 73.66) (xy 91.44 73.66)
-		)
-		(stroke
-			(width 0)
-			(type default)
-		)
-	)
-	(wire
-		(pts
 			(xy 107.95 87.63) (xy 107.95 91.44)
 		)
@@
 	(wire
 		(pts
-			(xy 71.12 73.66) (xy 68.58 73.66)
+			(xy 68.58 73.66) (xy 91.44 73.66)
 		)
 		(stroke
@@
 		(dnp no)
 		(fields_autoplaced yes)
-		(property "Reference" "C4"
+		(property "Reference" "C52"
 			(at 171.45 77.4699 0)
 			(effects
@@
 			(project "ecad"
 				(path "/b682b302-8ca4-4b40-b0cb-fd99f4675538/8ac99590-cdb7-457f-9b2c-c22421ccb183/b634cce5-68f2-492b-8de2-08cd2bb51e98"
-					(reference "C4")
-					(unit 1)
-				)
-			)
-		)
-	)
-	(symbol
-		(lib_id "power:PWR_FLAG")
-		(at 68.58 87.63 90)
-		(unit 1)
-		(exclude_from_sim no)
-		(in_bom yes)
-		(on_board yes)
-		(dnp no)
-		(fields_autoplaced yes)
-		(property "Reference" "#FLG02"
-			(at 66.675 87.63 0)
-			(effects
-				(font
-					(size 1.27 1.27)
-				)
-				(hide yes)
-			)
-		)
-		(property "Value" "PWR_FLAG"
-			(at 64.77 87.6299 90)
-			(effects
-				(font
-					(size 1.27 1.27)
-				)
-				(justify left)
-			)
-		)
-		(property "Footprint" ""
-			(at 68.58 87.63 0)
-			(effects
-				(font
-					(size 1.27 1.27)
-				)
-				(hide yes)
-			)
-		)
-		(property "Datasheet" "~"
-			(at 68.58 87.63 0)
-			(effects
-				(font
-					(size 1.27 1.27)
-				)
-				(hide yes)
-			)
-		)
-		(property "Description" "Special symbol for telling ERC where power comes from"
-			(at 68.58 87.63 0)
-			(effects
-				(font
-					(size 1.27 1.27)
-				)
-				(hide yes)
-			)
-		)
-		(pin "1"
-		)
-		(instances
-			(project "ecad"
-				(path "/b682b302-8ca4-4b40-b0cb-fd99f4675538/8ac99590-cdb7-457f-9b2c-c22421ccb183/b634cce5-68f2-492b-8de2-08cd2bb51e98"
-					(reference "#FLG02")
+					(reference "C52")
 					(unit 1)
 				)
@@
 		(dnp no)
 		(fields_autoplaced yes)
-		(property "Reference" "C2"
+		(property "Reference" "C50"
 			(at 127 57.15 90)
 			(effects
@@
 			(project "ecad"
 				(path "/b682b302-8ca4-4b40-b0cb-fd99f4675538/8ac99590-cdb7-457f-9b2c-c22421ccb183/b634cce5-68f2-492b-8de2-08cd2bb51e98"
-					(reference "C2")
+					(reference "C50")
 					(unit 1)
 				)
@@
 		(dnp no)
 		(fields_autoplaced yes)
-		(property "Reference" "C3"
+		(property "Reference" "C49"
 			(at 157.48 77.4699 0)
 			(effects
@@
 			(project "ecad"
 				(path "/b682b302-8ca4-4b40-b0cb-fd99f4675538/8ac99590-cdb7-457f-9b2c-c22421ccb183/b634cce5-68f2-492b-8de2-08cd2bb51e98"
-					(reference "C3")
+					(reference "C49")
 					(unit 1)
 				)
@@
 		(dnp no)
 		(fields_autoplaced yes)
-		(property "Reference" "U1"
+		(property "Reference" "U20"
 			(at 107.95 60.96 0)
 			(effects
@@
 			(project "ecad"
 				(path "/b682b302-8ca4-4b40-b0cb-fd99f4675538/8ac99590-cdb7-457f-9b2c-c22421ccb183/b634cce5-68f2-492b-8de2-08cd2bb51e98"
-					(reference "U1")
+					(reference "U20")
 					(unit 1)
 				)
@@
 		(dnp no)
 		(fields_autoplaced yes)
-		(property "Reference" "R41"
+		(property "Reference" "R51"
 			(at 127 69.85 90)
 			(effects
@@
 			(project "ecad"
 				(path "/b682b302-8ca4-4b40-b0cb-fd99f4675538/8ac99590-cdb7-457f-9b2c-c22421ccb183/b634cce5-68f2-492b-8de2-08cd2bb51e98"
-					(reference "R41")
+					(reference "R51")
 					(unit 1)
 				)
@@
 		(dnp no)
 		(fields_autoplaced yes)
-		(property "Reference" "R40"
+		(property "Reference" "R50"
 			(at 123.19 81.2799 0)
 			(effects
@@
 			(project "ecad"
 				(path "/b682b302-8ca4-4b40-b0cb-fd99f4675538/8ac99590-cdb7-457f-9b2c-c22421ccb183/b634cce5-68f2-492b-8de2-08cd2bb51e98"
-					(reference "R40")
+					(reference "R50")
 					(unit 1)
 				)
@@
 		(dnp no)
 		(fields_autoplaced yes)
-		(property "Reference" "L2"
+		(property "Reference" "L3"
 			(at 138.43 66.04 90)
 			(effects
@@
 			(project "ecad"
 				(path "/b682b302-8ca4-4b40-b0cb-fd99f4675538/8ac99590-cdb7-457f-9b2c-c22421ccb183/b634cce5-68f2-492b-8de2-08cd2bb51e98"
-					(reference "L2")
+					(reference "L3")
 					(unit 1)
 				)
@@
 	)
 	(symbol
-		(lib_id "Switch:SW_SPST")
-		(at 76.2 73.66 0)
-		(unit 1)
-		(exclude_from_sim no)
-		(in_bom yes)
-		(on_board yes)
-		(dnp no)
-		(property "Reference" "SW22"
-			(at 76.2 75.438 0)
-			(effects
-				(font
-					(size 1.27 1.27)
-				)
-			)
-		)
-		(property "Value" "SW_SPST"
-			(at 76.2 77.978 0)
-			(effects
-				(font
-					(size 1.27 1.27)
-				)
-			)
-		)
-		(property "Footprint" "Button_Switch_SMD:SW_DIP_SPSTx01_Slide_6.7x4.1mm_W6.73mm_P2.54mm_LowProfile_JPin"
-			(at 76.2 73.66 0)
-			(effects
-				(font
-					(size 1.27 1.27)
-				)
-				(hide yes)
-			)
-		)
-		(property "Datasheet" "~"
-			(at 76.2 73.66 0)
-			(effects
-				(font
-					(size 1.27 1.27)
-				)
-				(hide yes)
-			)
-		)
-		(property "Description" "Single Pole Single Throw (SPST) switch"
-			(at 76.2 73.66 0)
-			(effects
-				(font
-					(size 1.27 1.27)
-				)
-				(hide yes)
-			)
-		)
-		(pin "1"
-		)
-		(pin "2"
-		)
-		(instances
-			(project "ecad"
-				(path "/b682b302-8ca4-4b40-b0cb-fd99f4675538/8ac99590-cdb7-457f-9b2c-c22421ccb183/b634cce5-68f2-492b-8de2-08cd2bb51e98"
-					(reference "SW22")
-					(unit 1)
-				)
-			)
-		)
-	)
-	(symbol
 		(lib_id "Device:C")
 		(at 68.58 82.55 0)
@@
 		(dnp no)
 		(fields_autoplaced yes)
-		(property "Reference" "C1"
+		(property "Reference" "C51"
 			(at 72.39 81.2799 0)
 			(effects
@@
 			(project "ecad"
 				(path "/b682b302-8ca4-4b40-b0cb-fd99f4675538/8ac99590-cdb7-457f-9b2c-c22421ccb183/b634cce5-68f2-492b-8de2-08cd2bb51e98"
-					(reference "C1")
+					(reference "C51")
 					(unit 1)
 				)
@@
 		(dnp no)
 		(fields_autoplaced yes)
-		(property "Reference" "R39"
+		(property "Reference" "R49"
 			(at 93.98 80.0099 0)
 			(effects
@@
 			(project "ecad"
 				(path "/b682b302-8ca4-4b40-b0cb-fd99f4675538/8ac99590-cdb7-457f-9b2c-c22421ccb183/b634cce5-68f2-492b-8de2-08cd2bb51e98"
-					(reference "R39")
+					(reference "R49")
 					(unit 1)
 				)
