File: ecad/ecad.kicad_pcb (KiCad board)
At the start: 4 copper layers, 12 parts, among them SW1 SW_SPST, U1 MCP16331x-xCH

Commit message: To add front panel
Parts:
- removed D1: 1N5819, Diode_THT:D_DO-41_SOD81_P10.16mm_Horizontal
- removed L1: L, Inductor_SMD:L_0201_0603Metric
- moved SW1 47.9 mm to (38.0, 28.5), turned to 180 degrees
- moved L2 37.8 mm to (38.0, 34.5), turned to 180 degrees
- moved R2 36.3 mm to (34.0, 44.5)
- moved C4 35.4 mm to (31.5, 35.5)
- moved U1 34.8 mm to (38.0, 39.5)
- moved R3 33.7 mm to (41.5, 44.5), turned to 90 degrees
- moved C2 33.0 mm to (45.0, 41.0), turned to 0 degrees
- moved C3 30.2 mm to (31.5, 41.0)
- moved R1 29.4 mm to (38.0, 44.5), turned to 90 degrees
- moved C1 27.6 mm to (45.0, 35.0)
Routing:
- net Net-(SW1-B): track 27.8 -> 19.2 mm, vias 3 -> 0
- net Net-(C3-Pad1): track 20.9 -> 27.4 mm, vias 1 -> 2
- net Net-(U1-SW): track 18.4 -> 13.3 mm, vias 0 -> 3
- net GND: track 35.2 -> 39.5 mm, vias 0 -> 2
- net Net-(D1-K): track 3.92 -> 0.00 mm
- net Net-(U1-V_{FB}): track 16.2 -> 13.8 mm, vias 2 -> 0
- net +5V: track 17.5 -> 19.0 mm, vias 3 -> 2
- added copper zone on B.Cu, net GND
Other:
- board outline added: 31 x 28 mm
- board text added: "ECE 47700 - Team 15"
- board text removed: "Team 15"

Commit message: Ready for Layout
Parts:
- added C1: 100n, Capacitor_SMD:CP_Elec_3x5.4, F.Cu at (105.2, 41.6)
- added C10: 100n, Capacitor_SMD:CP_Elec_3x5.4, F.Cu at (111.9, 51.3)
- added C11: 100n, Capacitor_SMD:CP_Elec_3x5.4, F.Cu at (111.9, 56.2)
- added C12: 100n, Capacitor_SMD:CP_Elec_3x5.4, F.Cu at (111.9, 61.0)
- added C13: 100n, Capacitor_SMD:CP_Elec_3x5.4, F.Cu at (111.9, 65.9)
- added C14: 10u, Capacitor_SMD:CP_Elec_3x5.4, F.Cu at (111.9, 70.7)
- added C15: 15p, Capacitor_SMD:CP_Elec_3x5.4, F.Cu at (118.7, 41.6)
- added C16: 15p, Capacitor_SMD:CP_Elec_3x5.4, F.Cu at (118.7, 46.5)
- added C17: 100n, Capacitor_SMD:CP_Elec_3x5.4, F.Cu at (118.7, 51.3)
- added C18: 4.7u, Capacitor_SMD:CP_Elec_3x5.4, F.Cu at (118.7, 56.2)
- added C19: 4.7u, Capacitor_SMD:CP_Elec_3x5.4, F.Cu at (118.7, 61.0)
- added C2: 4.7u, Capacitor_SMD:CP_Elec_3x5.4, F.Cu at (105.2, 46.5)
- added C20: 4.7u, Capacitor_SMD:CP_Elec_3x5.4, F.Cu at (118.7, 65.9)
- added C21: 10u, Capacitor_SMD:CP_Elec_3x5.4, F.Cu at (118.7, 70.7)
- added C22: 10u, Capacitor_SMD:CP_Elec_3x5.4, F.Cu at (125.4, 41.6)
- added C23: 100n, Capacitor_SMD:CP_Elec_3x5.4, F.Cu at (125.4, 46.5)
- added C24: 100n, Capacitor_SMD:CP_Elec_3x5.4, F.Cu at (125.4, 51.3)
- added C25: 100n, Capacitor_SMD:CP_Elec_3x5.4, F.Cu at (125.4, 56.2)
- added C26: 100n, Capacitor_SMD:CP_Elec_3x5.4, F.Cu at (125.4, 61.0)
- added C27: 100n, Capacitor_SMD:CP_Elec_3x5.4, F.Cu at (105.2, 82.2)
- added C28: 4.7u, Capacitor_SMD:CP_Elec_3x5.4, F.Cu at (105.2, 87.0)
- added C29: 100n, Capacitor_SMD:CP_Elec_3x5.4, F.Cu at (105.2, 91.9)
- added C3: 100n, Capacitor_SMD:CP_Elec_3x5.4, F.Cu at (105.2, 51.3)
- added C30: 100n, Capacitor_SMD:CP_Elec_3x5.4, F.Cu at (105.2, 96.7)
- added C31: 100n, Capacitor_SMD:CP_Elec_3x5.4, F.Cu at (105.2, 101.6)
- added C32: 100n, Capacitor_SMD:CP_Elec_3x5.4, F.Cu at (105.2, 106.4)
- added C33: 100n, Capacitor_SMD:CP_Elec_3x5.4, F.Cu at (105.2, 111.3)
- added C34: 100n, Capacitor_SMD:CP_Elec_3x5.4, F.Cu at (111.9, 82.2)
- added C35: 100n, Capacitor_SMD:CP_Elec_3x5.4, F.Cu at (111.9, 87.0)
- added C36: 100n, Capacitor_SMD:CP_Elec_3x5.4, F.Cu at (111.9, 91.9)
- added C37: 100n, Capacitor_SMD:CP_Elec_3x5.4, F.Cu at (111.9, 96.7)
- added C38: 100n, Capacitor_SMD:CP_Elec_3x5.4, F.Cu at (111.9, 101.6)
- added C39: 100n, Capacitor_SMD:CP_Elec_3x5.4, F.Cu at (111.9, 106.4)
- added C4: 100n, Capacitor_SMD:CP_Elec_3x5.4, F.Cu at (105.2, 56.2)
- added C40: 10u, Capacitor_SMD:CP_Elec_3x5.4, F.Cu at (111.9, 111.3)
- added C41: 10u, Capacitor_SMD:CP_Elec_3x5.4, F.Cu at (118.7, 82.2)
- added C42: 10u, Capacitor_SMD:CP_Elec_3x5.4, F.Cu at (118.7, 87.0)
- added C43: 100n, Capacitor_SMD:CP_Elec_3x5.4, F.Cu at (118.7, 91.9)
- added C44: 100n, Capacitor_SMD:CP_Elec_3x5.4, F.Cu at (118.7, 96.7)
- added C45: 100n, Capacitor_SMD:CP_Elec_3x5.4, F.Cu at (118.7, 101.6)
- added C46: 4.7u, Capacitor_SMD:CP_Elec_3x5.4, F.Cu at (118.7, 106.4)
- added C47: 4.7u, Capacitor_SMD:CP_Elec_3x5.4, F.Cu at (118.7, 111.3)
- added C48: 4.7u, Capacitor_SMD:CP_Elec_3x5.4, F.Cu at (125.4, 82.2)
- added C49: C, Capacitor_SMD:CP_Elec_3x5.3, F.Cu at (160.0, 82.2)
- added C5: 100n, Capacitor_SMD:CP_Elec_3x5.4, F.Cu at (105.2, 61.0)
- added C50: C, Capacitor_SMD:CP_Elec_3x5.3, F.Cu at (160.0, 87.0)
- added C51: C, Capacitor_SMD:CP_Elec_3x5.3, F.Cu at (160.0, 91.9)
- added C52: C, Capacitor_SMD:CP_Elec_3x5.3, F.Cu at (160.0, 96.7)
- added C53: 15p, Capacitor_SMD:CP_Elec_3x5.4, F.Cu at (125.4, 87.0)
- added C54: 15p, Capacitor_SMD:CP_Elec_3x5.4, F.Cu at (125.4, 91.9)
- added C6: 100n, Capacitor_SMD:CP_Elec_3x5.4, F.Cu at (105.2, 65.9)
- added C7: 100n, Capacitor_SMD:CP_Elec_3x5.4, F.Cu at (105.2, 70.7)
- added C8: 100n, Capacitor_SMD:CP_Elec_3x5.4, F.Cu at (111.9, 41.6)
- added C9: 100n, Capacitor_SMD:CP_Elec_3x5.4, F.Cu at (111.9, 46.5)
- added D1: LED, LED_SMD:LED_Osram_Lx_P47F_D2mm_ReverseMount, F.Cu at (154.3, 69.8)
- added D10: LED, LED_SMD:LED_1206_3216Metric_ReverseMount_Hole1.8x2.4mm, F.Cu at (185.4, 61.5)
- added D11: LED, LED_SMD:LED_1206_3216Metric_ReverseMount_Hole1.8x2.4mm, F.Cu at (185.4, 65.6)
- added D12: LED, LED_SMD:LED_1206_3216Metric_ReverseMount_Hole1.8x2.4mm, F.Cu at (185.4, 69.6)
- added D13: LED, LED_SMD:LED_1206_3216Metric_ReverseMount_Hole1.8x2.4mm, F.Cu at (185.4, 73.6)
- added D14: LED, LED_SMD:LED_1206_3216Metric_ReverseMount_Hole1.8x2.4mm, F.Cu at (191.0, 53.4)
- added D15: LED, LED_SMD:LED_1206_3216Metric_ReverseMount_Hole1.8x2.4mm, F.Cu at (191.0, 57.5)
- added D16: LED, LED_SMD:LED_1206_3216Metric_ReverseMount_Hole1.8x2.4mm, F.Cu at (191.0, 61.5)
- added D17: LED, LED_SMD:LED_1206_3216Metric_ReverseMount_Hole1.8x2.4mm, F.Cu at (191.0, 65.6)
- added D18: LED, LED_SMD:LED_1206_3216Metric_ReverseMount_Hole1.8x2.4mm, F.Cu at (191.0, 69.6)
- added D19: LED, LED_SMD:LED_1206_3216Metric_ReverseMount_Hole1.8x2.4mm, F.Cu at (191.0, 73.6)
- added D2: LED, LED_SMD:LED_1206_3216Metric_ReverseMount_Hole1.8x2.4mm, F.Cu at (179.7, 53.4)
- added D20: LED, LED_SMD:LED_1206_3216Metric_ReverseMount_Hole1.8x2.4mm, F.Cu at (196.7, 53.4)
- added D21: LED, LED_SMD:LED_1206_3216Metric_ReverseMount_Hole1.8x2.4mm, F.Cu at (196.7, 57.5)
- added D22: LED, LED_SMD:LED_1206_3216Metric_ReverseMount_Hole1.8x2.4mm, F.Cu at (196.7, 61.5)
- added D23: LED, LED_SMD:LED_1206_3216Metric_ReverseMount_Hole1.8x2.4mm, F.Cu at (196.7, 65.6)
- added D24: LED, LED_SMD:LED_1206_3216Metric_ReverseMount_Hole1.8x2.4mm, F.Cu at (196.7, 69.6)
- added D3: LED, LED_SMD:LED_1206_3216Metric_ReverseMount_Hole1.8x2.4mm, F.Cu at (179.7, 57.5)
- added D4: LED, LED_SMD:LED_1206_3216Metric_ReverseMount_Hole1.8x2.4mm, F.Cu at (179.7, 61.5)
- added D5: LED, LED_SMD:LED_1206_3216Metric_ReverseMount_Hole1.8x2.4mm, F.Cu at (179.7, 65.6)
- added D6: LED, LED_SMD:LED_1206_3216Metric_ReverseMount_Hole1.8x2.4mm, F.Cu at (179.7, 69.6)
- added D7: LED, LED_SMD:LED_1206_3216Metric_ReverseMount_Hole1.8x2.4mm, F.Cu at (179.7, 73.6)
- added D8: LED, LED_SMD:LED_1206_3216Metric_ReverseMount_Hole1.8x2.4mm, F.Cu at (185.4, 53.4)
- added D9: LED, LED_SMD:LED_1206_3216Metric_ReverseMount_Hole1.8x2.4mm, F.Cu at (185.4, 57.5)
- added J1: Conn_01x03_Pin, Connector:Banana_Jack_1Pin, F.Cu at (170.6, 57.7)
- added J2: USB_C_Receptacle_USB2.0_14P, Connector_USB:USB_C_Receptacle_Palconn_UTC16-G, F.Cu at (134.6, 71.9)
- added J3: USB_C_Receptacle_USB2.0_14P, Connector_USB:USB_C_Receptacle_Palconn_UTC16-G, F.Cu at (147.1, 116.3)
- added J4: Conn_01x03_Pin, Connector:Banana_Jack_1Pin, F.Cu at (135.1, 101.4)
- added JP27: SolderJumper_3_Open, Jumper:SolderJumper-3_P1.3mm_Open_RoundedPad1.0x1.5mm, F.Cu at (131.6, 81.5)
- added JP28: SolderJumper_3_Open, Jumper:SolderJumper-3_P1.3mm_Open_RoundedPad1.0x1.5mm, F.Cu at (131.6, 85.4)
- added JP29: SolderJumper_3_Open, Jumper:SolderJumper-3_P1.3mm_Open_RoundedPad1.0x1.5mm, F.Cu at (131.6, 89.2)
- added JP30: SolderJumper_3_Open, Jumper:SolderJumper-3_P1.3mm_Open_RoundedPad1.0x1.5mm, F.Cu at (131.6, 93.1)
- added JP31: SolderJumper_3_Open, Jumper:SolderJumper-3_P1.3mm_Open_RoundedPad1.0x1.5mm, F.Cu at (137.3, 81.5)
- added JP32: SolderJumper_3_Open, Jumper:SolderJumper-3_P1.3mm_Open_RoundedPad1.0x1.5mm, F.Cu at (137.3, 85.4)
- added JP33: SolderJumper_3_Open, Jumper:SolderJumper-3_P1.3mm_Open_RoundedPad1.0x1.5mm, F.Cu at (137.3, 89.2)
- added JP34: SolderJumper_3_Open, Jumper:SolderJumper-3_P1.3mm_Open_RoundedPad1.0x1.5mm, F.Cu at (137.3, 93.1)
- added JP35: SolderJumper_3_Open, Jumper:SolderJumper-3_P1.3mm_Open_RoundedPad1.0x1.5mm, F.Cu at (142.9, 81.5)
- added JP36: SolderJumper_3_Open, Jumper:SolderJumper-3_P1.3mm_Open_RoundedPad1.0x1.5mm, F.Cu at (142.9, 85.4)
- added JP37: SolderJumper_3_Open, Jumper:SolderJumper-3_P1.3mm_Open_RoundedPad1.0x1.5mm, F.Cu at (142.9, 89.2)
- added JP38: SolderJumper_3_Open, Jumper:SolderJumper-3_P1.3mm_Open_RoundedPad1.0x1.5mm, F.Cu at (142.9, 93.1)
- added JP39: SolderJumper_3_Open, Jumper:SolderJumper-3_P1.3mm_Open_RoundedPad1.0x1.5mm, F.Cu at (148.6, 81.5)
- added JP40: SolderJumper_3_Open, Jumper:SolderJumper-3_P1.3mm_Open_RoundedPad1.0x1.5mm, F.Cu at (148.6, 85.4)
- added JP41: SolderJumper_3_Open, Jumper:SolderJumper-3_P1.3mm_Open_RoundedPad1.0x1.5mm, F.Cu at (148.6, 89.2)
- added JP42: SolderJumper_3_Open, Jumper:SolderJumper-3_P1.3mm_Open_RoundedPad1.0x1.5mm, F.Cu at (148.6, 93.1)
- added L1: 3.3u, Inductor_SMD:L_0201_0603Metric, F.Cu at (159.6, 68.7)
- added L2: 3.3u, Inductor_SMD:L_0201_0603Metric, F.Cu at (130.0, 131.6)
- added L3: L, Inductor_SMD:L_0201_0603Metric, F.Cu at (164.6, 90.5)
- added Q1: NMOS, Transistor_Power:GaN_Systems_GaNPX-3_5x6.6mm_Drain2.93x0.6mm, F.Cu at (167.6, 23.0)
- added Q10: NMOS, Transistor_Power:GaN_Systems_GaNPX-3_5x6.6mm_Drain2.93x0.6mm, F.Cu at (180.7, 31.1)
- added Q11: NMOS, Transistor_Power:GaN_Systems_GaNPX-3_5x6.6mm_Drain2.93x0.6mm, F.Cu at (187.3, 31.1)
- added Q12: NMOS, Transistor_Power:GaN_Systems_GaNPX-3_5x6.6mm_Drain2.93x0.6mm, F.Cu at (193.9, 31.1)
- added Q13: NMOS, Transistor_Power:GaN_Systems_GaNPX-3_5x6.6mm_Drain2.93x0.6mm, F.Cu at (200.5, 31.1)
- added Q14: NMOS, Transistor_Power:GaN_Systems_GaNPX-3_5x6.6mm_Drain2.93x0.6mm, F.Cu at (207.0, 31.1)
- added Q15: NMOS, Transistor_Power:GaN_Systems_GaNPX-3_5x6.6mm_Drain2.93x0.6mm, F.Cu at (167.6, 39.2)
- added Q16: NMOS, Transistor_Power:GaN_Systems_GaNPX-3_5x6.6mm_Drain2.93x0.6mm, F.Cu at (174.2, 39.2)
- added Q17: NMOS, Transistor_Power:GaN_Systems_GaNPX-3_5x6.6mm_Drain2.93x0.6mm, F.Cu at (180.7, 39.2)
- added Q18: NMOS, Transistor_Power:GaN_Systems_GaNPX-3_5x6.6mm_Drain2.93x0.6mm, F.Cu at (187.3, 39.2)
- added Q19: NMOS, Transistor_Power:GaN_Systems_GaNPX-3_5x6.6mm_Drain2.93x0.6mm, F.Cu at (193.9, 39.2)
- added Q2: NMOS, Transistor_Power:GaN_Systems_GaNPX-3_5x6.6mm_Drain2.93x0.6mm, F.Cu at (174.2, 23.0)
- added Q20: NMOS, Transistor_Power:GaN_Systems_GaNPX-3_5x6.6mm_Drain2.93x0.6mm, F.Cu at (200.5, 39.2)
- added Q21: NMOS, Transistor_Power:GaN_Systems_GaNPX-3_5x6.6mm_Drain2.93x0.6mm, F.Cu at (207.0, 39.2)
- added Q22: NMOS, Transistor_Power:GaN_Systems_GaNPX-3_5x6.6mm_Drain2.93x0.6mm, F.Cu at (167.6, 47.4)
- added Q23: NMOS, Transistor_Power:GaN_Systems_GaNPX-3_5x6.6mm_Drain2.93x0.6mm, F.Cu at (174.2, 47.4)
- added Q24: NMOS, Transistor_Power:GaN_Systems_GaNPX-3_5x6.6mm_Drain2.93x0.6mm, F.Cu at (180.7, 47.4)
- added Q3: NMOS, Transistor_Power:GaN_Systems_GaNPX-3_5x6.6mm_Drain2.93x0.6mm, F.Cu at (180.7, 23.0)
- added Q4: NMOS, Transistor_Power:GaN_Systems_GaNPX-3_5x6.6mm_Drain2.93x0.6mm, F.Cu at (187.3, 23.0)
- added Q5: NMOS, Transistor_Power:GaN_Systems_GaNPX-3_5x6.6mm_Drain2.93x0.6mm, F.Cu at (193.9, 23.0)
- added Q6: NMOS, Transistor_Power:GaN_Systems_GaNPX-3_5x6.6mm_Drain2.93x0.6mm, F.Cu at (200.5, 23.0)
- added Q7: NMOS, Transistor_Power:GaN_Systems_GaNPX-3_5x6.6mm_Drain2.93x0.6mm, F.Cu at (207.0, 23.0)
- added Q8: NMOS, Transistor_Power:GaN_Systems_GaNPX-3_5x6.6mm_Drain2.93x0.6mm, F.Cu at (167.6, 31.1)
- added Q9: NMOS, Transistor_Power:GaN_Systems_GaNPX-3_5x6.6mm_Drain2.93x0.6mm, F.Cu at (174.2, 31.1)
- added R1: 220, Resistor_SMD:R_0201_0603Metric_Pad0.64x0.40mm_HandSolder, F.Cu at (205.7, -31.5)
- added R10: 220, Resistor_SMD:R_0201_0603Metric_Pad0.64x0.40mm_HandSolder, F.Cu at (208.5, -31.5)
- added R11: 220, Resistor_SMD:R_0201_0603Metric_Pad0.64x0.40mm_HandSolder, F.Cu at (208.5, -29.7)
- added R12: 220, Resistor_SMD:R_0201_0603Metric_Pad0.64x0.40mm_HandSolder, F.Cu at (208.5, -28.0)
- added R13: 220, Resistor_SMD:R_0201_0603Metric_Pad0.64x0.40mm_HandSolder, F.Cu at (208.5, -26.2)
- added R14: 220, Resistor_SMD:R_0201_0603Metric_Pad0.64x0.40mm_HandSolder, F.Cu at (208.5, -24.5)
- added R15: 220, Resistor_SMD:R_0201_0603Metric_Pad0.64x0.40mm_HandSolder, F.Cu at (208.5, -22.7)
- added R16: 220, Resistor_SMD:R_0201_0603Metric_Pad0.64x0.40mm_HandSolder, F.Cu at (208.5, -21.0)
- added R17: 220, Resistor_SMD:R_0201_0603Metric_Pad0.64x0.40mm_HandSolder, F.Cu at (208.5, -19.2)
- added R18: 220, Resistor_SMD:R_0201_0603Metric_Pad0.64x0.40mm_HandSolder, F.Cu at (208.5, -17.5)
- added R19: 220, Resistor_SMD:R_0201_0603Metric_Pad0.64x0.40mm_HandSolder, F.Cu at (211.3, -31.5)
- added R2: 220, Resistor_SMD:R_0201_0603Metric_Pad0.64x0.40mm_HandSolder, F.Cu at (205.7, -29.7)
- added R20: 220, Resistor_SMD:R_0201_0603Metric_Pad0.64x0.40mm_HandSolder, F.Cu at (211.3, -29.7)
- added R21: 220, Resistor_SMD:R_0201_0603Metric_Pad0.64x0.40mm_HandSolder, F.Cu at (211.3, -28.0)
- added R22: 220, Resistor_SMD:R_0201_0603Metric_Pad0.64x0.40mm_HandSolder, F.Cu at (211.3, -26.2)
- added R23: 220, Resistor_SMD:R_0201_0603Metric_Pad0.64x0.40mm_HandSolder, F.Cu at (211.3, -24.5)
- added R24: 220, Resistor_SMD:R_0201_0603Metric_Pad0.64x0.40mm_HandSolder, F.Cu at (211.3, -22.7)
- added R25: 27, Resistor_SMD:R_0201_0603Metric_Pad0.64x0.40mm_HandSolder, F.Cu at (211.3, -21.0)
- added R26: 27, Resistor_SMD:R_0201_0603Metric_Pad0.64x0.40mm_HandSolder, F.Cu at (211.3, -19.2)
- added R28: 1k, Resistor_SMD:R_0201_0603Metric_Pad0.64x0.40mm_HandSolder, F.Cu at (211.3, -17.5)
- added R29: 1k, Resistor_SMD:R_0201_0603Metric_Pad0.64x0.40mm_HandSolder, F.Cu at (214.1, -31.5)
- added R3: 220, Resistor_SMD:R_0201_0603Metric_Pad0.64x0.40mm_HandSolder, F.Cu at (205.7, -28.0)
- added R30: 1k, Resistor_SMD:R_0201_0603Metric_Pad0.64x0.40mm_HandSolder, F.Cu at (214.1, -29.7)
- added R31: 33, Resistor_SMD:R_0201_0603Metric_Pad0.64x0.40mm_HandSolder, F.Cu at (214.1, -28.0)
- added R32: 5.1k, Resistor_SMD:R_0201_0603Metric_Pad0.64x0.40mm_HandSolder, F.Cu at (214.1, -26.2)
- added R33: 5.1k, Resistor_SMD:R_0201_0603Metric_Pad0.64x0.40mm_HandSolder, F.Cu at (214.1, -24.5)
- added R34: 1k, Resistor_SMD:R_0201_0603Metric_Pad0.64x0.40mm_HandSolder, F.Cu at (130.2, 121.1)
- added R35: 27, Resistor_SMD:R_0201_0603Metric_Pad0.64x0.40mm_HandSolder, F.Cu at (130.2, 122.8)
- added R36: 27, Resistor_SMD:R_0201_0603Metric_Pad0.64x0.40mm_HandSolder, F.Cu at (130.2, 124.6)
- added R37: 5.1k, Resistor_SMD:R_0201_0603Metric_Pad0.64x0.40mm_HandSolder, F.Cu at (130.2, 126.3)
- added R38: 5.1k, Resistor_SMD:R_0201_0603Metric_Pad0.64x0.40mm_HandSolder, F.Cu at (130.2, 128.1)
- added R39: 100k, Resistor_SMD:R_0201_0603Metric_Pad0.64x0.40mm_HandSolder, F.Cu at (130.2, 129.8)
- added R4: 220, Resistor_SMD:R_0201_0603Metric_Pad0.64x0.40mm_HandSolder, F.Cu at (205.7, -26.2)
- added R40: 100k, Resistor_SMD:R_0201_0603Metric_Pad0.64x0.40mm_HandSolder, F.Cu at (133.0, 121.1)
- added R41: 1k, Resistor_SMD:R_0201_0603Metric_Pad0.64x0.40mm_HandSolder, F.Cu at (133.0, 122.8)
- added R42: 1k, Resistor_SMD:R_0201_0603Metric_Pad0.64x0.40mm_HandSolder, F.Cu at (133.0, 124.6)
- added R43: 1k, Resistor_SMD:R_0201_0603Metric_Pad0.64x0.40mm_HandSolder, F.Cu at (133.0, 126.3)
- added R49: ?, Resistor_SMD:R_0201_0603Metric_Pad0.64x0.40mm_HandSolder, F.Cu at (164.8, 80.6)
- added R5: 220, Resistor_SMD:R_0201_0603Metric_Pad0.64x0.40mm_HandSolder, F.Cu at (205.7, -24.5)
- added R50: R_US, Resistor_SMD:R_0201_0603Metric_Pad0.64x0.40mm_HandSolder, F.Cu at (164.8, 82.4)
- added R51: R_US, Resistor_SMD:R_0201_0603Metric_Pad0.64x0.40mm_HandSolder, F.Cu at (164.8, 84.1)
- added R6: 220, Resistor_SMD:R_0201_0603Metric_Pad0.64x0.40mm_HandSolder, F.Cu at (205.7, -22.7)
- added R7: 220, Resistor_SMD:R_0201_0603Metric_Pad0.64x0.40mm_HandSolder, F.Cu at (205.7, -21.0)
- added R8: 220, Resistor_SMD:R_0201_0603Metric_Pad0.64x0.40mm_HandSolder, F.Cu at (205.7, -19.2)
- added R9: 220, Resistor_SMD:R_0201_0603Metric_Pad0.64x0.40mm_HandSolder, F.Cu at (205.7, -17.5)
- added SW1: SW_SPDT, Button_Switch_THT:SW_E-Switch_EG1224_SPDT_Angled, F.Cu at (105.6, -28.7)
- added SW10: SW_SPDT, Button_Switch_THT:SW_E-Switch_EG1224_SPDT_Angled, F.Cu at (121.3, 7.05)
- added SW11: SW_SPDT, Button_Switch_THT:SW_E-Switch_EG1224_SPDT_Angled, F.Cu at (136.9, 7.05)
- added SW12: SW_SPDT, Button_Switch_THT:SW_E-Switch_EG1224_SPDT_Angled, F.Cu at (152.5, 7.05)
- added SW13: SW_SPDT, Button_Switch_THT:SW_E-Switch_EG1224_SPDT_Angled, F.Cu at (105.6, 24.9)
- added SW14: SW_SPDT, Button_Switch_THT:SW_E-Switch_EG1224_SPDT_Angled, F.Cu at (121.3, 24.9)
- added SW15: SW_SPDT, Button_Switch_THT:SW_E-Switch_EG1224_SPDT_Angled, F.Cu at (136.9, 24.9)
- added SW16: SW_SPDT, Button_Switch_THT:SW_E-Switch_EG1224_SPDT_Angled, F.Cu at (152.5, 24.9)
- added SW17: SW_Push, Button_Switch_THT:SW_Push_1P2T_Vertical_E-Switch_800UDP8P1A1M6, F.Cu at (165.9, -30.6)
- added SW18: SW_Push, Button_Switch_THT:SW_Push_1P2T_Vertical_E-Switch_800UDP8P1A1M6, F.Cu at (165.9, -22.0)
- added SW19: SW_Push, Button_Switch_THT:SW_Push_1P2T_Vertical_E-Switch_800UDP8P1A1M6, F.Cu at (165.9, -13.5)
- added SW2: SW_SPDT, Button_Switch_THT:SW_E-Switch_EG1224_SPDT_Angled, F.Cu at (121.3, -28.7)
- added SW20: SW_Push, Button_Switch_THT:SW_Push_1P2T_Vertical_E-Switch_800UDP8P1A1M6, F.Cu at (165.9, -4.94)
- added SW21: SW_Push, Button_Switch_THT:SW_Push_1P2T_Vertical_E-Switch_800UDP8P1A1M6, F.Cu at (165.9, 3.61)
- added SW23: SW_Push, Button_Switch_THT:SW_Push_1P2T_Vertical_E-Switch_800UDP8P1A1M6, F.Cu at (165.9, 12.2)
- added SW24: SW_Push, Button_Switch_THT:SW_Push_1P2T_Vertical_E-Switch_800UDP8P1A1M6, F.Cu at (179.2, -30.6)
- added SW25: SW_Push, Button_Switch_THT:SW_Push_1P2T_Vertical_E-Switch_800UDP8P1A1M6, F.Cu at (179.2, -22.0)
- added SW26: SW_Push, Button_Switch_THT:SW_Push_1P2T_Vertical_E-Switch_800UDP8P1A1M6, F.Cu at (179.2, -13.5)
- added SW27: SW_Push, Button_Switch_THT:SW_Push_1P2T_Vertical_E-Switch_800UDP8P1A1M6, F.Cu at (179.2, -4.94)
- added SW28: SW_Push, Button_Switch_THT:SW_Push_1P2T_Vertical_E-Switch_800UDP8P1A1M6, F.Cu at (179.2, 3.61)
- added SW29: SW_Push, Button_Switch_THT:SW_Push_1P2T_Vertical_E-Switch_800UDP8P1A1M6, F.Cu at (179.2, 12.2)
- added SW3: SW_SPDT, Button_Switch_THT:SW_E-Switch_EG1224_SPDT_Angled, F.Cu at (136.9, -28.7)
- added SW30: SW_Push, Button_Switch_THT:SW_Push_1P2T_Vertical_E-Switch_800UDP8P1A1M6, F.Cu at (192.6, -30.6)
- added SW31: SW_Push, Button_Switch_THT:SW_Push_1P2T_Vertical_E-Switch_800UDP8P1A1M6, F.Cu at (192.6, -22.0)
- added SW32: SW_SPDT, Button_Switch_THT:SW_Push_1P2T_Vertical_E-Switch_800UDP8P1A1M6, F.Cu at (192.6, -13.5)
- added SW33: SPI TEST, Button_Switch_THT:SW_Push_1P2T_Vertical_E-Switch_800UDP8P1A1M6, F.Cu at (192.6, -4.94)
- added SW34: SW_Push, Button_Switch_THT:SW_Push_1P2T_Vertical_E-Switch_800UDP8P1A1M6, F.Cu at (142.9, 96.8)
- added SW35: FRONT PANEL TEST SWTICH, Button_Switch_THT:SW_Push_1P2T_Vertical_E-Switch_800UDP8P1A1M6, F.Cu at (192.6, 3.61)
- added SW36: SW_Push, Button_Switch_THT:SW_Push_1P2T_Vertical_E-Switch_800UDP8P1A1M6, F.Cu at (142.9, 105.4)
- added SW4: SW_SPDT, Button_Switch_THT:SW_E-Switch_EG1224_SPDT_Angled, F.Cu at (152.5, -28.7)
- added SW5: SW_SPDT, Button_Switch_THT:SW_E-Switch_EG1224_SPDT_Angled, F.Cu at (105.6, -10.8)
- added SW6: SW_SPDT, Button_Switch_THT:SW_E-Switch_EG1224_SPDT_Angled, F.Cu at (121.3, -10.8)
- added SW7: SW_SPDT, Button_Switch_THT:SW_E-Switch_EG1224_SPDT_Angled, F.Cu at (136.9, -10.8)
- added SW8: SW_SPDT, Button_Switch_THT:SW_E-Switch_EG1224_SPDT_Angled, F.Cu at (152.5, -10.8)
- added SW9: SW_SPDT, Button_Switch_THT:SW_E-Switch_EG1224_SPDT_Angled, F.Cu at (105.6, 7.05)
- added U1: TLC59211IN, footprints:N20, F.Cu at (137.9, 64.9)
- added U10: NCP1117-3.3_SOT223, Package_TO_SOT_SMD:SOT-223-3_TabPin2, F.Cu at (146.3, 126.4)
- added U11: MCP23017_SO, Package_SO:SOIC-28W_7.5x17.9mm_P1.27mm, F.Cu at (108.2, 123.6)
- added U12: MCP23017_SO, Package_SO:SOIC-28W_7.5x17.9mm_P1.27mm, F.Cu at (121.1, 123.6)
- added U2: TLC59211IN, footprints:N20, F.Cu at (148.5, 64.9)
- added U20: MCP16331x-xCH, Package_TO_SOT_SMD:SOT-23-6, F.Cu at (166.0, 87.4)
- added U3: TLC59211IN, footprints:N20, F.Cu at (159.0, 64.9)
- added U5: MCP23017_SO, Package_SO:SOIC-28W_7.5x17.9mm_P1.27mm, F.Cu at (205.9, 61.3)
- added U8: NCP1117-3.3_SOT223, Package_TO_SOT_SMD:SOT-223-3_TabPin2, F.Cu at (145.3, 72.0)
- added X1: ABM8-272-T3, Connector:Banana_Jack_1Pin, F.Cu at (170.6, 70.2)
- added X2: ABM8-272-T3, Connector:Banana_Jack_1Pin, F.Cu at (135.1, 113.9)
