File: ecad/Card_1.kicad_sch (KiCad schematic)
At the start: 61 parts, among them J3 Conn_01x03_Pin, J4 USB_C_Receptacle_USB2.0_14P, SW16 SW_Push, SW17 SW_Push, U10 MCP23017_SO, U11 NCP1117-3.3_SOT223, U12 MCP23017_SO, U8 W25Q128JVS, U9 RP2350_80QFN, X2 ABM8-272-T3

Commit message: Front Panel Schematic Done
Finished Part of the Schematic, need to check for ERC.
Parts:
- renumbered C43 to C10, C44 to C11, C45 to C12, C46 to C13, C48 to C14, C35 to C15, C30 to C16, C49 to C17, C37 to C18, C36 to C19, C34 to C20, C33 to C21, C31 to C22, C32 to C23, C29 to C24, C47 to C25, C52 to C26, C50 to C27, C51 to C28, C39 to C6, C40 to C7, C41 to C8, C42 to C9, JP27 to JP10, JP29 to JP11, JP31 to JP12, JP17 to JP13, JP20 to JP14, JP23 to JP15, JP26 to JP16, JP22 to JP2, JP25 to JP3, JP28 to JP4, JP30 to JP5, JP32 to JP6, JP18 to JP7, JP21 to JP8, JP24 to JP9, R22 to R11, R23 to R12, R20 to R13, R25 to R14, R24 to R15, R28 to R16, R29 to R17, R26 to R18, R27 to R19, SW17 to SW15, U12 to U6

Commit message: Testing Resets Placed
Other:
- company: (none) -> ECE 477: Digital Systems Design
- title: (none) -> CPU Card for Miniaturized Altair 8800 
- moved on the sheet: J4, R16, R17
Changed lines of the file:
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@@
 	(paper "A3")
 	(title_block
+		(title "CPU Card for Miniaturized Altair 8800 ")
+		(date "2025-02-26")
+		(company "ECE 477: Digital Systems Design")
 		(comment 1 "Brian Lu")
 		(comment 2 "Nathan Huang")
@@
 	)
 	(junction
-		(at 255.27 92.71)
+		(at 314.96 67.31)
 		(diameter 0)
 		(color 0 0 0 0)
@@
 	)
 	(junction
-		(at 255.27 97.79)
+		(at 314.96 72.39)
 		(diameter 0)
 		(color 0 0 0 0)
@@
 	)
 	(junction
-		(at 237.49 116.84)
+		(at 297.18 91.44)
 		(diameter 0)
 		(color 0 0 0 0)
@@
 	)
 	(junction
-		(at 275.59 97.79)
+		(at 335.28 72.39)
 		(diameter 0)
 		(color 0 0 0 0)
@@
 	(wire
 		(pts
-			(xy 267.97 97.79) (xy 275.59 97.79)
+			(xy 327.66 72.39) (xy 335.28 72.39)
 		)
 		(stroke
@@
 	(wire
 		(pts
-			(xy 237.49 116.84) (xy 237.49 118.11)
+			(xy 297.18 91.44) (xy 297.18 92.71)
 		)
 		(stroke
@@
 	(wire
 		(pts
-			(xy 252.73 90.17) (xy 255.27 90.17)
+			(xy 312.42 64.77) (xy 314.96 64.77)
 		)
 		(stroke
@@
 	(wire
 		(pts
-			(xy 255.27 90.17) (xy 255.27 92.71)
+			(xy 314.96 64.77) (xy 314.96 67.31)
 		)
 		(stroke
@@
 	(wire
 		(pts
-			(xy 237.49 115.57) (xy 237.49 116.84)
+			(xy 297.18 90.17) (xy 297.18 91.44)
 		)
 		(stroke
@@
 	(wire
 		(pts
-			(xy 252.73 95.25) (xy 255.27 95.25)
+			(xy 312.42 69.85) (xy 314.96 69.85)
 		)
 		(stroke
@@
 	(wire
 		(pts
-			(xy 255.27 74.93) (xy 255.27 77.47)
+			(xy 314.96 49.53) (xy 314.96 52.07)
 		)
 		(stroke
@@
 	(wire
 		(pts
-			(xy 275.59 97.79) (xy 275.59 99.06)
+			(xy 335.28 72.39) (xy 335.28 73.66)
 		)
 		(stroke
@@
 	(wire
 		(pts
-			(xy 275.59 97.79) (xy 275.59 95.25)
+			(xy 335.28 72.39) (xy 335.28 69.85)
 		)
 		(stroke
@@
 	(wire
 		(pts
-			(xy 267.97 95.25) (xy 267.97 97.79)
+			(xy 327.66 69.85) (xy 327.66 72.39)
 		)
 		(stroke
@@
 	(wire
 		(pts
-			(xy 275.59 82.55) (xy 275.59 87.63)
+			(xy 335.28 57.15) (xy 335.28 62.23)
 		)
 		(stroke
@@
 	(wire
 		(pts
-			(xy 252.73 97.79) (xy 255.27 97.79)
+			(xy 312.42 72.39) (xy 314.96 72.39)
 		)
 		(stroke
@@
 	(wire
 		(pts
-			(xy 255.27 92.71) (xy 264.16 92.71)
+			(xy 314.96 67.31) (xy 323.85 67.31)
 		)
 		(stroke
@@
 	(wire
 		(pts
-			(xy 255.27 95.25) (xy 255.27 97.79)
+			(xy 314.96 69.85) (xy 314.96 72.39)
 		)
 		(stroke
@@
 	(wire
 		(pts
-			(xy 252.73 82.55) (xy 275.59 82.55)
+			(xy 312.42 57.15) (xy 335.28 57.15)
 		)
 		(stroke
@@
 	(wire
 		(pts
-			(xy 255.27 97.79) (xy 264.16 97.79)
+			(xy 314.96 72.39) (xy 323.85 72.39)
 		)
 		(stroke
@@
 	(wire
 		(pts
-			(xy 255.27 77.47) (xy 252.73 77.47)
+			(xy 314.96 52.07) (xy 312.42 52.07)
 		)
 		(stroke
@@
 	(wire
 		(pts
-			(xy 229.87 116.84) (xy 237.49 116.84)
+			(xy 289.56 91.44) (xy 297.18 91.44)
 		)
 		(stroke
@@
 	(wire
 		(pts
-			(xy 229.87 115.57) (xy 229.87 116.84)
+			(xy 289.56 90.17) (xy 289.56 91.44)
 		)
 		(stroke
@@
 	(wire
 		(pts
-			(xy 267.97 85.09) (xy 267.97 87.63)
+			(xy 327.66 59.69) (xy 327.66 62.23)
 		)
 		(stroke
@@
 	(wire
 		(pts
-			(xy 252.73 85.09) (xy 267.97 85.09)
+			(xy 312.42 59.69) (xy 327.66 59.69)
 		)
 		(stroke
@@
 	(wire
 		(pts
-			(xy 252.73 92.71) (xy 255.27 92.71)
+			(xy 312.42 67.31) (xy 314.96 67.31)
 		)
 		(stroke
@@
 	)
 	(label "USB_D-"
-		(at 264.16 92.71 180)
+		(at 323.85 67.31 180)
 		(effects
 			(font
@@
 	)
 	(label "USB_D+"
-		(at 264.16 97.79 180)
+		(at 323.85 72.39 180)
 		(effects
 			(font
@@
 	(symbol
 		(lib_id "Device:R")
-		(at 267.97 91.44 0)
+		(at 327.66 66.04 0)
 		(unit 1)
 		(exclude_from_sim no)
@@
 		(dnp no)
 		(property "Reference" "R16"
-			(at 271.272 90.17 0)
+			(at 330.962 64.77 0)
 			(effects
 				(font
@@
 		)
 		(property "Value" "5.1k"
-			(at 271.526 92.456 0)
+			(at 331.216 67.056 0)
 			(effects
 				(font
@@
 		)
 		(property "Footprint" ""
-			(at 266.192 91.44 90)
+			(at 325.882 66.04 90)
 			(effects
 				(font
@@
 		)
 		(property "Datasheet" "~"
-			(at 267.97 91.44 0)
+			(at 327.66 66.04 0)
 			(effects
 				(font
@@
 		)
 		(property "Description" "Resistor"
-			(at 267.97 91.44 0)
+			(at 327.66 66.04 0)
 			(effects
 				(font
@@
 	(symbol
 		(lib_id "Connector:USB_C_Receptacle_USB2.0_14P")
-		(at 237.49 92.71 0)
+		(at 297.18 67.31 0)
 		(unit 1)
 		(exclude_from_sim no)
@@
 		(dnp no)
 		(property "Reference" "J4"
-			(at 246.634 73.406 0)
+			(at 306.324 48.006 0)
 			(effects
 				(font
@@
 		)
 		(property "Value" "USB_C_Receptacle_USB2.0_14P"
-			(at 253.746 112.268 0)
+			(at 313.436 86.868 0)
 			(effects
 				(font
@@
 		)
 		(property "Footprint" ""
-			(at 241.3 92.71 0)
+			(at 300.99 67.31 0)
 			(effects
 				(font
@@
 		)
 		(property "Datasheet" "https://www.usb.org/sites/default/files/documents/usb_type-c.zip"
-			(at 241.3 92.71 0)
+			(at 300.99 67.31 0)
 			(effects
 				(font
@@
 		)
 		(property "Description" "USB 2.0-only 14P Type-C Receptacle connector"
-			(at 237.49 92.71 0)
+			(at 297.18 67.31 0)
 			(effects
 				(font
@@
 	(symbol
 		(lib_id "Device:R")
-		(at 275.59 91.44 0)
+		(at 335.28 66.04 0)
 		(unit 1)
 		(exclude_from_sim no)
@@
 		(dnp no)
 		(property "Reference" "R17"
-			(at 278.892 90.17 0)
+			(at 338.582 64.77 0)
 			(effects
 				(font
@@
 		)
 		(property "Value" "5.1k"
-			(at 279.146 92.456 0)
+			(at 338.836 67.056 0)
 			(effects
 				(font
@@
 		)
 		(property "Footprint" ""
-			(at 273.812 91.44 90)
+			(at 333.502 66.04 90)
 			(effects
 				(font
@@
 		)
 		(property "Datasheet" "~"
-			(at 275.59 91.44 0)
+			(at 335.28 66.04 0)
 			(effects
 				(font
@@
 		)
 		(property "Description" "Resistor"
-			(at 275.59 91.44 0)
+			(at 335.28 66.04 0)
 			(effects
 				(font
@@
 	(symbol
 		(lib_id "power:VBUS")
-		(at 255.27 74.93 0)
+		(at 314.96 49.53 0)
 		(unit 1)
 		(exclude_from_sim no)
@@
 		(fields_autoplaced yes)
 		(property "Reference" "#PWR060"
-			(at 255.27 78.74 0)
+			(at 314.96 53.34 0)
 			(effects
 				(font
@@
 		)
 		(property "Value" "VBUS"
-			(at 255.27 69.85 0)
+			(at 314.96 44.45 0)
 			(effects
 				(font
@@
 		)
 		(property "Footprint" ""
-			(at 255.27 74.93 0)
+			(at 314.96 49.53 0)
 			(effects
 				(font
@@
 		)
 		(property "Datasheet" ""
-			(at 255.27 74.93 0)
+			(at 314.96 49.53 0)
 			(effects
 				(font
@@
 		)
 		(property "Description" "Power symbol creates a global label with name \"VBUS\""
-			(at 255.27 74.93 0)
+			(at 314.96 49.53 0)
 			(effects
 				(font
@@
 	(symbol
 		(lib_id "power:GND")
-		(at 275.59 99.06 0)
+		(at 335.28 73.66 0)
 		(unit 1)
 		(exclude_from_sim no)
@@
 		(fields_autoplaced yes)
 		(property "Reference" "#PWR020"
-			(at 275.59 105.41 0)
+			(at 335.28 80.01 0)
 			(effects
 				(font
@@
 		)
 		(property "Value" "GND"
-			(at 275.59 104.14 0)
+			(at 335.28 78.74 0)
 			(effects
 				(font
@@
 		)
 		(property "Footprint" ""
-			(at 275.59 99.06 0)
+			(at 335.28 73.66 0)
 			(effects
 				(font
@@
 		)
 		(property "Datasheet" ""
-			(at 275.59 99.06 0)
+			(at 335.28 73.66 0)
 			(effects
 				(font
@@
 		)
 		(property "Description" "Power symbol creates a global label with name \"GND\" , ground"
-			(at 275.59 99.06 0)
+			(at 335.28 73.66 0)
 			(effects
 				(font
@@
 	(symbol
 		(lib_id "power:GND")
-		(at 237.49 118.11 0)
+		(at 297.18 92.71 0)
 		(unit 1)
 		(exclude_from_sim no)
@@
 		(fields_autoplaced yes)
 		(property "Reference" "#PWR021"
-			(at 237.49 124.46 0)
+			(at 297.18 99.06 0)
 			(effects
 				(font
@@
 		)
 		(property "Value" "GND"
-			(at 237.49 123.19 0)
+			(at 297.18 97.79 0)
 			(effects
 				(font
@@
 		)
 		(property "Footprint" ""
-			(at 237.49 118.11 0)
+			(at 297.18 92.71 0)
 			(effects
 				(font
@@
 		)
 		(property "Datasheet" ""
-			(at 237.49 118.11 0)
+			(at 297.18 92.71 0)
 			(effects
 				(font
@@
 		)
 		(property "Description" "Power symbol creates a global label with name \"GND\" , ground"
-			(at 237.49 118.11 0)
+			(at 297.18 92.71 0)
 			(effects
 				(font

Commit message: new card boxes
Other:
- note added: "1.1V Regulated Power"
- note added: "3.3V Regulated Power"
- note added: "3.3V Regulator"
- note added: "4.7u (32) here far from VREG"
- note added: "8080 Bus Signalling"
- note added: "Ground"
- note added: "I/O Expansion A (Optional)"
- note added: "I/O Expansion B (Optional)"
- note added: "Oscillator"
- note added: "Polarity dot on 1V1 side"
- note added: "Pull CC1 and CC2 down using 5.1k This advertises as a UFP"
- note added: "QSPI Flash"
- note added: "Run/Reset"
- note added: "Serial Wire Debug"
- note added: "TODO! Investigate reverse current protection (diode?)"
- note added: "USB Regulator (Programming)"
- note added: "USB Signalling"
- note added: "USB-C Port (Programming)"
- title: CPU Card for Miniaturized Altair 8800  -> Generic Card for Miniaturized Altair 8800 
- moved on the sheet: C10, C11, C12, C13, C14, C15, C16, C17, C18, C19, C20, C21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

Commit message: Ready for Layout
Parts:
- removed R11, R12, R13: 1k, symbol Device:R
- removed R14, R15: 27, symbol Device:R
- removed R16, R17: 5.1k, symbol Device:R
- removed R18, R19: 100k, symbol Device:R
- removed R21: 33, symbol Device:R
- added R34, R41, R42, R43: 1k, Resistor_SMD:R_0201_0603Metric_Pad0.64x0.40mm_HandSolder, symbol Device:R_US
- added R35, R36: 27, Resistor_SMD:R_0201_0603Metric_Pad0.64x0.40mm_HandSolder, symbol Device:R_US
- added R37, R38: 5.1k, Resistor_SMD:R_0201_0603Metric_Pad0.64x0.40mm_HandSolder, symbol Device:R_US
- added R39, R40: 100k, Resistor_SMD:R_0201_0603Metric_Pad0.64x0.40mm_HandSolder, symbol Device:R_US
- C27: renamed from C20; footprint (none) -> Capacitor_SMD:CP_Elec_3x5.4
- C28: renamed from C19; footprint (none) -> Capacitor_SMD:CP_Elec_3x5.4
- C29: renamed from C18; footprint (none) -> Capacitor_SMD:CP_Elec_3x5.4
- C30: renamed from C38; footprint (none) -> Capacitor_SMD:CP_Elec_3x5.4
- C31: renamed from C6; footprint (none) -> Capacitor_SMD:CP_Elec_3x5.4
- C32: renamed from C7; footprint (none) -> Capacitor_SMD:CP_Elec_3x5.4
- C33: renamed from C8; footprint (none) -> Capacitor_SMD:CP_Elec_3x5.4
- C34: renamed from C9; footprint (none) -> Capacitor_SMD:CP_Elec_3x5.4
- C35: renamed from C10; footprint (none) -> Capacitor_SMD:CP_Elec_3x5.4
- C36: renamed from C11; footprint (none) -> Capacitor_SMD:CP_Elec_3x5.4
- C37: renamed from C12; footprint (none) -> Capacitor_SMD:CP_Elec_3x5.4
- C38: renamed from C13; footprint (none) -> Capacitor_SMD:CP_Elec_3x5.4
- C39: renamed from C14; footprint (none) -> Capacitor_SMD:CP_Elec_3x5.4
- C40: renamed from C17; footprint (none) -> Capacitor_SMD:CP_Elec_3x5.4
- C41: renamed from C27; footprint (none) -> Capacitor_SMD:CP_Elec_3x5.4
- C42: renamed from C28; footprint (none) -> Capacitor_SMD:CP_Elec_3x5.4
- C43: renamed from C25; footprint (none) -> Capacitor_SMD:CP_Elec_3x5.4
- C44: renamed from C26; footprint (none) -> Capacitor_SMD:CP_Elec_3x5.4
- C45: renamed from C22; footprint (none) -> Capacitor_SMD:CP_Elec_3x5.4
- C46: renamed from C21; footprint (none) -> Capacitor_SMD:CP_Elec_3x5.4
- C47: renamed from C16; footprint (none) -> Capacitor_SMD:CP_Elec_3x5.4
- C48: renamed from C15; footprint (none) -> Capacitor_SMD:CP_Elec_3x5.4
- C53: renamed from C23; footprint (none) -> Capacitor_SMD:CP_Elec_3x5.4
- C54: renamed from C24; footprint (none) -> Capacitor_SMD:CP_Elec_3x5.4
- J3: renamed from J4; footprint (none) -> Connector_USB:USB_C_Receptacle_Palconn_UTC16-G
- J4: renamed from J3; footprint (none) -> Connector:Banana_Jack_1Pin
- JP27: renamed from JP16; footprint (none) -> Jumper:SolderJumper-3_P1.3mm_Open_RoundedPad1.0x1.5mm
- JP28: renamed from JP15; footprint (none) -> Jumper:SolderJumper-3_P1.3mm_Open_RoundedPad1.0x1.5mm
- JP29: renamed from JP14; footprint (none) -> Jumper:SolderJumper-3_P1.3mm_Open_RoundedPad1.0x1.5mm
- JP30: renamed from JP13; footprint (none) -> Jumper:SolderJumper-3_P1.3mm_Open_RoundedPad1.0x1.5mm
- JP31: renamed from JP12; footprint (none) -> Jumper:SolderJumper-3_P1.3mm_Open_RoundedPad1.0x1.5mm
- JP32: renamed from JP11; footprint (none) -> Jumper:SolderJumper-3_P1.3mm_Open_RoundedPad1.0x1.5mm
- JP33: renamed from JP10; footprint (none) -> Jumper:SolderJumper-3_P1.3mm_Open_RoundedPad1.0x1.5mm
- JP34: renamed from JP9; footprint (none) -> Jumper:SolderJumper-3_P1.3mm_Open_RoundedPad1.0x1.5mm
- JP35: renamed from JP8; footprint (none) -> Jumper:SolderJumper-3_P1.3mm_Open_RoundedPad1.0x1.5mm
- JP36: renamed from JP7; footprint (none) -> Jumper:SolderJumper-3_P1.3mm_Open_RoundedPad1.0x1.5mm
- JP37: renamed from JP6; footprint (none) -> Jumper:SolderJumper-3_P1.3mm_Open_RoundedPad1.0x1.5mm
- JP38: renamed from JP5; footprint (none) -> Jumper:SolderJumper-3_P1.3mm_Open_RoundedPad1.0x1.5mm
- JP39: renamed from JP4; footprint (none) -> Jumper:SolderJumper-3_P1.3mm_Open_RoundedPad1.0x1.5mm
- JP40: renamed from JP3; footprint (none) -> Jumper:SolderJumper-3_P1.3mm_Open_RoundedPad1.0x1.5mm
- JP41: renamed from JP2; footprint (none) -> Jumper:SolderJumper-3_P1.3mm_Open_RoundedPad1.0x1.5mm
- JP42: renamed from JP19; footprint (none) -> Jumper:SolderJumper-3_P1.3mm_Open_RoundedPad1.0x1.5mm
- L2: renamed from L3; footprint (none) -> Inductor_SMD:L_0201_0603Metric
- SW34: renamed from SW16; footprint (none) -> Button_Switch_THT:SW_Push_1P2T_Vertical_E-Switch_800UDP8P1A1M6
- SW36: renamed from SW15; footprint (none) -> Button_Switch_THT:SW_Push_1P2T_Vertical_E-Switch_800UDP8P1A1M6
- X2: footprint ABM8-272-T3_ABR -> Connector:Banana_Jack_1Pin
- renumbered U11 to U10, U10 to U11, U6 to U12, U8 to U13
Connections:
- net +3V3: now also R39.1, R40.1; no longer C47.1, U9.64 (VREG_VIN)
- net GND: now also R37.2, R38.2, R42.1
- net QSPI_SS: now also R43.2
- net USB_D+: now also R35.2
- net USB_D-: now also R36.2
- net ~{RESET}: now also R39.2, R40.2
- net ~{USB_BOOT}: now also R43.1
- net at SW36.1: now also R42.2
- net at J3.B5 (CC2): now also R37.1
- net at C53.2, X2.3: now also R41.1
- net at U9.31 (XOUT): now also R41.2
- net at J3.A5 (CC1): now also R38.1
- net at U9.66 (USB_DM): now also R36.1
- net at U9.67 (USB_DP): now also R35.1
- net VREG_AVDD: no longer names the net of C48.1, U9.61 (VREG_AVDD)
- net VREG_AVDD: now also R34.2
- new net 3.3V: C47.1, R34.1, U9.64 (VREG_VIN)
- no-connect marks 4 -> 20
Other:
- note added: "PWR_FLAGs"
- moved on the sheet: X2
