File: ecad (Updated)/front_panel/front_panel.kicad_sch (KiCad schematic)
At the start: 0 parts

Commit message: New Component Library
Parts:
- added C1, C10, C11, C12, C13, C14, C17, C2, C22, C23, C26, C4, C5, C6, C7, C8, C9: 100n, Capacitor_SMD:CP_Elec_3x5.4, symbol Device:C
- added C15, C20, C21: 10u, Capacitor_SMD:CP_Elec_3x5.4, symbol Device:C
- added C16, C18, C19, C3: 4.7u, Capacitor_SMD:CP_Elec_3x5.4, symbol Device:C
- added C24, C25: 15p, Capacitor_SMD:CP_Elec_3x5.4, symbol Device:C
- added D1: LED, LED_SMD:LED_Osram_Lx_P47F_D2mm_ReverseMount, symbol Device:LED
- added D10, D11, D12, D13, D14, D15, D16, D17, D18, D19, D2, D20, D21, D22, D23, D24, D3, D4, D5, D6, D7, D8, D9: LED, LED_SMD:LED_1206_3216Metric_ReverseMount_Hole1.8x2.4mm, symbol Device:LED
- added J1: USB_C_Receptacle_USB2.0_14P, Connector_USB:USB_C_Receptacle_Palconn_UTC16-G, symbol Connector:USB_C_Receptacle_USB2.0_14P
- added J2: Conn_01x03_Pin, Connector:Banana_Jack_1Pin, symbol Connector:Conn_01x03_Pin
- added L1: 3.3u, Inductor_SMD:L_0201_0603Metric, symbol Device:L
- added Q1, Q10, Q11, Q12, Q13, Q14, Q15, Q16, Q17, Q18, Q19, Q2, Q20, Q21, Q22, Q23, Q24, Q3, Q4, Q5, Q6, Q7, Q8, Q9: NMOS, Transistor_Power:GaN_Systems_GaNPX-3_5x6.6mm_Drain2.93x0.6mm, symbol Simulation_SPICE:NMOS
- added R1, R10, R11, R13, R14, R15, R16, R19, R2, R20, R22, R23, R25, R26, R27, R28, R29, R3, R30, R31, R32, R4, R5, R8: 220, Resistor_SMD:R_0201_0603Metric_Pad0.64x0.40mm_HandSolder, symbol Device:R_US
- added R12, R21, R24: 1k, Resistor_SMD:R_0201_0603Metric_Pad0.64x0.40mm_HandSolder, symbol Device:R_US
- added R17, R18: 5.1k, Resistor_SMD:R_0201_0603Metric_Pad0.64x0.40mm_HandSolder, symbol Device:R_US
- added R6: 33, Resistor_SMD:R_0201_0603Metric_Pad0.64x0.40mm_HandSolder, symbol Device:R_US
- added R7, R9: 27, Resistor_SMD:R_0201_0603Metric_Pad0.64x0.40mm_HandSolder, symbol Device:R_US
- added SW1, SW10, SW11, SW12, SW14, SW15, SW16, SW17, SW18, SW2, SW3, SW4, SW5, SW6, SW8, SW9: SW_SPDT, Button_Switch_THT:SW_E-Switch_EG1224_SPDT_Angled, symbol Switch:SW_SPDT
- added SW13: FRONT PANEL TEST SWTICH, Button_Switch_THT:SW_Push_1P2T_Vertical_E-Switch_800UDP8P1A1M6, symbol Switch:SW_Push
- added SW19, SW20, SW21, SW22, SW23, SW24, SW25, SW26, SW27, SW28, SW29, SW30, SW31, SW32: SW_Push, Button_Switch_THT:SW_Push_1P2T_Vertical_E-Switch_800UDP8P1A1M6, symbol Switch:SW_Push
- added SW33: SW_SPDT, Button_Switch_THT:SW_Push_1P2T_Vertical_E-Switch_800UDP8P1A1M6, symbol Switch:SW_SPDT
- added SW7: SPI TEST, Button_Switch_THT:SW_Push_1P2T_Vertical_E-Switch_800UDP8P1A1M6, symbol Switch:SW_Push
- added U1, U2, U3: TLC59211IN, footprints:N20, symbol 2025-02-26_04-26-50:TLC59211IN
- added U4: MCP23017_SO, Package_SO:SOIC-28W_7.5x17.9mm_P1.27mm, symbol Interface_Expansion:MCP23017_SO
- added U5: W25Q128JVS, Package_SO:SOIC-8_5.23x5.23mm_P1.27mm, symbol Memory_Flash:W25Q128JVS
- added U6: RP2350_80QFN, RP2350_80QFN_minimal:RP2350-QFN-80-1EP_10x10_P0.4mm_EP3.4x3.4mm_ThermalVias, symbol MCU_RaspberryPi_RP2350:RP2350_80QFN
- added U7: NCP1117-3.3_SOT223, Package_TO_SOT_SMD:SOT-223-3_TabPin2, symbol Regulator_Linear:NCP1117-3.3_SOT223
- added X1: ABM8-272-T3, Connector:Banana_Jack_1Pin, symbol 2025-02-12_11-47-03:ABM8-272-T3
Connections:
- new net: D22.2 (A), R30.1
- new net: D13.2 (A), R19.1
- new net: D12.2 (A), R16.1
- new net: J1.A5 (CC1), R17.1
- new net: J1.B5 (CC2), R18.1
- new net: D15.2 (A), R22.1
- new net: U5.2 (DO(IO1)), U6.73 (QSPI_SD2)
- new net: U5.3 (IO2), U6.74 (QSPI_SD1)
- new net: U5.5 (DI(IO0)), U6.70 (QSPI_SD3)
- new net: U5.6 (CLK), U6.71 (QSPI_SCLK)
- new net: U5.7 (IO3), U6.72 (QSPI_SD0)
- new net: R9.1, U6.66 (USB_DM)
- new net: D8.2 (A), R11.1
- new net: R24.1, SW13.1
- new net: SW13.2, U6.35 (RUN)
- new net: D19.2 (A), R27.1
- new net: D5.2 (A), R5.1
- new net: R7.1, U6.67 (USB_DP)
- new net: D17.2 (A), R25.1
- new net: D9.2 (A), R13.1
- new net: D11.2 (A), R15.1
- new net: D18.2 (A), R26.1
- new net: D6.2 (A), R8.1
- new net: D7.2 (A), R10.1
- new net: D14.2 (A), R20.1
- new net: D3.2 (A), R3.1
- new net: C25.2, R21.1, X1.3
- new net: D23.2 (A), R31.1
- new net: D20.2 (A), R28.1
- new net: R21.2, U6.31 (XOUT)
- new net: D2.2 (A), R2.1
- new net: C24.1, U6.30 (XIN), X1.1
- new net: D21.2 (A), R29.1
- new net: D16.2 (A), R23.1
- new net: D4.2 (A), R4.1
- new net: D24.2 (A), R32.1
- new net: D1.2 (A), R1.1
- new net: C16.2, R6.2, U6.61 (VREG_AVDD)
- new net: D10.2 (A), R14.1
- new net: J2.1 (Pin_1), U6.33 (SWCLK)
- new net: J2.3 (Pin_3), U6.34 (SWD)
- new net +1V1: C19.1, C2.1, C3.1, C4.1, L1.1, U6.10 (DVDD), U6.32 (DVDD), U6.51 (DVDD), U6.65 (VREG_FB)
- new net +3V3: C10.1, C11.1, C12.1, C13.1, C14.1, C15.1, C18.1, C23.1, C5.1, C6.1, C7.1, C8.1, C9.1, R6.1, U5.8 (VCC), U6.15 (IOVDD), U6.24 (IOVDD), U6.29 (IOVDD), U6.41 (IOVDD), U6.5 (IOVDD), U6.50 (IOVDD), U6.59 (ADC_AVDD), U6.60 (IOVDD), U6.64 (VREG_VIN), U6.68 (USB_OTP_VDD), U6.69 (QSPI_IOVDD), U6.76 (IOVDD)
- new net 3.3V: C1.1, C17.1, C21.1, C22.1, C26.1, R1.2, R10.2, R11.2, R13.2, R14.2, R15.2, R16.2, R19.2, R2.2, R20.2, R22.2, R23.2, R25.2, R26.2, R27.2, R28.2, R29.2, R3.2, R30.2, R31.2, R32.2, R4.2, R5.2, R8.2, SW1.2 (B), SW10.2 (B), SW11.2 (B), SW12.2 (B), SW14.2 (B), SW15.2 (B), SW16.2 (B), SW17.2 (B), SW18.2 (B), SW19.1, SW2.2 (B), SW20.1, SW21.1, SW22.1, SW23.1, SW24.1, SW25.1, SW26.1, SW27.1, SW28.1, SW29.1, SW3.2 (B), SW30.1, SW31.1, SW32.1, SW33.2 (B), SW4.2 (B), SW5.2 (B), SW6.2 (B), SW8.2 (B), SW9.2 (B), U1.20 (VCC), U2.20 (VCC), U3.20 (VCC), U4.9 (VDD), U7.2 (VO)
- new net A0: Q1.2 (G), SW1.1 (A), U1.2 (D1)
- new net A0_LED: D1.1 (K), U1.19 (*Y1)
- new net A1: Q2.2 (G), SW2.1 (A), U1.3 (D2)
- new net A10: Q11.2 (G), SW12.1 (A), U2.4 (D3)
- new net A10_LED: D11.1 (K), U2.17 (*Y3)
- new net A11: Q12.2 (G), SW14.1 (A), U2.5 (D4)
- new net A11_LED: D12.1 (K), U2.16 (*Y4)
- new net A12: Q13.2 (G), SW15.1 (A), U2.6 (D5)
- new net A12_LED: D13.1 (K), U2.15 (*Y5)
- new net A13: Q14.2 (G), SW16.1 (A), U2.7 (D6)
- new net A13_LED: D14.1 (K), U2.14 (*Y6)
- new net A14: Q15.2 (G), SW17.1 (A), U2.8 (D7)
- new net A14_LED: D15.1 (K), U2.13 (*Y7)
- new net A15: Q16.2 (G), SW18.1 (A), U2.9 (D8)
- new net A15_LED: D16.1 (K), U2.12 (*Y8)
- new net A1_LED: D2.1 (K), U1.18 (*Y2)
- new net A2: Q3.2 (G), SW3.1 (A), U1.4 (D3)
- new net A2_LED: D3.1 (K), U1.17 (*Y3)
- new net A3: Q4.2 (G), SW4.1 (A), U1.5 (D4)
- new net A3_LED: D4.1 (K), U1.16 (*Y4)
- new net A4: Q5.2 (G), SW5.1 (A), U1.6 (D5)
- new net A4_LED: D5.1 (K), U1.15 (*Y5)
- new net A5: Q6.2 (G), SW6.1 (A), U1.7 (D6)
- new net A5_LED: D6.1 (K), U1.14 (*Y6)
- new net A6: Q7.2 (G), SW8.1 (A), U1.8 (D7)
- new net A6_LED: D7.1 (K), U1.13 (*Y7)
- new net A7: Q8.2 (G), SW9.1 (A), U1.9 (D8)
- new net A7_LED: D8.1 (K), U1.12 (*Y8)
- new net A8: Q9.2 (G), SW10.1 (A), U2.2 (D1)
- new net A8_LED: D9.1 (K), U2.19 (*Y1)
- new net A9: Q10.2 (G), SW11.1 (A), U2.3 (D2)
- new net A9_LED: D10.1 (K), U2.18 (*Y2)
- new net ADDR00: U6.25 (GPIO24)
- new net ADDR01: U6.26 (GPIO25)
- new net ADDR02: U6.27 (GPIO26)
- new net ADDR03: U6.28 (GPIO27)
- new net ADDR04: U6.36 (GPIO28)
- new net ADDR05: U6.37 (GPIO29)
- new net ADDR06: U6.38 (GPIO30)
- new net ADDR07: U6.39 (GPIO31)
- new net ADDR08: U6.40 (GPIO32)
- new net ADDR09: U6.42 (GPIO33)
- new net ADDR10: U6.43 (GPIO34)
- new net ADDR11: U6.44 (GPIO35)
- new net ADDR12: U6.45 (GPIO36)
- new net ADDR13: U6.46 (GPIO37)
- new net ADDR14: U6.47 (GPIO38)
- new net ADDR15: U6.48 (GPIO39)
- new net AUX1: SW31.2
- new net AUX2: SW32.2
- new net BUS04: U6.77 (GPIO0)
- new net BUS05: U6.78 (GPIO1)
- new net BUS06: U6.79 (GPIO2)
- new net BUS07: U6.80 (GPIO3)
- new net BUS20: U6.13 (GPIO14)
- new net BUS21: U6.14 (GPIO15)
- new net BUS22: U6.16 (GPIO16)
- new net BUS23: U6.17 (GPIO17)
- new net CLR: SW28.2
- new net COL1: Q1.3 (S), Q13.3 (S), Q17.3 (S), Q21.3 (S), Q5.3 (S), Q9.3 (S), U4.7 (GPB6)
- new net COL2: Q10.3 (S), Q14.3 (S), Q18.3 (S), Q2.3 (S), Q22.3 (S), Q6.3 (S), U4.8 (GPB7)
- new net COL3: Q11.3 (S), Q15.3 (S), Q19.3 (S), Q23.3 (S), Q3.3 (S), Q7.3 (S), U4.21 (GPA0)
- new net COL4: Q12.3 (S), Q16.3 (S), Q20.3 (S), Q24.3 (S), Q4.3 (S), Q8.3 (S), U4.22 (GPA1)
- new net D0: Q17.2 (G), U3.2 (D1)
- new net D0_LED: D17.1 (K), U3.19 (*Y1)
- new net D1: Q18.2 (G), U3.3 (D2)
- new net D1_LED: D18.1 (K), U3.18 (*Y2)
- new net D2: Q19.2 (G), U3.4 (D3)
- new net D2_LED: D19.1 (K), U3.17 (*Y3)
- new net D3: Q20.2 (G), U3.5 (D4)
- new net D3_LED: D20.1 (K), U3.16 (*Y4)
- new net D4: Q21.2 (G), U3.6 (D5)
- new net D4_LED: D21.1 (K), U3.15 (*Y5)
- new net D5: Q22.2 (G), U3.7 (D6)
- new net D5_LED: D22.1 (K), U3.14 (*Y6)
- new net D6: Q23.2 (G), U3.8 (D7)
- new net D6_LED: D23.1 (K), U3.13 (*Y7)
- new net D7: Q24.2 (G), U3.9 (D8)
- new net D7_LED: D24.1 (K), U3.12 (*Y8)
- new net DATA0: U6.49 (GPIO40_ADC0)
- new net DATA1: U6.52 (GPIO41_ADC1)
- new net DATA2: U6.53 (GPIO42_ADC2)
- new net DATA3: U6.54 (GPIO43_ADC3)
- new net DATA4: U6.55 (GPIO44_ADC4)
- new net DATA5: U6.56 (GPIO45_ADC5)
- new net DATA6: U6.57 (GPIO46_ADC6)
- new net DATA7: U6.58 (GPIO47_ADC7)
- new net DEPOSIT: SW25.2
- new net DEPOSIT_NEXT: SW26.2
- new net EXAMINE: SW23.2
- new net EXAMINE_NEXT: SW24.2
- new net GND: C1.2, C10.2, C11.2, C12.2, C13.2, C14.2, C15.2, C16.1, C17.2, C18.2, C19.2, C2.2, C20.2, C21.2, C22.2, C23.2, C24.2, C25.1, C26.2, C3.2, C4.2, C5.2, C6.2, C7.2, C8.2, C9.2, J1.A1 (GND), J1.A12 (GND), J1.B1 (GND), J1.B12 (GND), J1.S1 (SHIELD), J2.2 (Pin_2), R17.2, R18.2, R24.2, SW1.3 (C), SW10.3 (C), SW11.3 (C), SW12.3 (C), SW14.3 (C), SW15.3 (C), SW16.3 (C), SW17.3 (C), SW18.3 (C), SW2.3 (C), SW3.3 (C), SW33.3 (C), SW4.3 (C), SW5.3 (C), SW6.3 (C), SW7.1, SW8.3 (C), SW9.3 (C), U1.11 (GND), U2.11 (GND), U3.11 (GND), U4.10 (VSS), U4.15 (A0), U4.16 (A1), U4.17 (A2), U5.4 (GND), U6.62 (VREG_PGND), U6.81 (GND), U7.1 (GND), X1.2, X1.4
- new net IQR_Handler_COL: U4.20 (INTA)
- new net IQR_Handler_ROW: U4.19 (INTB)
- new net ON: SW33.1 (A), U4.18 (~{RESET})
- new net PROTECT: SW29.2
- new net QSPI_SS: R12.2, U5.1 (~{CS}), U6.75 (QSPI_SS)
- new net RESET: SW27.2
- new net ROW1: Q1.1 (D), Q2.1 (D), Q3.1 (D), Q4.1 (D), U4.1 (GPB0)
- new net ROW2: Q5.1 (D), Q6.1 (D), Q7.1 (D), Q8.1 (D), U4.2 (GPB1)
- new net ROW3: Q10.1 (D), Q11.1 (D), Q12.1 (D), Q9.1 (D), U4.3 (GPB2)
- new net ROW4: Q13.1 (D), Q14.1 (D), Q15.1 (D), Q16.1 (D), U4.4 (GPB3)
- new net ROW5: Q17.1 (D), Q18.1 (D), Q19.1 (D), Q20.1 (D), U4.5 (GPB4)
- new net ROW6: Q21.1 (D), Q22.1 (D), Q23.1 (D), Q24.1 (D), U4.6 (GPB5)
- new net RUN: SW20.2
- new net SCL: U4.12 (SCK), U6.1 (GPIO4)
- new net SDA: U4.13 (SDA), U6.2 (GPIO5)
- new net SINGLE: SW21.2
- new net STEP: SW22.2
- new net STOP: SW19.2
- new net UNPROTECT: SW30.2
- new net USB_D+: J1.A6 (D+), J1.B6 (D+), R7.2
- new net USB_D-: J1.A7 (D-), J1.B7 (D-), R9.2
- new net VBUS: C20.1, J1.A4 (VBUS), J1.A9 (VBUS), J1.B4 (VBUS), J1.B9 (VBUS), U7.3 (VI)
- new net VREG_LX: L1.2, U6.63 (VREG_LX)
- new net ~{USB_BOOT}: R12.1, SW7.2
- no-connect marks 0 -> 44
Other:
- note added: "*(1) BOLD ON A LABEL MEANS IT IS NOT CURRENTLY BEING USED"
- note added: "*1 OPTIONAL LABELS, MAY USE LATER"
- note added: "*Figure out later"
- note added: "*How are we going to get 1V1 and 3V3 Lines?"
- note added: "*How are we going to reset to whole device?"
- note added: "53, 54, 68, 69 SHARE PINS"
- note added: "ADDRESS I/O EXPANDER"
- note added: "ADDRESS LINE LEDs"
- note added: "Converted Size: X inches (length of front panel) x X inches (height of front panel) x X inches (depth of machine)"
- note added: "DATA LINE LEDs"
- note added: "DECOUPLING CAPACITORS (11)"
- note added: "DECOUPLING CAPACITORS (3)"
- note added: "EXTERNAL OSCILLATOR"
- note added: "FOOTNOTES"
- note added: "FRONT PANEL (NEW)"
- note added: "FRONT PANEL (OLD)"
- note added: "KEEP D- and D+ Pins Close"
- note added: "LEDs"
- note added: "MATRIX SCANNING"
- note added: "MICROCONTROLLER (1)"
- note added: "ON (IMPORTANT)"
- note added: "Original Size: 17 inches (length of front panel) x 7 inches (height of front panel) x 18 inches (depth of machine)"
- note added: "PWR_FLAGs"
- note added: "QSPI + CS"
- note added: "QUESTIONS"
- note added: "SINK DRIVERS"
- note added: "SWITCHES"
- note added: "USB Connector"
- note added: "VIOLATION EXCLUSIONS (REMOVE LATER)"
- note added: "VOLTAGE LEVEL REGULATOR"
- note added: "VOLTAGE REGULATION"
