File: ecad/panel/panel.kicad_sch (KiCad schematic)
At the start: 161 parts, among them J1 10145226-0241N13LF, J2 Conn_01x03_Pin, J3 USB4105-GF-A, J4 5017868090, SW1 SW_SPDT, SW10 SW_SPDT, SW11 SW_SPDT, SW12 SW_SPDT, SW13 SW_SPDT, SW14 SW_SPDT, SW15 SW_SPDT, SW16 SW_SPDT, SW17 SW_Push, SW18 SW_Push, SW19 SW_Push, SW2 SW_SPDT, SW20 SW_Push, SW21 SW_Push, SW22 SW_Push, SW23 SW_Push, SW24 SW_Push, SW25 SW_Push, SW26 SW_Push, SW27 SW_Push, SW28 SW_Push, SW29 SW_Push, SW3 SW_SPDT, SW30 SW_Push, SW31 SW_Push, SW4 SW_SPDT, SW5 SW_SPDT, SW6 SW_SPDT, SW7 SW_SPDT, SW8 SW_SPDT, SW9 SW_SPDT, U1 TLC59211IN, U2 TLC59211IN, U3 TLC59211IN, U4 TLC59211IN, U5 TLC59211IN, U6 RP2350_80QFN, U7 W25Q128JVS, U8 MCP23017_SO, U9 MCP23017_SO, X1 ABM8-272-T3

Commit message: PCB Changes
Other:
- note added: "ADDR00"
- note added: "ADDR01"
- note added: "ADDR02"
- note added: "ADDR03"
- note added: "ADDR04"
- note added: "ADDR05"
- note added: "ADDR06"
- note added: "ADDR07"
- note added: "ADDR08"
- note added: "ADDR09"
- note added: "ADDR10"
- note added: "ADDR11"
- note added: "ADDR12"
- note added: "ADDR13"
- note added: "ADDR14"
- note added: "ADDR15"
- note added: "BUS00"
- note added: "BUS01"
- note added: "BUS02"
- note added: "BUS03"
- note added: "BUS04"
- note added: "BUS05"
- note added: "BUS06"
- note added: "BUS07"
- note added: "BUS08"
- note added: "BUS09"
- note added: "BUS10"
- note added: "BUS11"
- note added: "BUS12"
- note added: "BUS13"
- note added: "BUS14"
- note added: "BUS15"
- note added: "BUS16"
- note added: "BUS17"
- note added: "BUS18"
- note added: "BUS19"
- note added: "DATA00"
- note added: "DATA01"
- note added: "DATA02"
- note added: "DATA03"
- note added: "DATA04"
- note added: "DATA05"
- note added: "DATA06"
- note added: "DATA07"
- note added: "UNUSED"
- note added: "USED"
- note added: "https://upload.wikimedia.org/wikipedia/commons/b/b2/MITS_Altair_8800_Front_Panel.jpg"
- moved on the sheet: J3, JP1, JP2, JP3, JP4, JP5, JP6, JP7, JP8, R29, R30

Commit message: Update PCB
Parts:
- removed JP1, JP3, JP5, JP7: Jumper_2_Bridged, Resistor_SMD:R_0402_1005Metric_Pad0.72x0.64mm_HandSolder, symbol Jumper:Jumper_2_Bridged
- removed JP2, JP4, JP6, JP8: Jumper_2_Open, Resistor_SMD:R_0402_1005Metric_Pad0.72x0.64mm_HandSolder, symbol Jumper:Jumper_2_Open
- J4: footprint CON_5017868090 -> Library:CON_5017868090
- U8, U9: footprint Package_SO:SOIC-28W_7.5x17.9mm_P1.27mm -> Library:QFN28_IO_Expander
- renumbered U3 to U2, U2 to U3
Connections:
- net BUS01 is gone; now on net A10: J4.15, U6.22 (GPIO22)
- net BUS04 is gone; now on net D7: J4.63, U6.19 (GPIO19)
- net BUS05 is gone; now on net D6: J4.17, U6.18 (GPIO18)
- net BUS08 is gone; now on net D3: J4.59, U6.14 (GPIO15)
- net BUS11 is gone; now on net D0: J4.22, U6.11 (GPIO12)
- net BUS17 is gone; now on net A2: J4.27, U6.3 (GPIO6)
- net BUS18 is gone; now on net A1: J4.52, U6.2 (GPIO5)
- net BUS19 is gone; now on net A0: J4.28, U6.1 (GPIO4)
- net I2C0_SCK is gone; now on net BUS22: U8.12 (SCK)
- net I2C0_SDA is gone; now on net BUS23: U8.13 (SDA)
- net I2C1_SCK is gone; now on net BUS20: U9.12 (SCK)
- net I2C1_SDA is gone; now on net BUS21: U9.13 (SDA)
- net A0: no longer J4.77, U6.25 (GPIO24)
- net A1: no longer J4.3, U6.26 (GPIO25)
- net A10: no longer J4.70, U6.43 (GPIO34)
- net A11: now also J4.65, U6.23 (GPIO23); no longer J4.10, U6.44 (GPIO35)
- net A12: now also J4.77, U6.25 (GPIO24); no longer J4.69, U6.45 (GPIO36)
- net A13: now also J4.3, U6.26 (GPIO25); no longer J4.11, U6.46 (GPIO37)
- net A14: now also J4.76, U6.27 (GPIO26); no longer J4.68, U6.47 (GPIO38)
- net A15: now also J4.4, U6.28 (GPIO27); no longer J4.12, U6.48 (GPIO39)
- net A2: no longer J4.76, U6.27 (GPIO26)
- net A3: now also J4.53, U6.4 (GPIO7); no longer J4.4, U6.28 (GPIO27)
- net A4: now also J4.24, U6.6 (GPIO8); no longer J4.75, U6.36 (GPIO28)
- net A5: now also J4.56, U6.7 (GPIO9); no longer J4.5, U6.37 (GPIO29)
- net A6: now also J4.23, U6.8 (GPIO10); no longer J4.74, U6.38 (GPIO30)
- net A7: now also J4.57, U6.9 (GPIO11); no longer J4.6, U6.39 (GPIO31)
- net A8: now also J4.16, U6.20 (GPIO20); no longer J4.71, U6.40 (GPIO32)
- net A9: now also J4.64, U6.21 (GPIO21); no longer J4.9, U6.42 (GPIO33)
- net BUS20: now also U6.80 (GPIO3)
- net BUS21: now also U6.79 (GPIO2)
- net BUS22: now also U6.78 (GPIO1)
- net BUS23: now also U6.77 (GPIO0)
- net D0: no longer J4.47, U6.49 (GPIO40_ADC0)
- net D1: now also J4.58, U6.12 (GPIO13); no longer J4.33, U6.52 (GPIO41_ADC1)
- net D2: now also J4.21, U6.13 (GPIO14); no longer J4.46, U6.53 (GPIO42_ADC2)
- net D3: no longer J4.34, U6.54 (GPIO43_ADC3)
- net D4: now also J4.18, U6.16 (GPIO16); no longer J4.45, U6.55 (GPIO44_ADC4)
- net D5: now also J4.62, U6.17 (GPIO17); no longer J4.35, U6.56 (GPIO45_ADC5)
- net D6: no longer J4.44, U6.57 (GPIO46_ADC6)
- net D7: no longer J4.36, U6.58 (GPIO47_ADC7)
- net HDLA_LED: now also U5.12 (*Y8); no longer U5.16 (*Y4)
- net HLDA: now also J4.68, U5.7 (D6), U6.47 (GPIO38); no longer J4.57, U5.5 (D4), U6.9 (GPIO11)
- net HLTA: now also J4.6, U4.6 (D5), U6.39 (GPIO31); no longer J4.56, U4.3 (D2), U6.7 (GPIO9)
- net INP: now also J4.70, U4.3 (D2), U6.43 (GPIO34); no longer J4.62, U4.6 (D5), U6.17 (GPIO17)
- net INT: now also J4.75, U6.36 (GPIO28); no longer J4.64, U5.3 (D2), U6.21 (GPIO21)
- net INTE: now also J4.11, U5.8 (D7), U6.46 (GPIO37); no longer J4.65, U6.23 (GPIO23)
- net INT_LED: now also U5.14 (*Y6); no longer U5.18 (*Y2)
- net M1: now also J4.9, U4.4 (D3), U6.42 (GPIO33); no longer J4.24, U4.5 (D4), U6.6 (GPIO8)
- net MEMR: now also J4.10, U4.2 (D1), U6.44 (GPIO35); no longer J4.16, U4.7 (D6), U6.20 (GPIO20)
- net OUT: now also J4.71, U4.5 (D4), U6.40 (GPIO32); no longer J4.18, U4.4 (D3), U6.16 (GPIO16)
- net PROT: now also J4.69, U5.9 (D8), U6.45 (GPIO36); no longer J4.53, U4.8 (D7), U6.4 (GPIO7)
- net STACK: now also J4.74, U4.7 (D6), U6.38 (GPIO30); no longer J4.23, U4.2 (D1), U6.8 (GPIO10)
- net WAIT: now also J4.12, U5.6 (D5), U6.48 (GPIO39); no longer J4.21, U5.2 (D1), U6.13 (GPIO14)
- net WAIT_LED: now also U5.13 (*Y7); no longer U5.17 (*Y3)
- net WO: now also J4.5, U4.8 (D7), U6.37 (GPIO29); no longer J4.58, U5.4 (D3), U6.12 (GPIO13)
- net WO_LED: now also U5.15 (*Y5); no longer U5.19 (*Y1)
- new net DATA00: J4.47, U6.49 (GPIO40_ADC0)
- new net DATA01: J4.33, U6.52 (GPIO41_ADC1)
- new net DATA02: J4.46, U6.53 (GPIO42_ADC2)
- new net DATA03: J4.34, U6.54 (GPIO43_ADC3)
- new net DATA04: J4.45, U6.55 (GPIO44_ADC4)
- new net DATA05: J4.35, U6.56 (GPIO45_ADC5)
- new net DATA06: J4.44, U6.57 (GPIO46_ADC6)
- new net DATA07: J4.36, U6.58 (GPIO47_ADC7)
Other:
- note added: "I2C LINES"
- note removed: "JUMPERS"

Commit message: change
Parts:
- added R45, R46, R47, R48, R49, R50, R51, R52, R53, R54, R55, R56, R57, R58, R59, R60, R61, R62, R63, R64, R65, R66, R67, R68, R69, R70, R71, R72, R73, R74, R75, R76, R77, R78, R79, R80, R81, R82, R83, R84, R85, R86, R87, R88: 330, Resistor_SMD:R_0402_1005Metric_Pad0.72x0.64mm_HandSolder, symbol Device:R_Small
- SW17, SW18, SW19, SW20, SW21, SW22, SW23, SW24, SW25, SW26, SW27, SW28, SW29, SW30, SW31: footprint Library:SW_1437565-5 -> Library:SW_1825910-6-4
- renumbered U3 to U2, U2 to U3
Connections:
- net A0: now also J4.16, U5.2 (D1), R80.2; no longer J4.28, U1.9 (D8), U6.1 (GPIO4)
- net A0_LED: now also U5.19 (*Y1); no longer U1.19 (*Y1)
- net A0_SW: now also U9.8 (GPB7); no longer U8.1 (GPB0)
- net A1: now also J4.17, U5.3 (D2), R79.2; no longer J4.52, U1.8 (D7), U6.2 (GPIO5)
- net A10: now also J4.46, U3.4 (D3), R62.2; no longer J4.15, U2.7 (D6), U6.22 (GPIO22)
- net A10_LED: now also U3.17 (*Y3); no longer U2.17 (*Y3)
- net A10_SW: now also U8.6 (GPB5); no longer U8.23 (GPA2)
- net A11: now also J4.47, U3.5 (D4), R61.2; no longer J4.65, U2.6 (D5), U6.23 (GPIO23)
- net A11_LED: now also U3.16 (*Y4); no longer U2.16 (*Y4)
- net A11_SW: now also U8.5 (GPB4); no longer U8.24 (GPA3)
- net A12: now also J4.50, U3.6 (D5), R60.2; no longer J4.77, U2.5 (D4), U6.25 (GPIO24)
- net A12_LED: now also U3.15 (*Y5); no longer U2.15 (*Y5)
- net A12_SW: now also U8.4 (GPB3); no longer U8.25 (GPA4)
- net A13: now also J4.51, U3.7 (D6), R59.2; no longer J4.3, U2.4 (D3), U6.26 (GPIO25)
- net A13_LED: now also U3.14 (*Y6); no longer U2.14 (*Y6)
- net A13_SW: now also U8.3 (GPB2); no longer U8.26 (GPA5)
- net A14: now also J4.52, U3.8 (D7), R58.2; no longer J4.76, U2.3 (D2), U6.27 (GPIO26)
- net A14_LED: now also U3.13 (*Y7); no longer U2.13 (*Y7)
- net A14_SW: now also U8.2 (GPB1); no longer U8.27 (GPA6)
- net A15: now also J4.53, U3.9 (D8), R57.2; no longer J4.4, U2.2 (D1), U6.28 (GPIO27)
- net A15_LED: now also U3.12 (*Y8); no longer U2.12 (*Y8)
- net A15_SW: now also U8.1 (GPB0); no longer U8.28 (GPA7)
- net A1_LED: now also U5.18 (*Y2); no longer U1.18 (*Y2)
- net A1_SW: now also U9.7 (GPB6); no longer U8.2 (GPB1)
- net A2: now also J4.18, U5.4 (D3), R78.2; no longer J4.27, U1.7 (D6), U6.3 (GPIO6)
- net A2_LED: now also U5.17 (*Y3); no longer U1.17 (*Y3)
- net A2_SW: now also U9.6 (GPB5); no longer U8.3 (GPB2)
- net A3: now also J4.21, U5.5 (D4), R77.2; no longer J4.53, U1.6 (D5), U6.4 (GPIO7)
- net A3_LED: now also U5.16 (*Y4); no longer U1.16 (*Y4)
- net A3_SW: now also U9.5 (GPB4); no longer U8.4 (GPB3)
- net A4: now also J4.22, U5.6 (D5), R76.2; no longer J4.24, U1.5 (D4), U6.6 (GPIO8)
- net A4_LED: now also U5.15 (*Y5); no longer U1.15 (*Y5)
- net A4_SW: now also U9.4 (GPB3); no longer U8.5 (GPB4)
- net A5: now also J4.23, U5.7 (D6), R75.2; no longer J4.56, U1.4 (D3), U6.7 (GPIO9)
- net A5_LED: now also U5.14 (*Y6); no longer U1.14 (*Y6)
- net A5_SW: now also U9.3 (GPB2); no longer U8.6 (GPB5)
- net A6: now also J4.24, U5.8 (D7), R74.2; no longer J4.23, U1.3 (D2), U6.8 (GPIO10)
- net A6_LED: now also U5.13 (*Y7); no longer U1.13 (*Y7)
- net A6_SW: now also U9.2 (GPB1); no longer U8.7 (GPB6)
- net A7: now also J4.27, U5.9 (D8), R73.2; no longer J4.57, U1.2 (D1), U6.9 (GPIO11)
- net A7_LED: now also U5.12 (*Y8); no longer U1.12 (*Y8)
- net A7_SW: now also U9.1 (GPB0); no longer U8.8 (GPB7)
- net A8: now also J4.44, U3.2 (D1), R64.2; no longer J4.16, U2.9 (D8), U6.20 (GPIO20)
- net A8_LED: now also U3.19 (*Y1); no longer U2.19 (*Y1)
- net A8_SW: now also U8.8 (GPB7); no longer U8.21 (GPA0)
- net A9: now also J4.45, U3.3 (D2), R63.2; no longer J4.64, U2.8 (D7), U6.21 (GPIO21)
- net A9_LED: now also U3.18 (*Y2); no longer U2.18 (*Y2)
- net A9_SW: now also U8.7 (GPB6); no longer U8.22 (GPA1)
- net AUX1: now also U9.22 (GPA1); no longer U9.25 (GPA4)
- net AUX2: now also U9.21 (GPA0); no longer U9.26 (GPA5)
- net CLR: now also U9.25 (GPA4); no longer U9.22 (GPA1)
- net D0: now also J4.28, U4.2 (D1), R72.2; no longer J4.22, U3.9 (D8), U6.11 (GPIO12)
- net D0_LED: now also U4.19 (*Y1); no longer U3.19 (*Y1)
- net D1: now also J4.29, U4.3 (D2), R71.2; no longer J4.58, U3.8 (D7), U6.12 (GPIO13)
- net D1_LED: now also U4.18 (*Y2); no longer U3.18 (*Y2)
- net D2: now also J4.30, U4.4 (D3), R70.2; no longer J4.21, U3.7 (D6), U6.13 (GPIO14)
- net D2_LED: now also U4.17 (*Y3); no longer U3.17 (*Y3)
- net D3: now also J4.33, U4.5 (D4), R69.2; no longer J4.59, U3.6 (D5), U6.14 (GPIO15)
- net D3_LED: now also U4.16 (*Y4); no longer U3.16 (*Y4)
- net D4: now also J4.34, U4.6 (D5), R68.2; no longer J4.18, U3.5 (D4), U6.16 (GPIO16)
- net D4_LED: now also U4.15 (*Y5); no longer U3.15 (*Y5)
- net D5: now also J4.35, U4.7 (D6), R67.2; no longer J4.62, U3.4 (D3), U6.17 (GPIO17)
- net D5_LED: now also U4.14 (*Y6); no longer U3.14 (*Y6)
- net D6: now also J4.36, U4.8 (D7), R66.2; no longer J4.17, U3.3 (D2), U6.18 (GPIO18)
- net D6_LED: now also U4.13 (*Y7); no longer U3.13 (*Y7)
- net D7: now also U4.9 (D8), R65.2; no longer J4.63, U3.2 (D1), U6.19 (GPIO19)
- net D7_LED: now also U4.12 (*Y8); no longer U3.12 (*Y8)
- net DEPOSIT: now also U8.21 (GPA0); no longer U9.7 (GPB6)
- net DEPOSIT_NEXT: now also U8.22 (GPA1); no longer U9.8 (GPB7)
- net EXAMINE: now also U8.23 (GPA2); no longer U9.5 (GPB4)
- net EXAMINE_NEXT: now also U8.24 (GPA3); no longer U9.6 (GPB5)
- net HDLA_LED: now also U1.15 (*Y5); no longer U5.12 (*Y8)
- net HLDA: now also U1.6 (D5), R48.2; no longer U5.7 (D6), U6.47 (GPIO38)
- net HLTA: now also J4.59, U2.5 (D4), R53.2; no longer J4.6, U4.6 (D5), U6.39 (GPIO31)
- net HLTA_LED: now also U2.16 (*Y4); no longer U4.13 (*Y7)
- net INP: now also J4.64, U2.8 (D7), R50.2; no longer J4.70, U4.3 (D2), U6.43 (GPIO34)
- net INP_LED: now also U2.13 (*Y7); no longer U4.16 (*Y4)
- net INT: now also J4.56, U2.2 (D1), R56.2; no longer J4.75, U4.9 (D8), U6.36 (GPIO28)
- net INTE: now also J4.71, U1.9 (D8), R45.2; no longer J4.11, U5.8 (D7), U6.46 (GPIO37)
- net INTE_LED: now also U1.13 (*Y7); no longer U4.19 (*Y1)
- net INT_LED: now also U2.19 (*Y1); no longer U5.14 (*Y6)
- net M1: now also J4.63, U2.7 (D6), R51.2; no longer J4.9, U4.4 (D3), U6.42 (GPIO33)
- net MEMR: now also J4.65, U2.9 (D8), R49.2; no longer J4.10, U4.2 (D1), U6.44 (GPIO35)
- net MEMR_LED: now also U2.12 (*Y8); no longer U4.17 (*Y3)
- net MI_LED: now also U2.14 (*Y6); no longer U4.15 (*Y5)
- net OUT: now also J4.62, U2.6 (D5), R52.2; no longer J4.71, U4.5 (D4), U6.40 (GPIO32)
- net OUT_LED: now also U2.15 (*Y5); no longer U4.14 (*Y6)
- net PROT: now also J4.70, U1.8 (D7), R46.2; no longer J4.69, U5.9 (D8), U6.45 (GPIO36)
- net PROTECT: now also U9.24 (GPA3); no longer U9.23 (GPA2)
- net PROT_LED: now also U1.12 (*Y8); no longer U4.18 (*Y2)
- net RESET: now also U9.26 (GPA5); no longer U9.21 (GPA0)
- net RUN: now also U8.27 (GPA6); no longer U9.2 (GPB1)
- net SINGLE: now also U8.26 (GPA5); no longer U9.3 (GPB2)
- net STACK: now also J4.58, U2.4 (D3), R54.2; no longer J4.74, U4.7 (D6), U6.38 (GPIO30)
- net STACK_LED: now also U2.17 (*Y3); no longer U4.12 (*Y8)
- net STEP: now also U8.25 (GPA4); no longer U9.4 (GPB3)
- net STOP: now also U8.28 (GPA7); no longer U9.1 (GPB0)
- net UNPROTECT: now also U9.23 (GPA2); no longer U9.24 (GPA3)
- net WAIT: now also J4.69, U1.7 (D6), R47.2; no longer J4.12, U5.6 (D5), U6.48 (GPIO39)
- net WAIT_LED: now also U1.14 (*Y6); no longer U5.13 (*Y7)
- net WO: now also J4.57, U2.3 (D2), R55.2; no longer J4.5, U4.8 (D7), U6.37 (GPIO29)
- net WO_LED: now also U2.18 (*Y2); no longer U5.15 (*Y5)
- net BUS20 renamed I2C1_SCK
- net I2C1_SCK: now also J4.74; no longer J4.51
- net BUS21 renamed I2C1_SDA
- net I2C1_SDA: now also J4.75; no longer J4.29
- net BUS22 renamed I2C0_SCK
- net I2C0_SCK: now also J4.76; no longer J4.50
- net BUS23 renamed I2C0_SDA
- net I2C0_SDA: now also J4.77; no longer J4.30
- net DATA00: no longer names the net of U6.49 (GPIO40_ADC0)
- net DATA00: now also R81.1; no longer J4.47
- net DATA01: no longer names the net of U6.52 (GPIO41_ADC1)
- net DATA01: now also R82.1; no longer J4.33
- net DATA02: no longer names the net of U6.53 (GPIO42_ADC2)
- net DATA02: now also R83.1; no longer J4.46
- net DATA03: no longer names the net of U6.54 (GPIO43_ADC3)
- net DATA03: now also R84.1; no longer J4.34
- net DATA04: no longer names the net of U6.55 (GPIO44_ADC4)
- net DATA04: now also R85.1; no longer J4.45
- net DATA05: no longer names the net of U6.56 (GPIO45_ADC5)
- net DATA05: now also R86.1; no longer J4.35
- net DATA06: no longer names the net of U6.57 (GPIO46_ADC6)
- net DATA06: now also R87.1; no longer J4.44
- net DATA07: no longer names the net of U6.58 (GPIO47_ADC7)
- net DATA07: now also R88.1; no longer J4.36
- new net: R76.1, U6.44 (GPIO35)
- new net: R69.1, U6.36 (GPIO28)
- new net: R63.1, U6.22 (GPIO22)
- new net: R47.1, U6.3 (GPIO6)
- new net: R52.1, U6.9 (GPIO11)
- new net: R53.1, U6.11 (GPIO12)
- new net: R62.1, U6.21 (GPIO21)
- new net: R55.1, U6.13 (GPIO14)
- new net: R59.1, U6.18 (GPIO18)
- new net: R71.1, U6.38 (GPIO30)
- new net: R67.1, U6.27 (GPIO26)
- new net: R70.1, U6.37 (GPIO29)
- new net: R74.1, U6.42 (GPIO33)
- new net: R80.1, U6.48 (GPIO39)
- new net: R66.1, U6.26 (GPIO25)
- new net: R77.1, U6.45 (GPIO36)
- new net: R57.1, U6.16 (GPIO16)
- new net: R79.1, U6.47 (GPIO38)
- new net: R50.1, U6.7 (GPIO9)
- new net: R48.1, U6.4 (GPIO7)
- new net: R75.1, U6.43 (GPIO34)
- new net: R78.1, U6.46 (GPIO37)
- new net: R54.1, U6.12 (GPIO13)
- new net: R45.1, U6.1 (GPIO4)
- new net: R56.1, U6.14 (GPIO15)
- new net: R58.1, U6.17 (GPIO17)
- new net: R60.1, U6.19 (GPIO19)
- new net: R46.1, U6.2 (GPIO5)
- new net: R61.1, U6.20 (GPIO20)
- new net: R64.1, U6.23 (GPIO23)
- new net: R65.1, U6.25 (GPIO24)
- new net: R68.1, U6.28 (GPIO27)
- new net: R72.1, U6.39 (GPIO31)
- new net: R73.1, U6.40 (GPIO32)
- new net: R49.1, U6.6 (GPIO8)
- new net: R51.1, U6.8 (GPIO10)
- new net BUS03: J4.3
- new net BUS04: J4.4, R88.2
- new net BUS05: J4.5, R87.2
- new net BUS06: J4.6, R86.2
- new net BUS09: J4.9, R85.2
- new net BUS10: J4.10, R84.2
- new net BUS11: J4.11, R83.2
- new net BUS12: J4.12, R82.2
- new net BUS15: J4.15, R81.2

Commit message: various changes
Parts:
- added H1, H2, H3, H4: MountingHole, MountingHole:MountingHole_3.5mm, symbol Mechanical:MountingHole
Other:
- note added: "Pin 53 & 54, and 68 & 69, shared"

Commit message: more panel layout changes
Parts:
- C7, C8: footprint Capacitor_SMD:C_0402_1005Metric -> Capacitor_SMD:C_0603_1608Metric
Connections:
- net 3.3V: no longer C8.2, U6.62 (VREG_PGND)
- net GND: now also C8.2, U6.62 (VREG_PGND)
Other:
- moved on the sheet: C7
Changed lines of the file:
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@@
 	)
 	(junction
-		(at 100.33 91.44)
-		(diameter 0)
-		(color 0 0 0 0)
-	)
-	(junction
 		(at 215.9 43.18)
 		(diameter 0)
@@
 	)
 	(junction
+		(at 100.33 91.44)
+		(diameter 0)
+		(color 0 0 0 0)
+	)
+	(junction
 		(at 111.76 91.44)
 		(diameter 0)
@@
 	(wire
 		(pts
-			(xy 100.33 91.44) (xy 100.33 72.39)
+			(xy 100.33 91.44) (xy 100.33 88.9)
 		)
 		(stroke
@@
 	(wire
 		(pts
+			(xy 100.33 91.44) (xy 100.33 93.98)
+		)
+		(stroke
+			(width 0)
+			(type default)
+		)
+	)
+	(wire
+		(pts
 			(xy 427.99 100.33) (xy 417.83 100.33)
 		)
@@
 	(wire
 		(pts
+			(xy 100.33 81.28) (xy 100.33 72.39)
+		)
+		(stroke
+			(width 0)
+			(type default)
+		)
+	)
+	(wire
+		(pts
 			(xy 118.11 184.15) (xy 130.81 184.15)
 		)
@@
 	)
 	(rectangle
-		(start 82.55 52.07)
-		(end 129.54 95.25)
+		(start 82.55 57.15)
+		(end 129.54 100.33)
 		(stroke
 			(width 0)
@@
 	(symbol
 		(lib_id "power:GND")
-		(at 92.71 91.44 270)
+		(at 100.33 93.98 0)
 		(unit 1)
 		(exclude_from_sim no)
@@
 		(fields_autoplaced yes)
 		(property "Reference" "#PWR063"
-			(at 86.36 91.44 0)
+			(at 100.33 100.33 0)
 			(effects
 				(font
@@
 		)
 		(property "Value" "GND"
-			(at 88.9 91.4399 90)
+			(at 100.33 99.06 0)
 			(effects
 				(font
 					(size 1.27 1.27)
 				)
-				(justify right)
 			)
 		)
 		(property "Footprint" ""
-			(at 92.71 91.44 0)
+			(at 100.33 93.98 0)
 			(effects
 				(font
@@
 		)
 		(property "Datasheet" ""
-			(at 92.71 91.44 0)
+			(at 100.33 93.98 0)
 			(effects
 				(font
@@
 		)
 		(property "Description" "Power symbol creates a global label with name \"GND\" , ground"
-			(at 92.71 91.44 0)
+			(at 100.33 93.98 0)
 			(effects
 				(font
@@
 	(symbol
 		(lib_id "Device:C")
-		(at 96.52 91.44 270)
+		(at 100.33 85.09 0)
 		(unit 1)
 		(exclude_from_sim no)
@@
 		(fields_autoplaced yes)
 		(property "Reference" "C7"
-			(at 96.52 83.82 90)
+			(at 104.14 83.8199 0)
 			(effects
 				(font
 					(size 1.27 1.27)
 				)
+				(justify left)
 			)
 		)
 		(property "Value" "4.7u"
-			(at 96.52 86.36 90)
+			(at 104.14 86.3599 0)
 			(effects
 				(font
 					(size 1.27 1.27)
 				)
+				(justify left)
 			)
 		)
-		(property "Footprint" "Capacitor_SMD:C_0402_1005Metric"
-			(at 92.71 92.4052 0)
+		(property "Footprint" "Capacitor_SMD:C_0603_1608Metric"
+			(at 101.2952 88.9 0)
 			(effects
 				(font
@@
 		)
 		(property "Datasheet" "~"
-			(at 96.52 91.44 0)
+			(at 100.33 85.09 0)
 			(effects
 				(font
@@
 		)
 		(property "Description" "Unpolarized capacitor"
-			(at 96.52 91.44 0)
+			(at 100.33 85.09 0)
 			(effects
 				(font
@@
 			)
 		)
-		(property "Footprint" "Capacitor_SMD:C_0402_1005Metric"
+		(property "Footprint" "Capacitor_SMD:C_0603_1608Metric"
 			(at 112.7252 88.9 0)
 			(effects
