File: ecad/panel/panel.kicad_sch (KiCad schematic)
At the start: 209 parts, among them J2 Conn_01x03_Pin, J3 USB4235-03-C, J4 5017868090, SW1 SW_SPDT, SW10 SW_SPDT, SW11 SW_SPDT, SW12 SW_SPDT, SW13 SW_SPDT, SW14 SW_SPDT, SW15 SW_SPDT, SW16 SW_SPDT, SW17 SW_Push, SW18 SW_Push, SW19 SW_Push, SW2 SW_SPDT, SW20 SW_Push, SW21 SW_Push, SW22 SW_Push, SW23 SW_Push, SW24 SW_Push, SW25 SW_Push, SW26 SW_Push, SW27 SW_Push, SW28 SW_Push, SW29 SW_Push, SW3 SW_SPDT, SW30 SW_Push, SW31 SW_Push, SW4 SW_SPDT, SW5 SW_SPDT, SW6 SW_SPDT, SW7 SW_SPDT, SW8 SW_SPDT, SW9 SW_SPDT, U1 TLC59211IN, U10 NCP1117-3.3_SOT223, U2 TLC59211IN, U3 TLC59211IN, U4 TLC59211IN, U5 TLC59211IN, U6 RP2350_80QFN, U7 W25Q128JVS, U8 MCP23017_SO, U9 MCP23017_SO, X1 ABM8-272-T3

Commit message: BOM change
Parts:
- C1, C2, C26, C27, C3: JLCPCB Part # (none) -> C1570
- C10, C12, C13, C14, C15, C16, C17, C18, C19, C20, C21, C22, C24, C25, C6: JLCPCB Part # (none) -> C1525
- C11, C7, C8, C9: JLCPCB Part # (none) -> C23733
- C23, C28, C29: JLCPCB Part # (none) -> C15525
- C4, C5: JLCPCB Part # (none) -> C1548
- D37: JLCPCB Part # (none) -> C2290
- D38, D39, D41: JLCPCB Part # (none) -> C3757764
- H1, H2, H3, H4, J2, SW1, SW10, SW11, SW12, SW13, SW14, SW15, SW16, SW2, SW3, SW4, SW5, SW6, SW7, SW8, SW9: now not fitted
- J4: JLCPCB Part # (none) -> C6092927
- L1: JLCPCB Part # (none) -> C42411119
- R1, R10, R11, R12, R13, R14, R15, R16, R17, R18, R19, R2, R20, R21, R22, R23, R24, R3, R33, R34, R35, R36, R37, R38, R39, R4, R40, R41, R42, R43, R44, R5, R6, R7, R8, R9: JLCPCB Part # (none) -> C2909380
- R25: JLCPCB Part # (none) -> C25741
- R26, R27, R90: JLCPCB Part # (none) -> C11702
- R28: JLCPCB Part # (none) -> C25105
- R29, R30: JLCPCB Part # (none) -> C25905
- R31, R32: JLCPCB Part # (none) -> C138021
- R45, R46, R47, R48, R49, R50, R51, R52, R53, R54, R55, R56, R57, R58, R59, R60, R61, R62, R63, R64, R65, R66, R67, R68, R69, R70, R71, R72, R73, R74, R75, R76, R77, R78, R79, R80, R81, R82, R83, R84, R85, R86, R87, R88: JLCPCB Part # (none) -> C25104
- R89: JLCPCB Part # (none) -> C25082
- U1, U2, U3, U4, U5: JLCPCB Part # (none) -> C1554239
- U10: JLCPCB Part # (none) -> C26537
- U6: JLCPCB Part # (none) -> C42415655
- U7: JLCPCB Part # (none) -> C97521
- U8, U9: JLCPCB Part # (none) -> C639770
- X1: JLCPCB Part # (none) -> C20625731
