File: ecad/panel/panel.kicad_sch (KiCad schematic)
At the start: 222 parts, among them J2 Conn_01x03_Pin, J3 USB4235-03-C, J4 5017868090, SW1 SW_SPDT, SW10 SW_SPDT, SW11 SW_SPDT, SW12 SW_SPDT, SW13 SW_SPDT, SW14 SW_SPDT, SW15 SW_SPDT, SW16 SW_SPDT, SW17 SW_Push, SW18 SW_Push, SW19 SW_Push, SW2 SW_SPDT, SW20 SW_Push, SW21 SW_Push, SW22 SW_Push, SW23 SW_Push, SW24 SW_Push, SW25 SW_Push, SW26 SW_Push, SW27 SW_Push, SW28 SW_Push, SW29 SW_Push, SW3 SW_SPDT, SW30 TS-1187A-B-A-B, SW31 TS-1187A-B-A-B, SW4 SW_SPDT, SW5 SW_SPDT, SW6 SW_SPDT, SW7 SW_SPDT, SW8 SW_SPDT, SW9 SW_SPDT, U1 TLC59211IPWR, U10 AMS1117-3.3, U2 TLC59211IPWR, U3 TLC59211IPWR, U4 TLC59211IPWR, U5 TLC59211IPWR, U6 RP2350B, U7 W25Q128JVS, U8 MCP23017_SO, U9 MCP23017_SO, X1 ABM8-272-T3

Commit message: new panel routing
Parts:
- R100, R101, R102, R103, R91, R92, R93, R94, R95, R96, R97, R98, R99: footprint (none) -> Capacitor_SMD:C_0402_1005Metric
Connections:
- net 3.3V: now also R100.2, R101.2, R102.2, R103.2, R91.2, R92.2, R93.2, R94.2, R95.2, R96.2, R97.2, R98.2, R99.2; no longer SW17.1, SW18.1, SW19.1, SW20.1, SW21.1, SW22.1, SW23.1, SW24.1, SW25.1, SW26.1, SW27.1, SW28.1, SW29.1
- net GND: now also SW17.1, SW18.1, SW19.1, SW20.1, SW21.1, SW22.1, SW23.1, SW24.1, SW25.1, SW26.1, SW27.1, SW28.1, SW29.1; no longer R100.2, R101.2, R102.2, R103.2, R91.2, R92.2, R93.2, R94.2, R95.2, R96.2, R97.2, R98.2, R99.2

Commit message: stackup changes, prodction
Parts:
- J3, R31, R32: now not fitted
Changed lines of the file:
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@@
 		(in_bom yes)
 		(on_board yes)
-		(dnp no)
+		(dnp yes)
 		(property "Reference" "R31"
 			(at 205.74 70.358 90)
@@
 		(in_bom yes)
 		(on_board yes)
-		(dnp no)
+		(dnp yes)
 		(property "Reference" "R32"
 			(at 205.74 75.184 90)
@@
 		(in_bom yes)
 		(on_board yes)
-		(dnp no)
+		(dnp yes)
 		(fields_autoplaced yes)
 		(property "Reference" "J3"

Commit message: double up for HASL
Parts:
- R31, R32: footprint Capacitor_SMD:C_0603_1608Metric_Pad1.08x0.95mm_HandSolder -> Resistor_SMD:R_0603_1608Metric_Pad0.98x0.95mm_HandSolder
Changed lines of the file:
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@@
 			)
 		)
-		(property "Footprint" "Capacitor_SMD:C_0603_1608Metric_Pad1.08x0.95mm_HandSolder"
+		(property "Footprint" "Resistor_SMD:R_0603_1608Metric_Pad0.98x0.95mm_HandSolder"
 			(at 205.74 74.168 90)
 			(effects
@@
 			)
 		)
-		(property "Footprint" "Capacitor_SMD:C_0603_1608Metric_Pad1.08x0.95mm_HandSolder"
+		(property "Footprint" "Resistor_SMD:R_0603_1608Metric_Pad0.98x0.95mm_HandSolder"
 			(at 205.74 79.248 90)
 			(effects

Commit message: fixup panel io expansion pinout
Parts:
- U8, U9: value MCP23017_SO -> MCP23017_ML; footprint Library:QFN28_IO_Expander -> Package_DFN_QFN:QFN-28-1EP_6x6mm_P0.65mm_EP4.25x4.25mm; symbol Interface_Expansion:MCP23017_SO -> Interface_Expansion:MCP23017_ML
Connections:
- net 3.3V: now also U8.5 (VDD), U9.11 (A0), U9.5 (VDD); no longer U8.9 (VDD), U9.15 (A0), U9.9 (VDD)
- net A0_SW: now also U9.4 (GPB7); no longer U9.8 (GPB7)
- net A10_SW: now also U9.22 (GPA5); no longer U9.26 (GPA5)
- net A11_SW: now also U9.21 (GPA4); no longer U9.25 (GPA4)
- net A12_SW: now also U9.20 (GPA3); no longer U9.24 (GPA3)
- net A13_SW: now also U9.19 (GPA2); no longer U9.23 (GPA2)
- net A14_SW: now also U9.18 (GPA1); no longer U9.22 (GPA1)
- net A15_SW: now also U9.17 (GPA0); no longer U9.21 (GPA0)
- net A1_SW: now also U9.3 (GPB6); no longer U9.7 (GPB6)
- net A2_SW: now also U9.2 (GPB5); no longer U9.6 (GPB5)
- net A3_SW: now also U9.1 (GPB4); no longer U9.5 (GPB4)
- net A4_SW: now also U9.28 (GPB3); no longer U9.4 (GPB3)
- net A5_SW: now also U9.27 (GPB2); no longer U9.3 (GPB2)
- net A6_SW: now also U9.26 (GPB1); no longer U9.2 (GPB1)
- net A7_SW: now also U9.25 (GPB0); no longer U9.1 (GPB0)
- net A8_SW: now also U9.24 (GPA7); no longer U9.28 (GPA7)
- net A9_SW: now also U9.23 (GPA6); no longer U9.27 (GPA6)
- net AUX1: now also U8.24 (GPA7); no longer U8.3 (GPB2)
- net AUX2: now also U8.1 (GPB4); no longer U8.5 (GPB4)
- net CLR: now also U8.22 (GPA5); no longer U8.1 (GPB0)
- net DEPOSIT: now also U8.27 (GPB2); no longer U8.28 (GPA7)
- net DEPOSIT_NEXT: now also U8.21 (GPA4); no longer U8.26 (GPA5)
- net EXAMINE: now also U8.28 (GPB3); no longer U8.25 (GPA4)
- net EXAMINE_NEXT: now also U8.17 (GPA0); no longer U8.24 (GPA3)
- net GND: now also U8.11 (A0), U8.12 (A1), U8.13 (A2), U8.29 (EP), U8.6 (VSS), U9.12 (A1), U9.13 (A2), U9.29 (EP), U9.6 (VSS); no longer U8.10 (VSS), U8.15 (A0), U8.16 (A1), U8.17 (A2), U9.10 (VSS), U9.16 (A1), U9.17 (A2)
- net I2C1_SCK: now also U8.8 (SCK), U9.8 (SCK); no longer U8.12 (SCK), U9.12 (SCK)
- net I2C1_SDA: now also U8.9 (SDA), U9.9 (SDA); no longer U8.13 (SDA), U9.13 (SDA)
- net PROTECT: now also U8.25 (GPB0); no longer U8.4 (GPB3)
- net PUSH_INTA: now also U8.16 (INTA); no longer U8.20 (INTA)
- net PUSH_INTB: now also U8.15 (INTB); no longer U8.19 (INTB)
- net RESET: now also U8.26 (GPB1); no longer U8.27 (GPA6)
- net RUN: now also U8.18 (GPA1); no longer U8.21 (GPA0)
- net SINGLE_STEP: now also U8.20 (GPA3); no longer U8.23 (GPA2)
- net STOP: now also U8.19 (GPA2); no longer U8.22 (GPA1)
- net UNPROTECT: now also U8.23 (GPA6); no longer U8.2 (GPB1)
- net ~{RESET}: now also U8.14 (~{RESET}), U9.14 (~{RESET}); no longer U8.18 (~{RESET}), U9.18 (~{RESET})
- no-connect marks 114 -> 35

Commit message: production fixups
Parts:
- D37: LCSC Part # (none) -> C2286
- L1: LCSC Part # (none) -> C42411119
- U8, U9: LCSC Part # (none) -> C639770
Changed lines of the file:
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@@
 			)
 		)
+		(property "LCSC Part #" "C639770"
+			(at 176.53 360.68 0)
+			(effects
+				(font
+					(size 1.27 1.27)
+				)
+				(hide yes)
+			)
+		)
 		(pin "14"
 		)
@@
 			)
 		)
+		(property "LCSC Part #" "C2286"
+			(at 300.99 162.56 90)
+			(effects
+				(font
+					(size 1.27 1.27)
+				)
+				(hide yes)
+			)
+		)
 		(pin "1"
 		)
@@
 			)
 		)
+		(property "LCSC Part #" "C42411119"
+			(at 123.19 85.09 90)
+			(effects
+				(font
+					(size 1.27 1.27)
+				)
+				(hide yes)
+			)
+		)
 		(pin "1"
 		)
@@
 			(at 114.3 361.95 0)
 			(effects
+				(font
+					(size 1.27 1.27)
+				)
+				(hide yes)
+			)
+		)
+		(property "LCSC Part #" "C639770"
+			(at 114.3 361.95 0)
+			(effects

Commit message: additional production fixups
Parts:
- D1, D10, D11, D12, D13, D14, D15, D16, D17, D18, D19, D2, D20, D21, D22, D23, D24, D25, D26, D27, D28, D29, D3, D30, D31, D32, D33, D34, D35, D36, D4, D5, D6, D7, D8, D9, J2, U1, U2, U3, U4, U5: now not fitted
Changed lines of the file:
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@@
 		(in_bom yes)
 		(on_board yes)
-		(dnp no)
+		(dnp yes)
 		(fields_autoplaced yes)
 		(property "Reference" "D5"
@@
 		(in_bom yes)
 		(on_board yes)
-		(dnp no)
+		(dnp yes)
 		(fields_autoplaced yes)
 		(property "Reference" "J2"
@@
 		(in_bom yes)
 		(on_board yes)
-		(dnp no)
+		(dnp yes)
 		(fields_autoplaced yes)
 		(property "Reference" "D15"
@@
 		(in_bom yes)
 		(on_board yes)
-		(dnp no)
+		(dnp yes)
 		(fields_autoplaced yes)
 		(property "Reference" "D21"
@@
 		(in_bom yes)
 		(on_board yes)
-		(dnp no)
+		(dnp yes)
 		(fields_autoplaced yes)
 		(property "Reference" "U2"
@@
 		(in_bom yes)
 		(on_board yes)
-		(dnp no)
+		(dnp yes)
 		(fields_autoplaced yes)
 		(property "Reference" "D34"
@@
 		(in_bom yes)
 		(on_board yes)
-		(dnp no)
+		(dnp yes)
 		(fields_autoplaced yes)
 		(property "Reference" "D32"
@@
 		(in_bom yes)
 		(on_board yes)
-		(dnp no)
+		(dnp yes)
 		(fields_autoplaced yes)
 		(property "Reference" "D6"
@@
 		(in_bom yes)
 		(on_board yes)
-		(dnp no)
+		(dnp yes)
 		(fields_autoplaced yes)
 		(property "Reference" "D17"
@@
 		(in_bom yes)
 		(on_board yes)
-		(dnp no)
+		(dnp yes)
 		(fields_autoplaced yes)
 		(property "Reference" "D30"
@@
 		(in_bom yes)
 		(on_board yes)
-		(dnp no)
+		(dnp yes)
 		(fields_autoplaced yes)
 		(property "Reference" "U3"
@@
 		(in_bom yes)
 		(on_board yes)
-		(dnp no)
+		(dnp yes)
 		(fields_autoplaced yes)
 		(property "Reference" "D27"
@@
 		(in_bom yes)
 		(on_board yes)
-		(dnp no)
+		(dnp yes)
 		(fields_autoplaced yes)
 		(property "Reference" "D16"
@@
 		(in_bom yes)
 		(on_board yes)
-		(dnp no)
+		(dnp yes)
 		(fields_autoplaced yes)
 		(property "Reference" "D24"
@@
 		(in_bom yes)
 		(on_board yes)
-		(dnp no)
+		(dnp yes)
 		(fields_autoplaced yes)
 		(property "Reference" "U5"
@@
 		(in_bom yes)
 		(on_board yes)
-		(dnp no)
+		(dnp yes)
 		(fields_autoplaced yes)
 		(property "Reference" "U1"
@@
 		(in_bom yes)
 		(on_board yes)
-		(dnp no)
+		(dnp yes)
 		(fields_autoplaced yes)
 		(property "Reference" "D7"
@@
 		(in_bom yes)
 		(on_board yes)
-		(dnp no)
+		(dnp yes)
 		(fields_autoplaced yes)
 		(property "Reference" "D22"
@@
 		(in_bom yes)
 		(on_board yes)
-		(dnp no)
+		(dnp yes)
 		(fields_autoplaced yes)
 		(property "Reference" "D8"
@@
 		(in_bom yes)
 		(on_board yes)
-		(dnp no)
+		(dnp yes)
 		(fields_autoplaced yes)
 		(property "Reference" "D10"
@@
 		(in_bom yes)
 		(on_board yes)
-		(dnp no)
+		(dnp yes)
 		(fields_autoplaced yes)
 		(property "Reference" "D14"
@@
 		(in_bom yes)
 		(on_board yes)
-		(dnp no)
+		(dnp yes)
 		(fields_autoplaced yes)
 		(property "Reference" "D18"
@@
 		(in_bom yes)
 		(on_board yes)
-		(dnp no)
+		(dnp yes)
 		(fields_autoplaced yes)
 		(property "Reference" "D3"
@@
 		(in_bom yes)
 		(on_board yes)
-		(dnp no)
+		(dnp yes)
 		(fields_autoplaced yes)
 		(property "Reference" "D19"
@@
 		(in_bom yes)
 		(on_board yes)
-		(dnp no)
+		(dnp yes)
 		(fields_autoplaced yes)
 		(property "Reference" "D33"
@@
 		(in_bom yes)
 		(on_board yes)
-		(dnp no)
+		(dnp yes)
 		(fields_autoplaced yes)
 		(property "Reference" "D25"
@@
 		(in_bom yes)
 		(on_board yes)
-		(dnp no)
+		(dnp yes)
 		(fields_autoplaced yes)
 		(property "Reference" "D9"
@@
 		(in_bom yes)
 		(on_board yes)
-		(dnp no)
+		(dnp yes)
 		(fields_autoplaced yes)
 		(property "Reference" "D28"
@@
 		(in_bom yes)
 		(on_board yes)
-		(dnp no)
+		(dnp yes)
 		(fields_autoplaced yes)
 		(property "Reference" "D36"
@@
 		(in_bom yes)
 		(on_board yes)
-		(dnp no)
+		(dnp yes)
 		(fields_autoplaced yes)
 		(property "Reference" "D1"
@@
 		(in_bom yes)
 		(on_board yes)
-		(dnp no)
+		(dnp yes)
 		(fields_autoplaced yes)
 		(property "Reference" "D2"
@@
 		(in_bom yes)
 		(on_board yes)
-		(dnp no)
+		(dnp yes)
 		(fields_autoplaced yes)
 		(property "Reference" "D35"
@@
 		(in_bom yes)
 		(on_board yes)
-		(dnp no)
+		(dnp yes)
 		(fields_autoplaced yes)
 		(property "Reference" "D11"
@@
 		(in_bom yes)
 		(on_board yes)
-		(dnp no)
+		(dnp yes)
 		(fields_autoplaced yes)
 		(property "Reference" "D12"
@@
 		(in_bom yes)
 		(on_board yes)
-		(dnp no)
+		(dnp yes)
 		(fields_autoplaced yes)
 		(property "Reference" "D4"
@@
 		(in_bom yes)
 		(on_board yes)
-		(dnp no)
+		(dnp yes)
 		(fields_autoplaced yes)
 		(property "Reference" "D29"
@@
 		(in_bom yes)
 		(on_board yes)
-		(dnp no)
+		(dnp yes)
 		(fields_autoplaced yes)
 		(property "Reference" "D20"
@@
 		(in_bom yes)
 		(on_board yes)
-		(dnp no)
+		(dnp yes)
 		(fields_autoplaced yes)
 		(property "Reference" "D26"
@@
 		(in_bom yes)
 		(on_board yes)
-		(dnp no)
+		(dnp yes)
 		(fields_autoplaced yes)
 		(property "Reference" "D13"
@@
 		(in_bom yes)
 		(on_board yes)
-		(dnp no)
+		(dnp yes)
 		(fields_autoplaced yes)
 		(property "Reference" "U4"
@@
 		(in_bom yes)
 		(on_board yes)
-		(dnp no)
+		(dnp yes)
 		(fields_autoplaced yes)
 		(property "Reference" "D31"
@@
 		(in_bom yes)
 		(on_board yes)
-		(dnp no)
+		(dnp yes)
 		(fields_autoplaced yes)
 		(property "Reference" "D23"
