File: ecad/panel/panel.kicad_pcb (KiCad board)
At the start: 8 copper layers, 159 parts, among them J2 Conn_01x03_Pin, J3 USB4105-GF-A, SW1 SW_SPDT, SW10 SW_SPDT, SW11 SW_SPDT, SW12 SW_SPDT, SW13 SW_SPDT, SW14 SW_SPDT, SW15 SW_SPDT, SW16 SW_SPDT, SW17 SW_Push, SW18 SW_Push, SW19 SW_Push, SW2 SW_SPDT, SW20 SW_Push, SW21 SW_Push, SW22 SW_Push, SW23 SW_Push, SW24 SW_Push, SW25 SW_Push, SW26 SW_Push, SW27 SW_Push, SW28 SW_Push, SW29 SW_Push, SW3 SW_SPDT, SW30 SW_Push, SW31 SW_Push, SW4 SW_SPDT, SW5 SW_SPDT, SW6 SW_SPDT, SW7 SW_SPDT, SW8 SW_SPDT, SW9 SW_SPDT, U1 TLC59211IN, U2 TLC59211IN, U3 TLC59211IN, U4 TLC59211IN, U5 TLC59211IN, U6 RP2350_80QFN, U7 W25Q128JVS, U8 MCP23017_SO, U9 MCP23017_SO, X1 ABM8-272-T3

Commit message: PCB Changes
Parts:
- added J4: 5017868090, Library:CON_5017868090, F.Cu at (152.4, 118.6)

Commit message: Update PCB
Parts:
- removed JP1, JP3, JP5, JP7: Jumper_2_Bridged, Resistor_SMD:R_0402_1005Metric_Pad0.72x0.64mm_HandSolder
- removed JP2, JP4, JP6, JP8: Jumper_2_Open, Resistor_SMD:R_0402_1005Metric_Pad0.72x0.64mm_HandSolder
- C1, C10, C11, C12, C13, C14, C15, C16, C17, C18, C19, C2, C20, C21, C22, C23, C24, C25, C26, C27, C3, C4, C5, C6, C7, C8, C9, D1, D10, D11, D12, D13, D14, D15, D16, D17, D18, D19, D2, D20, D21, D22, D23, D24, D25, D26, D27, D28, D29, D3, D30, D31, D32, D33, D34, D35, D36, D4, D5, D6, D7, D8, D9, J2, J3, L1, R1, R10, R11, R12, R13, R14, R15, R16, R17, R18, R19, R2, R20, R21, R22, R23, R24, R25, R26, R27, R28, R29, R3, R30, R31, R32, R33, R34, R35, R36, R37, R38, R39, R4, R40, R41, R42, R43, R44, R5, R6, R7, R8, R9, U7, X1: moved to F.Cu
- U8, U9: footprint Package_SO:SOIC-28W_7.5x17.9mm_P1.27mm -> Library:QFN28_IO_Expander
- moved J4 372.0 mm to (285.1, 466.0), turned to 180 degrees
- moved D35 340.0 mm to (303.3, -75.1), turned to 0 degrees
- moved D34 332.1 mm to (303.3, -81.4), turned to 0 degrees
- moved D33 330.4 mm to (303.3, -87.7), turned to 0 degrees
- moved D36 329.2 mm to (303.3, -68.8), turned to 0 degrees
- moved D32 329.1 mm to (303.3, -94.0), turned to 0 degrees
- moved D31 328.1 mm to (303.3, -100.3), turned to 0 degrees
- moved D30 327.4 mm to (303.3, -106.6), turned to 0 degrees
- moved D28 327.2 mm to (303.3, -119.2), turned to 0 degrees
- moved D29 327.2 mm to (303.3, -112.9), turned to 0 degrees
- moved J2 325.9 mm to (311.7, -77.4), turned to 0 degrees
- moved D10 313.1 mm to (283.9, -119.2), turned to 0 degrees
- moved D16 312.0 mm to (283.9, -81.4), turned to 0 degrees
- moved D11 310.7 mm to (283.9, -112.9), turned to 0 degrees
- moved D13 310.5 mm to (283.9, -100.3), turned to 0 degrees
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Connections:
- J4 pad 10: A11 -> MEMR
- J4 pad 11: A13 -> INTE
- J4 pad 12: A15 -> WAIT
- J4 pad 15: /BUS01 -> A10
- J4 pad 16: MEMR -> A8
- J4 pad 17: /BUS05 -> D6
- J4 pad 18: OUT -> D4
- J4 pad 21: WAIT -> D2
- J4 pad 22: /BUS11 -> D0
- J4 pad 23: STACK -> A6
- J4 pad 24: M1 -> A4
- J4 pad 27: /BUS17 -> A2
- J4 pad 28: /BUS19 -> A0
- J4 pad 3: A1 -> A13
- J4 pad 33: D1 -> /DATA01
- J4 pad 34: D3 -> /DATA03
- J4 pad 35: D5 -> /DATA05
- J4 pad 36: D7 -> /DATA07
- J4 pad 4: A3 -> A15
- J4 pad 44: D6 -> /DATA06
- J4 pad 45: D4 -> /DATA04
- J4 pad 46: D2 -> /DATA02
- J4 pad 47: D0 -> /DATA00
- J4 pad 5: A5 -> WO
- J4 pad 52: /BUS18 -> A1
- J4 pad 53: PROT -> A3
- J4 pad 56: HLTA -> A5
- J4 pad 57: HLDA -> A7
- J4 pad 58: WO -> D1
- J4 pad 59: /BUS08 -> D3
- J4 pad 6: A7 -> HLTA
- J4 pad 62: INP -> D5
- J4 pad 63: /BUS04 -> D7
- J4 pad 64: INT -> A9
- J4 pad 65: INTE -> A11
- J4 pad 68: A14 -> HLDA
- J4 pad 69: A12 -> PROT
- J4 pad 70: A10 -> INP
- J4 pad 71: A8 -> OUT
- J4 pad 74: A6 -> STACK
- J4 pad 75: A4 -> INT
- J4 pad 76: A2 -> A14
- J4 pad 77: A0 -> A12
- J4 pad 9: A9 -> M1
- U2 pad 12: /A15_LED -> /D7_LED
- U2 pad 13: /A14_LED -> /D6_LED
- U2 pad 14: /A13_LED -> /D5_LED
- U2 pad 15: /A12_LED -> /D4_LED
- U2 pad 16: /A11_LED -> /D3_LED
- U2 pad 17: /A10_LED -> /D2_LED
- U2 pad 18: /A9_LED -> /D1_LED
- U2 pad 19: /A8_LED -> /D0_LED
- U2 pad 2: A15 -> D7
- U2 pad 3: A14 -> D6
- U2 pad 4: A13 -> D5
- U2 pad 5: A12 -> D4
- U2 pad 6: A11 -> D3
- U2 pad 7: A10 -> D2
- U2 pad 8: A9 -> D1
- U2 pad 9: A8 -> D0
- U3 pad 12: /D7_LED -> /A15_LED
- U3 pad 13: /D6_LED -> /A14_LED
- U3 pad 14: /D5_LED -> /A13_LED
- U3 pad 15: /D4_LED -> /A12_LED
- U3 pad 16: /D3_LED -> /A11_LED
- U3 pad 17: /D2_LED -> /A10_LED
- U3 pad 18: /D1_LED -> /A9_LED
- U3 pad 19: /D0_LED -> /A8_LED
- U3 pad 2: D7 -> A15
- U3 pad 3: D6 -> A14
- U3 pad 4: D5 -> A13
- U3 pad 5: D4 -> A12
- U3 pad 6: D3 -> A11
- U3 pad 7: D2 -> A10
- U3 pad 8: D1 -> A9
- U3 pad 9: D0 -> A8
- U4 pad 2: STACK -> MEMR
- U4 pad 3: HLTA -> INP
- U4 pad 4: OUT -> M1
- U4 pad 5: M1 -> OUT
- U4 pad 6: INP -> HLTA
- U4 pad 7: MEMR -> STACK
- U4 pad 8: PROT -> WO
- U5 pad 12: unconnected-(U5-*Y8-Pad12) -> /HDLA_LED
- U5 pad 13: unconnected-(U5-*Y7-Pad13) -> /WAIT_LED
- U5 pad 14: unconnected-(U5-*Y6-Pad14) -> /INT_LED
- U5 pad 15: unconnected-(U5-*Y5-Pad15) -> /WO_LED
- U5 pad 16: /HDLA_LED -> unconnected-(U5-*Y4-Pad16)
- U5 pad 17: /WAIT_LED -> unconnected-(U5-*Y3-Pad17)
- U5 pad 18: /INT_LED -> unconnected-(U5-*Y2-Pad18)
- U5 pad 19: /WO_LED -> unconnected-(U5-*Y1-Pad19)
- U5 pad 2: WAIT -> unconnected-(U5-D1-Pad2)
- U5 pad 3: INT -> unconnected-(U5-D2-Pad3)
- U5 pad 4: WO -> unconnected-(U5-D3-Pad4)
- U5 pad 5: HLDA -> unconnected-(U5-D4-Pad5)
- U5 pad 6: unconnected-(U5-D5-Pad6) -> WAIT
- U5 pad 7: unconnected-(U5-D6-Pad7) -> HLDA
- U5 pad 8: unconnected-(U5-D7-Pad8) -> INTE
- U5 pad 9: unconnected-(U5-D8-Pad9) -> PROT
- U6 pad 1: /BUS19 -> A0
- U6 pad 11: /BUS11 -> D0
- U6 pad 12: WO -> D1
- U6 pad 13: WAIT -> D2
- U6 pad 14: /BUS08 -> D3
- U6 pad 16: OUT -> D4
- U6 pad 17: INP -> D5
- U6 pad 18: /BUS05 -> D6
- U6 pad 19: /BUS04 -> D7
- U6 pad 2: /BUS18 -> A1
- U6 pad 20: MEMR -> A8
- U6 pad 21: INT -> A9
- U6 pad 22: /BUS01 -> A10
- U6 pad 23: INTE -> A11
- U6 pad 25: A0 -> A12
- U6 pad 26: A1 -> A13
- U6 pad 27: A2 -> A14
- U6 pad 28: A3 -> A15
- U6 pad 3: /BUS17 -> A2
- U6 pad 36: A4 -> INT
- U6 pad 37: A5 -> WO
- U6 pad 38: A6 -> STACK
- U6 pad 39: A7 -> HLTA
- U6 pad 4: PROT -> A3
- U6 pad 40: A8 -> OUT
- U6 pad 42: A9 -> M1
- U6 pad 43: A10 -> INP
- U6 pad 44: A11 -> MEMR
- U6 pad 45: A12 -> PROT
- U6 pad 46: A13 -> INTE
- U6 pad 47: A14 -> HLDA
- U6 pad 48: A15 -> WAIT
- U6 pad 49: D0 -> /DATA00
- U6 pad 52: D1 -> /DATA01
- U6 pad 53: D2 -> /DATA02
- U6 pad 54: D3 -> /DATA03
- U6 pad 55: D4 -> /DATA04
- U6 pad 56: D5 -> /DATA05
- U6 pad 57: D6 -> /DATA06
- U6 pad 58: D7 -> /DATA07
- U6 pad 6: M1 -> A4
- U6 pad 7: HLTA -> A5
- U6 pad 77: Net-(JP1-A) -> /BUS23
- U6 pad 78: Net-(JP3-A) -> /BUS22
- U6 pad 79: Net-(JP5-A) -> /BUS21
- U6 pad 8: STACK -> A6
- U6 pad 80: Net-(JP7-A) -> /BUS20
- U6 pad 9: HLDA -> A7
- U8 pad 12: /I2C0_SCK -> /BUS22
- U8 pad 13: /I2C0_SDA -> /BUS23
- U9 pad 12: /I2C1_SCK -> /BUS20
- U9 pad 13: /I2C1_SDA -> /BUS21
Routing:
- net Net-(U6-USB_DP): track 190.9 -> 0.00 mm
- net AUX2: track 187.0 -> 0.00 mm, vias 5 -> 0
- net /~{RESET}: track 167.4 -> 0.00 mm, vias 6 -> 0
- net AUX1: track 154.6 -> 0.00 mm
- net /HLTA_LED: track 152.4 -> 0.00 mm, vias 2 -> 0
- net 3.3V: track 148.9 -> 0.00 mm, vias 81 -> 0
- net GND: track 142.0 -> 0.00 mm, vias 47 -> 0
- net A0_SW: track 127.2 -> 0.00 mm, vias 4 -> 0
- net /I2C1_SDA: track 120.4 -> 0.00 mm, vias 2 -> 0
- net /MEMR_LED: track 114.0 -> 0.00 mm, vias 2 -> 0
- net /D1_LED: track 99.1 -> 0.00 mm, vias 2 -> 0
- net /INT_LED: track 97.7 -> 0.00 mm, vias 2 -> 0
- net CLR: track 94.6 -> 0.00 mm
- net PROTECT: track 93.1 -> 0.00 mm, vias 2 -> 0
- net /STACK_LED: track 92.7 -> 0.00 mm, vias 2 -> 0
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- added copper zone on B.Cu, net GND
- removed copper zone on In1.Cu, net 3.3V
- removed copper zone on In2.Cu, net GND
Other:
- board outline added: 386.8 x 304.8 mm
- copper layers 8 -> 4
- board text removed: "0"
- board text removed: "1"
- board text removed: "10"
- board text removed: "11"
- board text removed: "12"
- board text removed: "13"
- board text removed: "136 x 221 mm^2"
- board text removed: "14"
- board text removed: "15"
- board text removed: "2"
- board text removed: "3"
- board text removed: "4"
- board text removed: "5"
- board text removed: "6"
- board text removed: "7"
- board text removed: "8"
- board text removed: "9"
- board text removed: "A0"
- board text removed: "A1"
- board text removed: "A10"
- board text removed: "A11"
- board text removed: "A12"
- board text removed: "A13"
- board text removed: "A14"
- board text removed: "A15"
- board text removed: "A2"
- board text removed: "A3"
- board text removed: "A4"
- board text removed: "A5"
- board text removed: "A6"
- board text removed: "A7"
- board text removed: "A8"
- board text removed: "A9"
- board text removed: "ADDRESS"
- board text removed: "AUX"
- board text removed: "BOARD RESET"
- board text removed: "CLR"
- board text removed: "D0"
- board text removed: "D1"
- board text removed: "D2"
- board text removed: "D3"
- board text removed: "D4"
- board text removed: "D5"
- board text removed: "D6"
- board text removed: "D7"
- board text removed: "DATA"
- board text removed: "DEPOSIT"
- board text removed: "DEPOSIT NEXT"
- board text removed: "EXAMINE"
- board text removed: "EXAMINE NEXT"
- board text removed: "HLDA"
- board text removed: "HTLA"
- board text removed: "INP"
- board text removed: "INT"
- board text removed: "INTE"
- board text removed: "MEMR"
- board text removed: "MI"
- board text removed: "OUT"
- board text removed: "PROT"
- board text removed: "PROTECT"
- board text removed: "RESET"
- board text removed: "RUN"
- board text removed: "SINGLE"
- board text removed: "STACK"
- board text removed: "STATUS"
- board text removed: "STEP"
- board text removed: "STOP"
- board text removed: "UNPROTECT"
- board text removed: "WAIT"
- board text removed: "WO"

Commit message: change
Parts:
- added R45: 330, Resistor_SMD:R_0402_1005Metric_Pad0.72x0.64mm_HandSolder, B.Cu at (316.9, 210.6)
- added R46: 330, Resistor_SMD:R_0402_1005Metric_Pad0.72x0.64mm_HandSolder, B.Cu at (317.8, 210.6)
- added R47: 330, Resistor_SMD:R_0402_1005Metric_Pad0.72x0.64mm_HandSolder, B.Cu at (318.8, 210.6)
- added R48: 330, Resistor_SMD:R_0402_1005Metric_Pad0.72x0.64mm_HandSolder, B.Cu at (319.7, 210.7)
- added R49: 330, Resistor_SMD:R_0402_1005Metric_Pad0.72x0.64mm_HandSolder, B.Cu at (320.6, 210.6)
- added R50: 330, Resistor_SMD:R_0402_1005Metric_Pad0.72x0.64mm_HandSolder, B.Cu at (321.6, 210.6)
- added R51: 330, Resistor_SMD:R_0402_1005Metric_Pad0.72x0.64mm_HandSolder, B.Cu at (322.6, 210.6)
- added R52: 330, Resistor_SMD:R_0402_1005Metric_Pad0.72x0.64mm_HandSolder, B.Cu at (323.5, 210.6)
- added R53: 330, Resistor_SMD:R_0402_1005Metric_Pad0.72x0.64mm_HandSolder, B.Cu at (324.4, 210.6)
- added R54: 330, Resistor_SMD:R_0402_1005Metric_Pad0.72x0.64mm_HandSolder, B.Cu at (325.4, 210.6)
- added R55: 330, Resistor_SMD:R_0402_1005Metric_Pad0.72x0.64mm_HandSolder, B.Cu at (326.4, 210.6)
- added R56: 330, Resistor_SMD:R_0402_1005Metric_Pad0.72x0.64mm_HandSolder, B.Cu at (327.3, 210.6)
- added R57: 330, Resistor_SMD:R_0402_1005Metric_Pad0.72x0.64mm_HandSolder, B.Cu at (328.2, 210.7)
- added R58: 330, Resistor_SMD:R_0402_1005Metric_Pad0.72x0.64mm_HandSolder, B.Cu at (329.2, 210.6)
- added R59: 330, Resistor_SMD:R_0402_1005Metric_Pad0.72x0.64mm_HandSolder, B.Cu at (330.1, 210.6)
- added R60: 330, Resistor_SMD:R_0402_1005Metric_Pad0.72x0.64mm_HandSolder, B.Cu at (331.1, 210.6)
- added R61: 330, Resistor_SMD:R_0402_1005Metric_Pad0.72x0.64mm_HandSolder, B.Cu at (332.1, 210.6)
- added R62: 330, Resistor_SMD:R_0402_1005Metric_Pad0.72x0.64mm_HandSolder, B.Cu at (333.0, 210.6)
- added R63: 330, Resistor_SMD:R_0402_1005Metric_Pad0.72x0.64mm_HandSolder, B.Cu at (333.9, 210.7)
- added R64: 330, Resistor_SMD:R_0402_1005Metric_Pad0.72x0.64mm_HandSolder, B.Cu at (334.9, 210.7)
- added R65: 330, Resistor_SMD:R_0402_1005Metric_Pad0.72x0.64mm_HandSolder, B.Cu at (378.4, 220.0)
- added R66: 330, Resistor_SMD:R_0402_1005Metric_Pad0.72x0.64mm_HandSolder, B.Cu at (376.4, 220.0)
- added R67: 330, Resistor_SMD:R_0402_1005Metric_Pad0.72x0.64mm_HandSolder, B.Cu at (374.4, 220.0)
- added R68: 330, Resistor_SMD:R_0402_1005Metric_Pad0.72x0.64mm_HandSolder, B.Cu at (372.4, 220.0)
- added R69: 330, Resistor_SMD:R_0402_1005Metric_Pad0.72x0.64mm_HandSolder, B.Cu at (370.4, 220.0)
- added R70: 330, Resistor_SMD:R_0402_1005Metric_Pad0.72x0.64mm_HandSolder, B.Cu at (368.4, 220.0)
- added R71: 330, Resistor_SMD:R_0402_1005Metric_Pad0.72x0.64mm_HandSolder, B.Cu at (365.1, 219.9)
- added R72: 330, Resistor_SMD:R_0402_1005Metric_Pad0.72x0.64mm_HandSolder, F.Cu at (366.4, 216.7)
- added R73: 330, Resistor_SMD:R_0402_1005Metric_Pad0.72x0.64mm_HandSolder, F.Cu at (368.4, 216.7)
- added R74: 330, Resistor_SMD:R_0402_1005Metric_Pad0.72x0.64mm_HandSolder, F.Cu at (370.4, 216.7)
- added R75: 330, Resistor_SMD:R_0402_1005Metric_Pad0.72x0.64mm_HandSolder, F.Cu at (372.4, 216.7)
- added R76: 330, Resistor_SMD:R_0402_1005Metric_Pad0.72x0.64mm_HandSolder, F.Cu at (374.4, 216.7)
- added R77: 330, Resistor_SMD:R_0402_1005Metric_Pad0.72x0.64mm_HandSolder, F.Cu at (376.4, 216.7)
- added R78: 330, Resistor_SMD:R_0402_1005Metric_Pad0.72x0.64mm_HandSolder, F.Cu at (378.4, 216.7)
- added R79: 330, Resistor_SMD:R_0402_1005Metric_Pad0.72x0.64mm_HandSolder, F.Cu at (380.4, 216.7)
- added R80: 330, Resistor_SMD:R_0402_1005Metric_Pad0.72x0.64mm_HandSolder, F.Cu at (382.3, 216.7)
- added R81: 330, Resistor_SMD:R_0402_1005Metric_Pad0.72x0.64mm_HandSolder, F.Cu at (366.4, 213.5)
- added R82: 330, Resistor_SMD:R_0402_1005Metric_Pad0.72x0.64mm_HandSolder, F.Cu at (368.4, 213.5)
- added R83: 330, Resistor_SMD:R_0402_1005Metric_Pad0.72x0.64mm_HandSolder, F.Cu at (370.4, 213.5)
- added R84: 330, Resistor_SMD:R_0402_1005Metric_Pad0.72x0.64mm_HandSolder, F.Cu at (372.4, 213.5)
- added R85: 330, Resistor_SMD:R_0402_1005Metric_Pad0.72x0.64mm_HandSolder, F.Cu at (374.4, 213.5)
- added R86: 330, Resistor_SMD:R_0402_1005Metric_Pad0.72x0.64mm_HandSolder, F.Cu at (376.4, 213.5)
- added R87: 330, Resistor_SMD:R_0402_1005Metric_Pad0.72x0.64mm_HandSolder, F.Cu at (378.4, 213.5)
- added R88: 330, Resistor_SMD:R_0402_1005Metric_Pad0.72x0.64mm_HandSolder, F.Cu at (380.4, 213.5)
- D1, D10, D11, D12, D13, D14, D15, D16, D17, D18, D19, D2, D20, D21, D22, D23, D24, D25, D26, D27, D28, D29, D3, D30, D31, D32, D33, D34, D35, D36, D4, D5, D6, D7, D8, D9, J2, J3, J4, U7, X1: moved to B.Cu
- SW17, SW18, SW19, SW20, SW21, SW22, SW23, SW24, SW25, SW26, SW27, SW28, SW29, SW30: footprint Library:SW_1437565-5 -> Library:SW_1825910-6-4
- SW31: footprint Library:SW_1437565-5 -> Library:SW_1825910-6-4; moved to F.Cu
- moved D28 413.4 mm to (117.5, 250.1), turned to 180 degrees
- moved D29 404.0 mm to (126.0, 250.1), turned to 180 degrees
- moved D35 398.4 mm to (101.6, 268.4), turned to -90 degrees
- moved D30 394.7 mm to (134.5, 250.1), turned to 180 degrees
- moved D10 393.4 mm to (168.5, 256.9)
- moved D25 390.9 mm to (101.4, 259.0), turned to -90 degrees
- moved D36 390.2 mm to (107.0, 268.4), turned to -90 degrees
- moved D11 390.0 mm to (159.7, 256.8), turned to 180 degrees
- moved D12 387.1 mm to (151.0, 256.9)
- moved D31 385.4 mm to (143.0, 250.1)
- moved J2 385.2 mm to (198.2, 290.7)
- moved D13 384.6 mm to (141.0, 256.7)
- moved D26 382.8 mm to (106.9, 259.1), turned to -90 degrees
- moved D14 382.0 mm to (132.4, 256.6)
- moved D15 379.8 mm to (123.6, 256.6)
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- renumbered U3 to U2, U2 to U3
Connections:
- J4 pad 10: MEMR -> /BUS10
- J4 pad 11: INTE -> /BUS11
- J4 pad 12: WAIT -> /BUS12
- J4 pad 15: A10 -> /BUS15
- J4 pad 16: A8 -> A0
- J4 pad 17: D6 -> A1
- J4 pad 18: D4 -> A2
- J4 pad 21: D2 -> A3
- J4 pad 22: D0 -> A4
- J4 pad 23: A6 -> A5
- J4 pad 24: A4 -> A6
- J4 pad 27: A2 -> A7
- J4 pad 28: A0 -> D0
- J4 pad 29: /BUS21 -> D1
- J4 pad 3: A13 -> /BUS03
- J4 pad 30: /BUS23 -> D2
- J4 pad 33: /DATA01 -> D3
- J4 pad 34: /DATA03 -> D4
- J4 pad 35: /DATA05 -> D5
- J4 pad 36: /DATA07 -> D6
- J4 pad 4: A15 -> /BUS04
- J4 pad 44: /DATA06 -> A8
- J4 pad 45: /DATA04 -> A9
- J4 pad 46: /DATA02 -> A10
- J4 pad 47: /DATA00 -> A11
- J4 pad 5: WO -> /BUS05
- J4 pad 50: /BUS22 -> A12
- J4 pad 51: /BUS20 -> A13
- J4 pad 52: A1 -> A14
- J4 pad 53: A3 -> A15
- J4 pad 56: A5 -> INT
- J4 pad 57: A7 -> WO
- J4 pad 58: D1 -> STACK
- J4 pad 59: D3 -> HLTA
- J4 pad 6: HLTA -> /BUS06
- J4 pad 62: D5 -> OUT
- J4 pad 63: D7 -> M1
- J4 pad 64: A9 -> INP
- J4 pad 65: A11 -> MEMR
- J4 pad 69: PROT -> WAIT
- J4 pad 70: INP -> PROT
- J4 pad 71: OUT -> INTE
- J4 pad 74: STACK -> I2C1_SCK
- J4 pad 75: INT -> I2C1_SDA
- J4 pad 76: A14 -> I2C0_SCK
- J4 pad 77: A12 -> I2C0_SDA
- J4 pad 9: M1 -> /BUS09
- U1 pad 12: /A7_LED -> /PROT_LED
- U1 pad 13: /A6_LED -> /INTE_LED
- U1 pad 14: /A5_LED -> /WAIT_LED
- U1 pad 15: /A4_LED -> /HDLA_LED
- U1 pad 16: /A3_LED -> unconnected-(U1-*Y4-Pad16)
- U1 pad 17: /A2_LED -> unconnected-(U1-*Y3-Pad17)
- U1 pad 18: /A1_LED -> unconnected-(U1-*Y2-Pad18)
- U1 pad 19: /A0_LED -> unconnected-(U1-*Y1-Pad19)
- U1 pad 2: A7 -> unconnected-(U1-D1-Pad2)
- U1 pad 3: A6 -> unconnected-(U1-D2-Pad3)
- U1 pad 4: A5 -> unconnected-(U1-D3-Pad4)
- U1 pad 5: A4 -> unconnected-(U1-D4-Pad5)
- U1 pad 6: A3 -> HLDA
- U1 pad 7: A2 -> WAIT
- U1 pad 8: A1 -> PROT
- U1 pad 9: A0 -> INTE
- U2 pad 12: /A15_LED -> /MEMR_LED
- U2 pad 13: /A14_LED -> /INP_LED
- U2 pad 14: /A13_LED -> /MI_LED
- U2 pad 15: /A12_LED -> /OUT_LED
- U2 pad 16: /A11_LED -> /HLTA_LED
- U2 pad 17: /A10_LED -> /STACK_LED
- U2 pad 18: /A9_LED -> /WO_LED
- U2 pad 19: /A8_LED -> /INT_LED
- U2 pad 2: A15 -> INT
- U2 pad 3: A14 -> WO
- U2 pad 4: A13 -> STACK
- U2 pad 5: A12 -> HLTA
- U2 pad 6: A11 -> OUT
- U2 pad 7: A10 -> M1
- U2 pad 8: A9 -> INP
- U2 pad 9: A8 -> MEMR
- U3 pad 12: /D7_LED -> /A15_LED
- U3 pad 13: /D6_LED -> /A14_LED
- U3 pad 14: /D5_LED -> /A13_LED
- U3 pad 15: /D4_LED -> /A12_LED
- U3 pad 16: /D3_LED -> /A11_LED
- U3 pad 17: /D2_LED -> /A10_LED
- U3 pad 18: /D1_LED -> /A9_LED
- U3 pad 19: /D0_LED -> /A8_LED
- U3 pad 2: D7 -> A8
- U3 pad 3: D6 -> A9
- U3 pad 4: D5 -> A10
- U3 pad 5: D4 -> A11
- U3 pad 6: D3 -> A12
- U3 pad 7: D2 -> A13
- U3 pad 8: D1 -> A14
- U3 pad 9: D0 -> A15
- U4 pad 12: /STACK_LED -> /D7_LED
- U4 pad 13: /HLTA_LED -> /D6_LED
- U4 pad 14: /OUT_LED -> /D5_LED
- U4 pad 15: /MI_LED -> /D4_LED
- U4 pad 16: /INP_LED -> /D3_LED
- U4 pad 17: /MEMR_LED -> /D2_LED
- U4 pad 18: /PROT_LED -> /D1_LED
- U4 pad 19: /INTE_LED -> /D0_LED
- U4 pad 2: MEMR -> D0
- U4 pad 3: INP -> D1
- U4 pad 4: M1 -> D2
- U4 pad 5: OUT -> D3
- U4 pad 6: HLTA -> D4
- U4 pad 7: STACK -> D5
- U4 pad 8: WO -> D6
- U4 pad 9: INT -> D7
- U5 pad 12: /HDLA_LED -> /A7_LED
- U5 pad 13: /WAIT_LED -> /A6_LED
- U5 pad 14: /INT_LED -> /A5_LED
- U5 pad 15: /WO_LED -> /A4_LED
- U5 pad 16: unconnected-(U5-*Y4-Pad16) -> /A3_LED
- U5 pad 17: unconnected-(U5-*Y3-Pad17) -> /A2_LED
- U5 pad 18: unconnected-(U5-*Y2-Pad18) -> /A1_LED
- U5 pad 19: unconnected-(U5-*Y1-Pad19) -> /A0_LED
- U5 pad 2: unconnected-(U5-D1-Pad2) -> A0
- U5 pad 3: unconnected-(U5-D2-Pad3) -> A1
- U5 pad 4: unconnected-(U5-D3-Pad4) -> A2
- U5 pad 5: unconnected-(U5-D4-Pad5) -> A3
- U5 pad 6: WAIT -> A4
- U5 pad 7: HLDA -> A5
- U5 pad 8: INTE -> A6
- U5 pad 9: PROT -> A7
- U6 pad 1: A0 -> Net-(U6-GPIO4)
- U6 pad 11: D0 -> Net-(U6-GPIO12)
- U6 pad 12: D1 -> Net-(U6-GPIO13)
- U6 pad 13: D2 -> Net-(U6-GPIO14)
- U6 pad 14: D3 -> Net-(U6-GPIO15)
- U6 pad 16: D4 -> Net-(U6-GPIO16)
- U6 pad 17: D5 -> Net-(U6-GPIO17)
- U6 pad 18: D6 -> Net-(U6-GPIO18)
- U6 pad 19: D7 -> Net-(U6-GPIO19)
- U6 pad 2: A1 -> Net-(U6-GPIO5)
- U6 pad 20: A8 -> Net-(U6-GPIO20)
- U6 pad 21: A9 -> Net-(U6-GPIO21)
- U6 pad 22: A10 -> Net-(U6-GPIO22)
- U6 pad 23: A11 -> Net-(U6-GPIO23)
- U6 pad 25: A12 -> Net-(U6-GPIO24)
- U6 pad 26: A13 -> Net-(U6-GPIO25)
- U6 pad 27: A14 -> Net-(U6-GPIO26)
- U6 pad 28: A15 -> Net-(U6-GPIO27)
- U6 pad 3: A2 -> Net-(U6-GPIO6)
- U6 pad 36: INT -> Net-(U6-GPIO28)
- U6 pad 37: WO -> Net-(U6-GPIO29)
- U6 pad 38: STACK -> Net-(U6-GPIO30)
- U6 pad 39: HLTA -> Net-(U6-GPIO31)
- U6 pad 4: A3 -> Net-(U6-GPIO7)
- U6 pad 40: OUT -> Net-(U6-GPIO32)
- U6 pad 42: M1 -> Net-(U6-GPIO33)
- U6 pad 43: INP -> Net-(U6-GPIO34)
- U6 pad 44: MEMR -> Net-(U6-GPIO35)
- U6 pad 45: PROT -> Net-(U6-GPIO36)
- U6 pad 46: INTE -> Net-(U6-GPIO37)
- U6 pad 47: HLDA -> Net-(U6-GPIO38)
- U6 pad 48: WAIT -> Net-(U6-GPIO39)
- U6 pad 49: /DATA00 -> Net-(U6-GPIO40_ADC0)
- U6 pad 52: /DATA01 -> Net-(U6-GPIO41_ADC1)
- U6 pad 53: /DATA02 -> Net-(U6-GPIO42_ADC2)
- U6 pad 54: /DATA03 -> Net-(U6-GPIO43_ADC3)
- U6 pad 55: /DATA04 -> Net-(U6-GPIO44_ADC4)
- U6 pad 56: /DATA05 -> Net-(U6-GPIO45_ADC5)
- U6 pad 57: /DATA06 -> Net-(U6-GPIO46_ADC6)
- U6 pad 58: /DATA07 -> Net-(U6-GPIO47_ADC7)
- U6 pad 6: A4 -> Net-(U6-GPIO8)
- U6 pad 7: A5 -> Net-(U6-GPIO9)
- U6 pad 77: /BUS23 -> I2C0_SDA
- U6 pad 78: /BUS22 -> I2C0_SCK
- U6 pad 79: /BUS21 -> I2C1_SDA
- U6 pad 8: A6 -> Net-(U6-GPIO10)
- U6 pad 80: /BUS20 -> I2C1_SCK
- U6 pad 9: A7 -> Net-(U6-GPIO11)
- U8 pad 1: A0_SW -> A15_SW
- U8 pad 12: /BUS22 -> I2C0_SCK
- U8 pad 13: /BUS23 -> I2C0_SDA
- U8 pad 2: A1_SW -> A14_SW
- U8 pad 21: A8_SW -> DEPOSIT
- U8 pad 22: A9_SW -> DEPOSIT_NEXT
- U8 pad 23: A10_SW -> EXAMINE
- U8 pad 24: A11_SW -> EXAMINE_NEXT
- U8 pad 25: A12_SW -> STEP
- U8 pad 26: A13_SW -> SINGLE
- U8 pad 27: A14_SW -> RUN
- U8 pad 28: A15_SW -> STOP
- U8 pad 3: A2_SW -> A13_SW
- U8 pad 4: A3_SW -> A12_SW
- U8 pad 5: A4_SW -> A11_SW
- U8 pad 6: A5_SW -> A10_SW
- U8 pad 7: A6_SW -> A9_SW
- U8 pad 8: A7_SW -> A8_SW
- U9 pad 1: STOP -> A7_SW
- U9 pad 12: /BUS20 -> I2C1_SCK
- U9 pad 13: /BUS21 -> I2C1_SDA
- U9 pad 2: RUN -> A6_SW
- U9 pad 21: RESET -> AUX2
- U9 pad 22: CLR -> AUX1
- U9 pad 23: PROTECT -> UNPROTECT
- U9 pad 24: UNPROTECT -> PROTECT
- U9 pad 25: AUX1 -> CLR
- U9 pad 26: AUX2 -> RESET
- U9 pad 3: SINGLE -> A5_SW
- U9 pad 4: STEP -> A4_SW
- U9 pad 5: EXAMINE -> A3_SW
- U9 pad 6: EXAMINE_NEXT -> A2_SW
- U9 pad 7: DEPOSIT -> A1_SW
- U9 pad 8: DEPOSIT_NEXT -> A0_SW
Routing:
- net WAIT: track 34.4 -> 0.00 mm
- net HLDA: track 33.4 -> 0.00 mm
- net INTE: track 32.5 -> 0.00 mm
- net PROT: track 31.5 -> 0.00 mm
- net MEMR: track 28.2 -> 0.00 mm
- net INP: track 27.2 -> 0.00 mm
- net M1: track 26.3 -> 0.00 mm
- net A0: track 26.1 -> 0.00 mm
- net A1: track 25.6 -> 0.00 mm
- net A2: track 25.2 -> 0.00 mm
- net A3: track 24.8 -> 0.00 mm
- net A4: track 24.2 -> 0.00 mm
- net A5: track 23.7 -> 0.00 mm
- net A6: track 23.3 -> 0.00 mm
- net OUT: track 22.9 -> 0.00 mm
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- added copper zone on B.Cu, net (none)
- removed copper zone on B.Cu, net GND
Other:
- board text added: "BOX 1 SIZE"

Commit message: various changes
Parts:
- added H1: MountingHole, MountingHole:MountingHole_3.5mm, F.Cu at (40.7, 27.9)
- added H2: MountingHole, MountingHole:MountingHole_3.5mm, F.Cu at (196.2, 27.9)
- added H3: MountingHole, MountingHole:MountingHole_3.5mm, F.Cu at (40.7, 71.4)
- added H4: MountingHole, MountingHole:MountingHole_3.5mm, F.Cu at (196.2, 71.4)
- C1, C10, C11, C12, C13, C14, C15, C16, C17, C18, C19, C2, C20, C21, C22, C23, C24, C25, C26, C27, C3, C4, C5, C6, C7, C8, C9, L1, R1, R10, R11, R12, R13, R14, R15, R16, R17, R18, R19, R2, R20, R21, R22, R23, R24, R25, R26, R27, R28, R29, R3, R30, R31, R32, R33, R34, R35, R36, R37, R38, R39, R4, R40, R41, R42, R43, R44, R5, R6, R7, R72, R73, R74, R75, R76, R77, R78, R79, R8, R80, R81, R82, R83, R84, R85, R86, R87, R88, R9, SW31: moved to B.Cu
- moved R80 311.4 mm to (94.1, 98.8)
- moved R79 307.7 mm to (96.1, 98.8)
- moved R88 307.7 mm to (96.1, 95.5)
- moved R78 304.1 mm to (98.1, 98.8)
- moved R87 304.1 mm to (98.1, 95.5)
- moved R77 300.4 mm to (100.1, 98.8)
- moved R86 300.4 mm to (100.1, 95.5)
- moved R45 296.7 mm to (44.5, 92.7)
- moved R46 296.7 mm to (45.5, 92.7)
- moved R47 296.7 mm to (46.5, 92.7)
- moved R48 296.7 mm to (47.4, 92.7)
- moved R50 296.7 mm to (49.3, 92.7)
- moved R51 296.7 mm to (50.2, 92.7)
- moved R52 296.7 mm to (51.2, 92.7)
- moved R53 296.7 mm to (52.1, 92.7)
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Routing:
- net A12: track 0.00 -> 97.5 mm, vias 0 -> 1
- net A13: track 0.00 -> 97.1 mm, vias 0 -> 1
- net A14: track 0.00 -> 96.8 mm, vias 0 -> 1
- net A15: track 0.00 -> 96.5 mm, vias 0 -> 1
- net INT: track 0.00 -> 76.5 mm, vias 0 -> 1
- net WO: track 0.00 -> 76.1 mm, vias 0 -> 1
- net AUX2: track 0.00 -> 75.2 mm
- net GND: track 0.00 -> 71.5 mm, vias 0 -> 53
- net STACK: track 0.00 -> 71.2 mm, vias 0 -> 1
- net HLTA: track 0.00 -> 70.8 mm, vias 0 -> 1
- net OUT: track 0.00 -> 69.6 mm, vias 0 -> 1
- net M1: track 0.00 -> 69.2 mm, vias 0 -> 1
- net INP: track 0.00 -> 68.8 mm, vias 0 -> 1
- net MEMR: track 0.00 -> 68.2 mm, vias 0 -> 1
- net AUX1: track 0.00 -> 65.4 mm
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- added copper zone on B.Cu, net +1V1
- added copper zone on In2.Cu, net +1V1
- added copper zone on B.Cu, net 3.3V
- added copper zone on In1.Cu, net 3.3V
- added copper zone on B.Cu, net GND
- added copper zone on F.Cu, net GND
- added copper zone on In2.Cu, net GND
- added copper zone on B.Cu, net Net-(U6-VREG_LX)
Other:
- board size 386.8 x 304.8 mm -> 165.5 x 51.6 mm
- board text removed: "BOX 1 SIZE"

Commit message: more panel layout changes
Parts:
- C7, C8: footprint Capacitor_SMD:C_0402_1005Metric -> Capacitor_SMD:C_0603_1608Metric
- moved C1 141.4 mm to (57.9, 37.7), turned to 0 degrees
- moved R45 127.8 mm to (148.1, 17.8)
- moved R46 127.8 mm to (149.1, 17.8)
- moved R47 127.8 mm to (150.0, 17.8)
- moved C2 127.2 mm to (73.9, 37.6), turned to 0 degrees
- moved R37 121.1 mm to (64.4, 27.6), turned to 180 degrees
- moved R49 116.3 mm to (155.0, 46.3)
- moved R52 114.7 mm to (156.1, 46.3)
- moved R48 114.4 mm to (154.2, 51.6)
- moved R50 114.0 mm to (154.6, 48.9)
- moved R55 113.0 mm to (157.1, 46.3)
- moved R51 112.9 mm to (155.4, 51.6)
- moved C3 112.6 mm to (90.5, 38.5), turned to 90 degrees
- moved R53 112.6 mm to (155.8, 48.9)
- moved R58 111.4 mm to (158.2, 46.3)
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Connections:
- C10 pad 2: GND -> +1V1
- C11 pad 2: GND -> +1V1
- C8 pad 2: 3.3V -> GND
- U6 pad 15: GND -> 3.3V
- U6 pad 24: GND -> 3.3V
- U6 pad 29: GND -> 3.3V
- U6 pad 41: GND -> 3.3V
- U6 pad 5: GND -> 3.3V
- U6 pad 50: GND -> 3.3V
- U6 pad 62: 3.3V -> GND
- U6 pad 68: GND -> 3.3V
- U6 pad 69: GND -> 3.3V
- U6 pad 76: GND -> 3.3V
Routing:
- net GND: track 71.5 -> 40.7 mm, vias 53 -> 45
- net 3.3V: track 34.3 -> 62.8 mm, vias 35 -> 43
- net Net-(U6-GPIO11): track 1.91 -> 17.1 mm, vias 1 -> 4
- net Net-(U6-GPIO20): track 1.65 -> 15.4 mm, vias 0 -> 2
- net Net-(U6-GPIO14): track 4.09 -> 16.7 mm, vias 1 -> 4
- net Net-(U6-GPIO9): track 1.35 -> 13.2 mm, vias 1 -> 2
- net Net-(U6-GPIO21): track 2.28 -> 13.8 mm, vias 1 -> 0
- net Net-(U6-GPIO17): track 5.52 -> 16.8 mm, vias 1 -> 4
- net A9: track 27.5 -> 37.9 mm
- net Net-(U6-GPIO8): track 5.25 -> 15.4 mm, vias 0 -> 2
- net Net-(U6-GPIO23): track 2.74 -> 12.2 mm, vias 1 -> 0
- net Net-(U6-GPIO15): track 3.97 -> 13.4 mm, vias 1 -> 2
- net Net-(U6-GPIO18): track 2.95 -> 11.9 mm
- net Net-(U6-GPIO22): track 2.51 -> 11.2 mm, vias 1 -> 0
- net Net-(U6-GPIO12): track 3.53 -> 11.4 mm
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- added copper zone on In1.Cu, net +1V1
- removed copper zone on In2.Cu, net +1V1
Other:
- outline, holes or cut-outs redrawn
