File: ecad/panel/panel.kicad_pcb (KiCad board)
At the start: 4 copper layers, 165.5 x 51.6 mm, 222 parts, among them J2 Conn_01x03_Pin, J3 USB4235-03-C, J4 5017868090, SW1 SW_SPDT, SW10 SW_SPDT, SW11 SW_SPDT, SW12 SW_SPDT, SW13 SW_SPDT, SW14 SW_SPDT, SW15 SW_SPDT, SW16 SW_SPDT, SW17 SW_Push, SW18 SW_Push, SW19 SW_Push, SW2 SW_SPDT, SW20 SW_Push, SW21 SW_Push, SW22 SW_Push, SW23 SW_Push, SW24 SW_Push, SW25 SW_Push, SW26 SW_Push, SW27 SW_Push, SW28 SW_Push, SW29 SW_Push, SW3 SW_SPDT, SW30 TS-1187A-B-A-B, SW31 TS-1187A-B-A-B, SW4 SW_SPDT, SW5 SW_SPDT, SW6 SW_SPDT, SW7 SW_SPDT, SW8 SW_SPDT, SW9 SW_SPDT, U1 TLC59211IPWR, U10 AMS1117-3.3, U2 TLC59211IPWR, U3 TLC59211IPWR, U4 TLC59211IPWR, U5 TLC59211IPWR, U6 RP2350B, U7 W25Q128JVS, U8 MCP23017_ML, U9 MCP23017_ML, X1 ABM8-272-T3

Commit message: additional production fixups
Routing:
- removed copper zone on B.Cu, net (none)

Commit message: Files for JLCPCB
Other:
- board text added: "αCassiopeiae 8800 Computer Front Panel Board rev. 01 3/17/2025"
- board text removed: "αCassiopeiae 8800 Computer Front Panel Board rev. 01 3/14/2025"
Changed lines of the file:
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@@
 		)
 	)
-	(gr_text "αCassiopeiae 8800 Computer\nFront Panel Board\nrev. 01 3/14/2025"
+	(gr_text "αCassiopeiae 8800 Computer\nFront Panel Board\nrev. 01 3/17/2025"
 		(at 196 66.1 0)
 		(layer "B.SilkS")
