File: ecad/backplane/backplane.kicad_sch (KiCad schematic)
At the start: 21 parts, among them J1 10145891-0320J13LF, J2 10145891-0320J13LF, J3 USB4105-GF-A, J4 10145891-0320J13LF, J5 10145891-0320J13LF, J6 5017868090, U1 MCP16331x-xCH

Commit message: Back panel changes
Connections:
- net 3.3V: now also J6.1, J6.13, J6.19, J6.25, J6.31, J6.37, J6.43, J6.49, J6.55, J6.61, J6.67, J6.7, J6.73, J6.79
- net BUS29: now also J6.29
- net BUS30: now also J6.30
- net GND: now also J6.14, J6.2, J6.20, J6.26, J6.32, J6.38, J6.42, J6.48, J6.54, J6.60, J6.66, J6.72, J6.78, J6.8
- net A1: now reaches J6.10
- net D1: now reaches J6.11
- net D0: now reaches J6.12
- net PANEL: now reaches J6.15
- net MWRT: now reaches J6.16
- net DBIN: now reaches J6.17
- net CLOCK: now reaches J6.18
- net RESET: now reaches J6.21
- net PRDY: now reaches J6.22
- net XRDY: now reaches J6.23
- net INTA: now reaches J6.24
- net BUS27: now reaches J6.27
- net BUS28: now reaches J6.28
- net A3: now reaches J6.3
- net D7: now reaches J6.33
- net D6: now reaches J6.34
- net A6: now reaches J6.35
- net A7: now reaches J6.36
- net D3: now reaches J6.4
- net A2: now reaches J6.5
- net D2: now reaches J6.6
- net A0: now reaches J6.9
- net D5: now reaches J6.44
- net A5: now reaches J6.45
- net D4: now reaches J6.46
- net A4: now reaches J6.47
- net PROT: now reaches J6.50
- net INTE: now reaches J6.51
- net WAIT: now reaches J6.52
- net HLDA: now reaches J6.53
- net A12: now reaches J6.56
- net A13: now reaches J6.57
- net OUT: now reaches J6.58
- net M1: now reaches J6.59
- net A14: now reaches J6.62
- net MEMR: now reaches J6.63
- net INP: now reaches J6.64
- net A15: now reaches J6.65
- net HLTA: now reaches J6.68
- net STACK: now reaches J6.69
- net A11: now reaches J6.70
- net WO: now reaches J6.71
- net A10: now reaches J6.74
- net INT: now reaches J6.75
- net A9: now reaches J6.76
- net A8: now reaches J6.77
- no-connect marks 856 -> 866
Other:
- moved on the sheet: DB1, J2B, J2D, J5B, J6B
