File: ecad/backplane/backplane.kicad_sch (KiCad schematic)
At the start: 21 parts, among them J1 10145891-0320J13LF, J2 10145891-0320J13LF, J3 USB4105-GF-A, J4 10145891-0320J13LF, J5 10145891-0320J13LF, J6 5017868090, U1 MCP16331x-xCH

Commit message: Changes
Parts:
- added D2, D3: D_Schottky, symbol Device:D_Schottky
- added S2: 500SSP1S1M7QEA, Library:SW_500SSP1S1M7QEA, symbol Project_Library:500SSP1S1M7QEA
Connections:
- net ADDR00 is gone; now on net A0: J1.29
- net ADDR01 is gone; now on net A1: J1.30
- net ADDR02 is gone; now on net A2: J1.31
- net ADDR03 is gone; now on net A3: J1.32
- net ADDR04 is gone; now on net A4: J1.33
- net ADDR05 is gone; now on net A5: J1.34
- net ADDR06 is gone; now on net A6: J1.35
- net ADDR07 is gone; now on net A7: J1.36
- net ADDR09 is gone; now on net A9: J1.43
- net BUS05 is gone; now on net RESET: J2.5, J4.5, J5.5
- net BUS06 is gone; now on net PRDY: J2.6, J4.6, J5.6
- net BUS07 is gone; now on net XRDY: J2.7, J4.7, J5.7
- net BUS08 is gone; now on net INTA: J2.8, J4.8, J5.8
- net BUS09 is gone; now on net PANEL: J2.9, J4.9, J5.9
- net BUS10 is gone; now on net MWRT: J2.10, J4.10, J5.10
- net BUS11 is gone; now on net DBIN: J2.11, J4.11, J5.11
- net BUS17 is gone; now on net D0: J2.17, J4.17, J5.17
- net BUS18 is gone; now on net D1: J2.18, J4.18, J5.18
- net BUS19 is gone; now on net D2: J2.19, J4.19, J5.19
- net BUS20 is gone; now on net D3: J2.20, J4.20, J5.20
- net BUS21 is gone; now on net D4: J2.21, J4.21, J5.21
- net BUS22 is gone; now on net D5: J2.22, J4.22, J5.22
- net BUS23 is gone; now on net D6: J2.23, J4.23, J5.23
- net BUS24 is gone; now on net D7: J2.24, J4.24, J5.24
- net BUS27 is gone; now on net PANEL: J6.27
- net BUS28 is gone; now on net MWRT: J6.28
- net BUS31 is gone; now on net A2: J2.31, J4.31, J5.31
- net BUS32 is gone; now on net A3: J2.32, J4.32, J5.32
- net BUS33 is gone; now on net A4: J2.33, J4.33, J5.33
- net BUS34 is gone; now on net A5: J2.34, J4.34, J5.34
- net BUS35 is gone; now on net A6: J2.35, J4.35, J5.35
- net BUS36 is gone; now on net A7: J2.36, J4.36, J5.36
- net BUS41 is gone; now on net A8: J1.41, J2.41, J4.41, J5.41
- net BUS42 is gone; now on net PROT: J2.42, J4.42, J5.42
- net BUS43 is gone; now on net A9: J2.43, J4.43, J5.43
- net BUS44 is gone; now on net INTE: J2.44, J4.44, J5.44
- net BUS45 is gone; now on net A10: J1.45, J2.45, J4.45, J5.45
- net BUS46 is gone; now on net WAIT: J1.46, J2.46, J4.46, J5.46
- net BUS47 is gone; now on net A11: J1.47, J2.47, J4.47, J5.47
- net BUS48 is gone; now on net HLDA: J1.48, J2.48, J4.48, J5.48
- net BUS53 is gone; now on net A12: J1.53, J2.53, J4.53, J5.53
- net BUS54 is gone; now on net A13: J1.54, J2.54, J4.54, J5.54
- net BUS55 is gone; now on net A14: J1.55, J2.55, J4.55, J5.55
- net BUS56 is gone; now on net A15: J1.56, J2.56, J4.56, J5.56
- net BUS57 is gone; now on net OUT: J1.57, J2.57, J4.57, J5.57
- net BUS58 is gone; now on net M1: J1.58, J2.58, J4.58, J5.58
- net BUS59 is gone; now on net MEMR: J1.59, J2.59, J4.59, J5.59
- net BUS60 is gone; now on net INP: J1.60, J2.60, J4.60, J5.60
- net BUS65 is gone; now on net HLTA: J1.65, J2.65, J4.65, J5.65
- net BUS66 is gone; now on net STACK: J1.66, J2.66, J4.66, J5.66
- net BUS67 is gone; now on net WO: J1.67, J2.67, J4.67, J5.67
- net BUS68 is gone; now on net INT: J1.68, J2.68, J4.68, J5.68
- net CTRL01 is gone; now on net PANEL: J1.9
- net CTRL02 is gone; now on net PRDY: J1.6
- net CTRL03 is gone; now on net RESET: J1.5
- net CTRL04 is gone; now on net XRDY: J1.7
- net CTRL05 is gone; now on net INTA: J1.8
- net CTRL06 is gone; now on net MWRT: J1.10
- net CTRL07 is gone; now on net DBIN: J1.11
- net CTRL18 is gone; now on net INTE: J1.44
- net CTRL19 is gone; now on net PROT: J1.42
- net DATA00 is gone; now on net D0: J1.17
- net DATA01 is gone; now on net D1: J1.18
- net DATA02 is gone; now on net D2: J1.19
- net DATA03 is gone; now on net D3: J1.20
- net DATA04 is gone; now on net D4: J1.21
- net DATA05 is gone; now on net D5: J1.22
- net DATA06 is gone; now on net D6: J1.23
- net DATA07 is gone; now on net D7: J1.24
- net 3.3V: now also J1.40, J2.40, J4.40, J5.40, D3.2 (A), S2.1; no longer S1.1
- net 3.3V IN: now also S2.2
- net A0: now also J2.29, J4.29, J5.29
- net A1: now also J2.30, J4.30, J5.30
- net CLOCK: now also J1.276, J2.276, J4.276, J5.276; no longer J6.18
- net DBIN: now also J6.29; no longer J6.17
- net GND: no longer J1.40, J2.40, J4.40, J5.40
- net MWRT: no longer J6.16
- net PANEL: no longer J6.15
- net VBUS: now also D2.2 (A); no longer J3.A4_B9 (VBUS), J3.B4_A9 (VBUS__1)
- removed net BUS12: J2.12, J4.12, J5.12
- removed net BUS29: J2.29, J4.29, J5.29, J6.29
- removed net BUS30: J2.30, J4.30, J5.30, J6.30
- removed net BUS69: J1.69, J2.69, J4.69, J5.69
- removed net BUS70: J1.70, J2.70, J4.70, J5.70
- removed net BUS71: J1.71, J2.71, J4.71, J5.71
- removed net BUS72: J1.72, J2.72, J4.72, J5.72
- net CTRL00: no longer names the net of J1.12
- new net: D2.1 (K), J3.A4_B9 (VBUS), J3.B4_A9 (VBUS__1)
- new net: D3.1 (K), S1.1
- no-connect marks 866 -> 883
Other:
- note added: "DIMM SLOT 1"
- note added: "DIMM SLOT 2"
- note added: "DIMM SLOT 3"
- note added: "DIMM SLOT 4"
- note added: "FFC CONNECTOR"
- note added: "POWER SWITCH"
- note added: "RESET SWITCH"
- note removed: "DIMM slot 1"
- note removed: "DIMM slot 2"
- note removed: "DIMM slot 3"
- note removed: "DIMM slot 4"
- note removed: "Power on"
- moved on the sheet: C1, C2, CB1, Cln_1, Cln_2, D1, DB1, J1A, J1B, J1C, J1D, J6A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

Commit message: Backplane changes
Parts:
- removed D2, D3: D_Schottky, symbol Device:D_Schottky
- removed J5: 10145891-0320J13LF, Library:AMPHENOL_10145891-0320J13LF, symbol Project_Library:10145891-0320J13LF
- removed S2: 500SSP1S1M7QEA, Library:SW_500SSP1S1M7QEA, symbol Project_Library:500SSP1S1M7QEA
- added D2, D4: HEARTBEAT, LED_SMD:LED_0603_1608Metric_Pad1.05x0.95mm_HandSolder, symbol Device:LED
- added J4: 10145891-0320J13LF, Library:AMPHENOL_10145891-0320J13LF, symbol Project_Library:10145891-0320J13LF
- added R4, R5: 150, Resistor_SMD:R_0402_1005Metric, symbol Device:R_US
- renumbered J4 to J3, J3 to J5, RBot1 to RBot, RTop1 to RTop
Connections:
- net 3.3V: now also C1.1, C2.1, DB1.2 (A), J1.102, J1.103, J1.114, J1.115, J1.126, J1.127, J1.138, J1.139, J1.145, J1.146, J1.157, J1.158, J1.169, J1.170, J1.181, J1.182, J1.193, J1.194, J1.205, J1.206, J1.217, J1.218, J1.222, J1.223, J1.234, J1.235, J1.246, J1.247, J1.258, J1.259, J1.270, J1.271, J1.282, J1.283, J1.78, J1.79, J1.90, J1.91, J2.102, J2.103, J2.114, J2.115, J2.126, J2.127, J2.138, J2.139, J2.145, J2.146, J2.157, J2.158, J2.169, J2.170, J2.181, J2.182, J2.193, J2.194, J2.205, J2.206, J2.217, J2.218, J2.222, J2.223, J2.234, J2.235, J2.246, J2.247, J2.258, J2.259, J2.270, J2.271, J2.282, J2.283, J2.78, J2.79, J2.90, J2.91, J3.102, J3.103, J3.114, J3.115, J3.126, J3.127, J3.138, J3.139, J3.145, J3.146, J3.157, J3.158, J3.169, J3.170, J3.181, J3.182, J3.193, J3.194, J3.205, J3.206, J3.217, J3.218, J3.222, J3.223, J3.234, J3.235, J3.246, J3.247, J3.258, J3.259, J3.270, J3.271, J3.282, J3.283, J3.78, J3.79, J3.90, J3.91, L1.2, R3.2, D2.2 (A), J4.1, J4.102, J4.103, J4.114, J4.115, J4.126, J4.127, J4.13, J4.138, J4.139, J4.14, J4.145, J4.146, J4.157, J4.158, J4.169, J4.170, J4.181, J4.182, J4.193, J4.194, J4.2, J4.205, J4.206, J4.217, J4.218, J4.222, J4.223, J4.234, J4.235, J4.246, J4.247, J4.25, J4.258, J4.259, J4.26, J4.270, J4.271, J4.282, J4.283, J4.37, J4.38, J4.49, J4.50, J4.61, J4.62, J4.73, J4.74, J4.78, J4.79, J4.90, J4.91; no longer J1.40, J2.40, J3.40
- net A0: now also J4.29
- net A1: now also J4.30
- net A10: now also J4.45
- net A11: now also J4.47
- net A12: now also J4.53
- net A13: now also J4.54
- net A14: now also J4.55
- net A15: now also J4.56
- net A2: now also J4.31
- net A3: now also J4.32
- net A4: now also J4.33
- net A5: now also J4.34
- net A6: now also J4.35
- net A7: now also J4.36
- net A8: now also J4.41
- net A9: now also J4.43
- net CLOCK: now also J1.12, J2.12, J3.12, J6.30, J4.12; no longer J1.276, J2.276, J3.276
- net D0: now also J4.17
- net D1: now also J4.18
- net D2: now also J4.19
- net D3: now also J4.20
- net D4: now also J4.21
- net D5: now also J4.22
- net D6: now also J4.23
- net D7: now also J4.24
- net DBIN: now also J4.11
- net GND: now also J1.104, J1.105, J1.116, J1.117, J1.128, J1.129, J1.140, J1.141, J1.147, J1.148, J1.159, J1.160, J1.171, J1.172, J1.183, J1.184, J1.195, J1.196, J1.207, J1.208, J1.219, J1.220, J1.224, J1.225, J1.236, J1.237, J1.248, J1.249, J1.260, J1.261, J1.272, J1.273, J1.284, J1.285, J1.40, J1.80, J1.81, J1.92, J1.93, J2.104, J2.105, J2.116, J2.117, J2.128, J2.129, J2.140, J2.141, J2.147, J2.148, J2.159, J2.160, J2.171, J2.172, J2.183, J2.184, J2.195, J2.196, J2.207, J2.208, J2.219, J2.220, J2.224, J2.225, J2.236, J2.237, J2.248, J2.249, J2.260, J2.261, J2.272, J2.273, J2.284, J2.285, J2.40, J2.80, J2.81, J2.92, J2.93, J3.104, J3.105, J3.116, J3.117, J3.128, J3.129, J3.140, J3.141, J3.147, J3.148, J3.159, J3.160, J3.171, J3.172, J3.183, J3.184, J3.195, J3.196, J3.207, J3.208, J3.219, J3.220, J3.224, J3.225, J3.236, J3.237, J3.248, J3.249, J3.260, J3.261, J3.272, J3.273, J3.284, J3.285, J3.40, J3.80, J3.81, J3.92, J3.93, J4.104, J4.105, J4.116, J4.117, J4.128, J4.129, J4.140, J4.141, J4.147, J4.148, J4.15, J4.159, J4.16, J4.160, J4.171, J4.172, J4.183, J4.184, J4.195, J4.196, J4.207, J4.208, J4.219, J4.220, J4.224, J4.225, J4.236, J4.237, J4.248, J4.249, J4.260, J4.261, J4.27, J4.272, J4.273, J4.28, J4.284, J4.285, J4.3, J4.39, J4.4, J4.40, J4.51, J4.52, J4.63, J4.64, J4.75, J4.76, J4.80, J4.81, J4.92, J4.93, J4.SH1 (SHIELD), J4.SH2 (SHIELD__1), J4.SH3 (SHIELD__2), R4.2, R5.2
- net HLDA: now also J4.48
- net HLTA: now also J4.65
- net INP: now also J4.60
- net INT: now also J4.68
- net INTA: now also J4.8
- net INTE: now also J4.44
- net M1: now also J4.58
- net MEMR: now also J4.59
- net MWRT: now also J4.10
- net OUT: now also J4.57
- net PANEL: now also J4.9
- net PRDY: now also J4.6
- net PROT: now also J4.42
- net RESET: now also J4.5
- net STACK: now also J4.66
- net VBUS: now also J5.A4_B9 (VBUS), J5.B4_A9 (VBUS__1), S1.2, D4.2 (A); no longer Cln_1.1, Cln_2.1, U1.5 (V_{IN})
- net WAIT: now also J4.46
- net WO: now also J4.67
- net XRDY: now also J4.7
- net 5V: now reaches S1.1
- net 5V: now also Cln_1.1, Cln_2.1, U1.5 (V_{IN})
- net BEX100: now reaches J3.100
- net BEX100: now also J1.100, J2.100, J4.100
- net BEX101: now reaches J3.101
- net BEX101: now also J1.101, J2.101, J4.101
- net BEX106: now reaches J3.106
- net BEX106: now also J1.106, J2.106, J4.106
- net BEX107: now reaches J3.107
- net BEX107: now also J1.107, J2.107, J4.107
- net BEX108: now reaches J3.108
- net BEX108: now also J1.108, J2.108, J4.108
- net BEX109: now reaches J3.109
- net BEX109: now also J1.109, J2.109, J4.109
- net BEX110: now reaches J3.110
- net BEX110: now also J1.110, J2.110, J4.110
- net BEX111: now reaches J3.111
- net BEX111: now also J1.111, J2.111, J4.111
- net BEX112: now reaches J3.112
- net BEX112: now also J1.112, J2.112, J4.112
- net BEX113: now reaches J3.113
- net BEX113: now also J1.113, J2.113, J4.113
- net BEX118: now reaches J3.118
- net BEX118: now also J1.118, J2.118, J4.118
- net BEX119: now reaches J3.119
- net BEX119: now also J1.119, J2.119, J4.119
- net BEX120: now reaches J3.120
- net BEX120: now also J1.120, J2.120, J4.120
- net BEX121: now reaches J3.121
- net BEX121: now also J1.121, J2.121, J4.121
- net BEX122: now reaches J3.122
- net BEX122: now also J1.122, J2.122, J4.122
- net BEX123: now reaches J3.123
- net BEX123: now also J1.123, J2.123, J4.123
- net BEX124: now reaches J3.124
- net BEX124: now also J1.124, J2.124, J4.124
- net BEX125: now reaches J3.125
- net BEX125: now also J1.125, J2.125, J4.125
- net BEX082: now reaches J3.82
- net BEX082: now also J1.82, J2.82, J4.82
- net BEX083: now reaches J3.83
- net BEX083: now also J1.83, J2.83, J4.83
- net BEX084: now reaches J3.84
- net BEX084: now also J1.84, J2.84, J4.84
- net BEX085: now reaches J3.85
- net BEX085: now also J1.85, J2.85, J4.85
- net BEX086: now reaches J3.86
- net BEX086: now also J1.86, J2.86, J4.86
- net BEX087: now reaches J3.87
- net BEX087: now also J1.87, J2.87, J4.87
- net BEX088: now reaches J3.88
- net BEX088: now also J1.88, J2.88, J4.88
- net BEX089: now reaches J3.89
- net BEX089: now also J1.89, J2.89, J4.89
- net BEX094: now reaches J3.94
- net BEX094: now also J1.94, J2.94, J4.94
- net BEX095: now reaches J3.95
- net BEX095: now also J1.95, J2.95, J4.95
- net BEX096: now reaches J3.96
- net BEX096: now also J1.96, J2.96, J4.96
- net BEX097: now reaches J3.97
- net BEX097: now also J1.97, J2.97, J4.97
- net BEX098: now reaches J3.98
- net BEX098: now also J1.98, J2.98, J4.98
- net BEX099: now reaches J3.99
- net BEX099: now also J1.99, J2.99, J4.99
- removed net 3.3V IN: C1.1, C2.1, DB1.2 (A), L1.2, R3.2, S1.2
- new net: D4.1 (K), R4.1
- new net: D2.1 (K), R5.1
- no-connect marks 883 -> 450
Other:
- note added: "POWER FLAGS"
- note removed: "RESET SWITCH"
- note removed: "add protection diode"
- moved on the sheet: C1, C2, CB1, Cln_1, Cln_2, D1, DB1, J3B, J3C, J3D, J6A, J6B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

Commit message: Back Panel Done
Parts:
- Cln_1, Cln_2: footprint Capacitor_SMD:C_0402_1005Metric_Pad0.74x0.62mm_HandSolder -> Capacitor_SMD:C_0603_1608Metric_Pad1.08x0.95mm_HandSolder
- D1: footprint Diode_SMD:D_0402_1005Metric_Pad0.77x0.64mm_HandSolder -> Library:DO-214BA_MCH-L
- L1: footprint Inductor_SMD:L_0402_1005Metric_Pad0.77x0.64mm_HandSolder -> Library:DR73-150-R
- renumbered C1 to Cout_1, C2 to Cout_2, RBot to RBot1, RTop to RTop1
Other:
- moved on the sheet: D1
Changed lines of the file:
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@@
 	(wire
 		(pts
+			(xy 266.7 375.92) (xy 266.7 386.08)
+		)
+		(stroke
+			(width 0)
+			(type default)
+		)
+	)
+	(wire
+		(pts
 			(xy 312.42 73.66) (xy 328.93 73.66)
 		)
@@
 	(wire
 		(pts
-			(xy 266.7 375.92) (xy 266.7 382.27)
-		)
-		(stroke
-			(width 0)
-			(type default)
-		)
-	)
-	(wire
-		(pts
 			(xy 85.09 118.11) (xy 77.47 118.11)
 		)
@@
 			)
 		)
-		(property "Footprint" "Capacitor_SMD:C_0402_1005Metric_Pad0.74x0.62mm_HandSolder"
+		(property "Footprint" "Capacitor_SMD:C_0603_1608Metric_Pad1.08x0.95mm_HandSolder"
 			(at 202.8952 391.16 0)
 			(effects
@@
 		(on_board yes)
 		(dnp no)
-		(fields_autoplaced yes)
-		(property "Reference" "C2"
-			(at 311.15 373.3799 0)
+		(property "Reference" "Cout_2"
+			(at 310.388 372.618 0)
 			(effects
 				(font
@@
 		)
 		(property "Value" "10u"
-			(at 311.15 375.9199 0)
+			(at 310.388 375.158 0)
 			(effects
 				(font
@@
 			(project "backplane"
 				(path "/37626d4a-e2f8-4dc8-ba70-7956f3e14d24"
-					(reference "C2")
+					(reference "Cout_2")
 					(unit 1)
 				)
@@
 		(on_board yes)
 		(dnp no)
-		(fields_autoplaced yes)
-		(property "Reference" "C1"
-			(at 300.99 373.3799 0)
+		(property "Reference" "Cout_1"
+			(at 288.036 372.364 0)
 			(effects
 				(font
@@
 		)
 		(property "Value" "10u"
-			(at 300.99 375.9199 0)
+			(at 288.036 374.904 0)
 			(effects
 				(font
@@
 			(project ""
 				(path "/37626d4a-e2f8-4dc8-ba70-7956f3e14d24"
-					(reference "C1")
+					(reference "Cout_1")
 					(unit 1)
 				)
@@
 			)
 		)
-		(property "Footprint" "Inductor_SMD:L_0402_1005Metric_Pad0.77x0.64mm_HandSolder"
+		(property "Footprint" "Library:DR73-150-R"
 			(at 271.78 375.92 0)
 			(effects
@@
 		(dnp no)
 		(fields_autoplaced yes)
-		(property "Reference" "RBot"
+		(property "Reference" "RBot1"
 			(at 256.54 383.5399 0)
 			(effects
@@
 			(project ""
 				(path "/37626d4a-e2f8-4dc8-ba70-7956f3e14d24"
-					(reference "RBot")
+					(reference "RBot1")
 					(unit 1)
 				)
@@
 		(dnp no)
 		(property "Reference" "R3"
-			(at 269.748 378.46 90)
+			(at 271.78 378.206 90)
 			(effects
 				(font
@@
 		)
 		(property "Value" "10"
-			(at 274.066 378.46 90)
+			(at 271.78 383.794 90)
 			(effects
 				(font
@@
 	(symbol
 		(lib_id "power:GND")
-		(at 266.7 389.89 0)
+		(at 266.7 393.7 0)
 		(unit 1)
 		(exclude_from_sim no)
@@
 		(fields_autoplaced yes)
 		(property "Reference" "#PWR032"
-			(at 266.7 396.24 0)
+			(at 266.7 400.05 0)
 			(effects
 				(font
@@
 		)
 		(property "Value" "GND"
-			(at 266.7 394.97 0)
+			(at 266.7 398.78 0)
 			(effects
 				(font
@@
 		)
 		(property "Footprint" ""
-			(at 266.7 389.89 0)
+			(at 266.7 393.7 0)
 			(effects
 				(font
@@
 		)
 		(property "Datasheet" ""
-			(at 266.7 389.89 0)
+			(at 266.7 393.7 0)
 			(effects
 				(font
@@
 		)
 		(property "Description" "Power symbol creates a global label with name \"GND\" , ground"
-			(at 266.7 389.89 0)
+			(at 266.7 393.7 0)
 			(effects
 				(font
@@
 		(dnp no)
 		(fields_autoplaced yes)
-		(property "Reference" "RTop"
+		(property "Reference" "RTop1"
 			(at 260.35 374.65 90)
 			(effects
@@
 			(project ""
 				(path "/37626d4a-e2f8-4dc8-ba70-7956f3e14d24"
-					(reference "RTop")
+					(reference "RTop1")
 					(unit 1)
 				)
@@
 	(symbol
 		(lib_id "Device:D_Schottky")
-		(at 266.7 386.08 270)
+		(at 266.7 389.89 270)
 		(unit 1)
 		(exclude_from_sim no)
@@
 		(fields_autoplaced yes)
 		(property "Reference" "D1"
-			(at 269.24 384.4924 90)
+			(at 269.24 388.3024 90)
 			(effects
 				(font
@@
 		)
 		(property "Value" "D_Schottky"
-			(at 269.24 387.0324 90)
+			(at 269.24 390.8424 90)
 			(effects
 				(font
@@
 			)
 		)
-		(property "Footprint" "Diode_SMD:D_0402_1005Metric_Pad0.77x0.64mm_HandSolder"
-			(at 266.7 386.08 0)
+		(property "Footprint" "Library:DO-214BA_MCH-L"
+			(at 266.7 389.89 0)
 			(effects
 				(font
@@
 		)
 		(property "Datasheet" "~"
-			(at 266.7 386.08 0)
+			(at 266.7 389.89 0)
 			(effects
 				(font
@@
 		)
 		(property "Description" "Schottky diode"
-			(at 266.7 386.08 0)
+			(at 266.7 389.89 0)
 			(effects
 				(font
@@
 			)
 		)
-		(property "Footprint" "Capacitor_SMD:C_0402_1005Metric_Pad0.74x0.62mm_HandSolder"
+		(property "Footprint" "Capacitor_SMD:C_0603_1608Metric_Pad1.08x0.95mm_HandSolder"
 			(at 214.3252 391.16 0)
 			(effects

Commit message: double up for HASL
Connections:
- net A0: now also J1.173, J2.173, J3.173, J4.173
- net A1: now also J1.174, J2.174, J3.174, J4.174
- net A10: now also J1.189, J2.189, J3.189, J4.189
- net A11: now also J1.191, J2.191, J3.191, J4.191
- net A12: now also J1.197, J2.197, J3.197, J4.197
- net A13: now also J1.198, J2.198, J3.198, J4.198
- net A14: now also J1.199, J2.199, J3.199, J4.199
- net A15: now also J1.200, J2.200, J3.200, J4.200
- net A2: now also J1.175, J2.175, J3.175, J4.175
- net A3: now also J1.176, J2.176, J3.176, J4.176
- net A4: now also J1.177, J2.177, J3.177, J4.177
- net A5: now also J1.178, J2.178, J3.178, J4.178
- net A6: now also J1.179, J2.179, J3.179, J4.179
- net A7: now also J1.180, J2.180, J3.180, J4.180
- net A8: now also J1.185, J2.185, J3.185, J4.185
- net A9: now also J1.187, J2.187, J3.187, J4.187
- net BEX082: now also J1.226, J2.226, J3.226, J4.226
- net BEX083: now also J1.227, J2.227, J3.227, J4.227
- net BEX084: now also J1.228, J2.228, J3.228, J4.228
- net BEX085: now also J1.229, J2.229, J3.229, J4.229
- net BEX086: now also J1.230, J2.230, J3.230, J4.230
- net BEX087: now also J1.231, J2.231, J3.231, J4.231
- net BEX088: now also J1.232, J2.232, J3.232, J4.232
- net BEX089: now also J1.233, J2.233, J3.233, J4.233
- net BEX094: now also J1.238, J2.238, J3.238, J4.238
- net BEX095: now also J1.239, J2.239, J3.239, J4.239
- net BEX096: now also J1.240, J2.240, J3.240, J4.240
- net BEX097: now also J1.241, J2.241, J3.241, J4.241
- net BEX098: now also J1.242, J2.242, J3.242, J4.242
- net BEX099: now also J1.243, J2.243, J3.243, J4.243
- net BEX100: now also J1.244, J2.244, J3.244, J4.244
- net BEX101: now also J1.245, J2.245, J3.245, J4.245
- net BEX106: now also J1.250, J2.250, J3.250, J4.250
- net BEX107: now also J1.251, J2.251, J3.251, J4.251
- net BEX108: now also J1.252, J2.252, J3.252, J4.252
- net BEX109: now also J1.253, J2.253, J3.253, J4.253
- net BEX110: now also J1.254, J2.254, J3.254, J4.254
- net BEX111: now also J1.255, J2.255, J3.255, J4.255
- net BEX112: now also J1.256, J2.256, J3.256, J4.256
- net BEX113: now also J1.257, J2.257, J3.257, J4.257
- net BEX118: now also J1.262, J2.262, J3.262, J4.262
- net BEX119: now also J1.263, J2.263, J3.263, J4.263
- net BEX120: now also J1.264, J2.264, J3.264, J4.264
- net BEX121: now also J1.265, J2.265, J3.265, J4.265
- net BEX122: now also J1.266, J2.266, J3.266, J4.266
- net BEX123: now also J1.267, J2.267, J3.267, J4.267
- net BEX124: now also J1.268, J2.268, J3.268, J4.268
- net BEX125: now also J1.269, J2.269, J3.269, J4.269
- net CLOCK: now also J1.156, J2.156, J3.156, J4.156
- net D0: now also J1.161, J2.161, J3.161, J4.161
- net D1: now also J1.162, J2.162, J3.162, J4.162
- net D2: now also J1.163, J2.163, J3.163, J4.163
- net D3: now also J1.164, J2.164, J3.164, J4.164
- net D4: now also J1.165, J2.165, J3.165, J4.165
- net D5: now also J1.166, J2.166, J3.166, J4.166
- net D6: now also J1.167, J2.167, J3.167, J4.167
- net D7: now also J1.168, J2.168, J3.168, J4.168
- net DBIN: now also J1.155, J2.155, J3.155, J4.155
- net HLDA: now also J1.192, J2.192, J3.192, J4.192
- net HLTA: now also J1.209, J2.209, J3.209, J4.209
- net INP: now also J1.204, J2.204, J3.204, J4.204
- net INT: now also J1.212, J2.212, J3.212, J4.212
- net INTA: now also J1.152, J2.152, J3.152, J4.152
- net INTE: now also J1.188, J2.188, J3.188, J4.188
- net M1: now also J1.202, J2.202, J3.202, J4.202
- net MEMR: now also J1.203, J2.203, J3.203, J4.203
- net MWRT: now also J1.154, J2.154, J3.154, J4.154
- net OUT: now also J1.201, J2.201, J3.201, J4.201
- net PANEL: now also J1.153, J2.153, J3.153, J4.153
- net PRDY: now also J1.150, J2.150, J3.150, J4.150
- net PROT: now also J1.186, J2.186, J3.186, J4.186
- net RESET: now also J1.149, J2.149, J3.149, J4.149
- net STACK: now also J1.210, J2.210, J3.210, J4.210
- net WAIT: now also J1.190, J2.190, J3.190, J4.190
- net WO: now also J1.211, J2.211, J3.211, J4.211
- net XRDY: now also J1.151, J2.151, J3.151, J4.151
- no-connect marks 450 -> 146
Other:
- note added: "USB-C Port (Power)"
- note removed: "USB-C Port (Programming)"
- moved on the sheet: D4, J1C, J1D, R1, R2, R4, S1
