File: ecad/backplane/backplane.kicad_pcb (KiCad board)
At the start: 2 copper layers, 160 x 220 mm, 22 parts, among them J1 10145891-0320J13LF, J2 10145891-0320J13LF, J3 USB4105-GF-A, J4 10145891-0320J13LF, J5 10145891-0320J13LF, J6 5017868090, U1 MCP16331x-xCH

Commit message: backplane with addr
Parts:
- removed R4: 5.1k, Resistor_SMD:R_0402_1005Metric
- R3: value 5.1k -> 10; footprint Resistor_SMD:R_0402_1005Metric -> Resistor_SMD:R_0402_1005Metric_Pad0.72x0.64mm_HandSolder
- moved J3 128.3 mm to (87.9, 35.7), turned to 180 degrees
- moved R3 123.2 mm to (92.5, 52.2), turned to 0 degrees
- moved R1 121.8 mm to (86.2, 43.0), turned to -90 degrees
- moved D1 120.5 mm to (85.4, 51.6), turned to 180 degrees
- moved R2 119.1 mm to (89.2, 42.8), turned to -90 degrees
- moved C1 116.3 mm to (82.3, 53.6), turned to 90 degrees
- moved DB1 116.0 mm to (90.0, 53.5), turned to 180 degrees
- moved C2 115.1 mm to (83.6, 53.5), turned to 90 degrees
- moved Cln_2 114.9 mm to (85.2, 49.3), turned to 180 degrees
- moved L1 114.8 mm to (87.3, 54.7), turned to 180 degrees
- moved Cln_1 114.8 mm to (85.2, 48.1), turned to 180 degrees
- moved U1 114.6 mm to (88.8, 49.3), turned to 180 degrees
- moved CB1 111.3 mm to (87.9, 51.8), turned to 180 degrees
- moved RBot1 110.9 mm to (92.3, 49.0), turned to 180 degrees
- moved RTop1 110.3 mm to (93.0, 50.5), turned to 180 degrees
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Connections:
- net +5V renamed VBUS
- CB1 pad 2: Net-(U1-BOOST) -> Net-(D1-K)
- J3 pad A5: unconnected-(J3-CC1-PadA5) -> Net-(J3-CC1)
- J3 pad B5: unconnected-(J3-CC2-PadB5) -> Net-(J3-CC2)
- J3 pad B6: Net-(J3-DP2) -> unconnected-(J3-DP2-PadB6)
- J3 pad B7: Net-(J3-DN2) -> unconnected-(J3-DN2-PadB7)
- R1 pad 1: Net-(J3-DN2) -> Net-(J3-CC2)
- R2 pad 1: Net-(J3-DP2) -> Net-(J3-CC1)
- R3 pad 1: Net-(J6-DN2) -> Net-(R3-Pad1)
- R3 pad 2: GND -> 3.3V IN
- RTop1 pad 2: 3.3V IN -> Net-(R3-Pad1)
- U1 pad 1: Net-(U1-BOOST) -> Net-(DB1-K)
Routing:
- net 3.3V IN: track 0.00 -> 190.4 mm, vias 0 -> 3
- net GND: track 24.8 -> 137.3 mm, vias 2 -> 72
- net VBUS: track 11.8 -> 1.90 mm
- net Net-(U1-V_{FB}): track 0.00 -> 5.36 mm
- net Net-(DB1-K): track 0.00 -> 5.11 mm
- net Net-(J6-DN2): track 3.30 -> 0.00 mm
- net Net-(J6-DP2): track 3.17 -> 0.00 mm
- net Net-(R3-Pad1): track 0.00 -> 3.00 mm, vias 0 -> 1
- net Net-(J3-CC2): track 0.00 -> 1.96 mm
- net Net-(J3-CC1): track 0.00 -> 1.81 mm
- net Net-(D1-K): vias 0 -> 1
- added copper zone on F.Cu, net 3.3V
- added copper zone on F.Cu, net 3.3V IN
- added copper zone on B.Cu, net GND
- added copper zone on F.Cu, net GND
- added copper zone on F.Cu, net Net-(D1-K)
- added copper zone on F.Cu, net VBUS

Commit message: Backplane changes
Parts:
- added D2: HEARTBEAT, LED_SMD:LED_0603_1608Metric_Pad1.05x0.95mm_HandSolder, F.Cu at (109.1, 66.5)
- added D3: D_Schottky, Diode_SMD:D_0402_1005Metric_Pad0.77x0.64mm_HandSolder, F.Cu at (95.7, 66.2)
- added D4: HEARTBEAT, LED_SMD:LED_0603_1608Metric_Pad1.05x0.95mm_HandSolder, F.Cu at (109.1, 69.0)
- added R4: 150, Resistor_SMD:R_0402_1005Metric, F.Cu at (112.8, 66.2)
- added R5: 150, Resistor_SMD:R_0402_1005Metric, F.Cu at (92.8, 36.8)
- J3: value USB4105-GF-A -> 10145891-0320J13LF; footprint Library:GCT_USB4105-GF-A -> Library:AMPHENOL_10145891-0320J13LF
- J5: value 10145891-0320J13LF -> USB4105-GF-A; footprint Library:AMPHENOL_10145891-0320J13LF -> Library:GCT_USB4105-GF-A
- moved R1 255.0 mm to (340.9, 53.8)
- moved R2 252.1 mm to (340.9, 55.7), turned to 90 degrees
- moved J5 229.4 mm to (347.0, 55.0)
- moved S1 200.5 mm to (140.8, 50.0), turned to 0 degrees
- moved J3 185.2 mm to (258.3, 108.3), turned to 0 degrees
- moved J2 156.0 mm to (258.3, 73.3), turned to 0 degrees
- moved J1 155.7 mm to (258.3, 178.3), turned to 0 degrees
- moved J4 105.4 mm to (258.3, 143.3), turned to 0 degrees
- moved J6 88.4 mm to (162.0, 158.6), turned to 90 degrees
- moved R3 72.9 mm to (160.8, 77.5)
- moved RBot1 72.0 mm to (160.9, 71.1)
- moved RTop1 71.8 mm to (160.8, 74.1)
- moved CB1 71.7 mm to (155.3, 76.2)
- moved U1 70.5 mm to (155.3, 72.5)
- moved DB1 70.0 mm to (155.3, 78.8)
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Connections:
- C1 pad 1: 3.3V IN -> 3.3V
- C2 pad 1: 3.3V IN -> 3.3V
- Cln_1 pad 1: VBUS -> 5V
- Cln_2 pad 1: VBUS -> 5V
- DB1 pad 2: 3.3V IN -> 3.3V
- J1 pad 10: /BUS10 -> MWRT
- J1 pad 100: unconnected-(J1-Pad100) -> BEX100
- J1 pad 101: unconnected-(J1-Pad101) -> BEX101
- J1 pad 102: unconnected-(J1-Pad102) -> 3.3V
- J1 pad 103: unconnected-(J1-Pad103) -> 3.3V
- J1 pad 104: unconnected-(J1-Pad104) -> GND
- J1 pad 105: unconnected-(J1-Pad105) -> GND
- J1 pad 106: unconnected-(J1-Pad106) -> BEX106
- J1 pad 107: unconnected-(J1-Pad107) -> BEX107
- J1 pad 108: unconnected-(J1-Pad108) -> BEX108
- J1 pad 109: unconnected-(J1-Pad109) -> BEX109
- J1 pad 11: /BUS11 -> DBIN
- J1 pad 110: unconnected-(J1-Pad110) -> BEX110
- J1 pad 111: unconnected-(J1-Pad111) -> BEX111
- J1 pad 112: unconnected-(J1-Pad112) -> BEX112
- J1 pad 113: unconnected-(J1-Pad113) -> BEX113
- J1 pad 114: unconnected-(J1-Pad114) -> 3.3V
- J1 pad 115: unconnected-(J1-Pad115) -> 3.3V
- J1 pad 116: unconnected-(J1-Pad116) -> GND
- J1 pad 117: unconnected-(J1-Pad117) -> GND
- J1 pad 118: unconnected-(J1-Pad118) -> BEX118
- J1 pad 119: unconnected-(J1-Pad119) -> BEX119
- J1 pad 12: /BUS12 -> CLOCK
- J1 pad 120: unconnected-(J1-Pad120) -> BEX120
- J1 pad 121: unconnected-(J1-Pad121) -> BEX121
- J1 pad 122: unconnected-(J1-Pad122) -> BEX122
- J1 pad 123: unconnected-(J1-Pad123) -> BEX123
- J1 pad 124: unconnected-(J1-Pad124) -> BEX124
- J1 pad 125: unconnected-(J1-Pad125) -> BEX125
- J1 pad 126: unconnected-(J1-Pad126) -> 3.3V
- J1 pad 127: unconnected-(J1-Pad127) -> 3.3V
- J1 pad 128: unconnected-(J1-Pad128) -> GND
- J1 pad 129: unconnected-(J1-Pad129) -> GND
- J1 pad 138: unconnected-(J1-Pad138) -> 3.3V
- J1 pad 139: unconnected-(J1-Pad139) -> 3.3V
- J1 pad 140: unconnected-(J1-Pad140) -> GND
- J1 pad 141: unconnected-(J1-Pad141) -> GND
- J1 pad 145: unconnected-(J1-Pad145) -> 3.3V
- J1 pad 146: unconnected-(J1-Pad146) -> 3.3V
- J1 pad 147: unconnected-(J1-Pad147) -> GND
- J1 pad 148: unconnected-(J1-Pad148) -> GND
- J1 pad 157: unconnected-(J1-Pad157) -> 3.3V
- J1 pad 158: unconnected-(J1-Pad158) -> 3.3V
- J1 pad 159: unconnected-(J1-Pad159) -> GND
- J1 pad 160: unconnected-(J1-Pad160) -> GND
- J1 pad 169: unconnected-(J1-Pad169) -> 3.3V
- J1 pad 17: /BUS17 -> D0
- J1 pad 170: unconnected-(J1-Pad170) -> 3.3V
- J1 pad 171: unconnected-(J1-Pad171) -> GND
- J1 pad 172: unconnected-(J1-Pad172) -> GND
- J1 pad 18: /BUS18 -> D1
- J1 pad 181: unconnected-(J1-Pad181) -> 3.3V
- J1 pad 182: unconnected-(J1-Pad182) -> 3.3V
- J1 pad 183: unconnected-(J1-Pad183) -> GND
- J1 pad 184: unconnected-(J1-Pad184) -> GND
- J1 pad 19: /BUS19 -> D2
- J1 pad 193: unconnected-(J1-Pad193) -> 3.3V
- J1 pad 194: unconnected-(J1-Pad194) -> 3.3V
- J1 pad 195: unconnected-(J1-Pad195) -> GND
- J1 pad 196: unconnected-(J1-Pad196) -> GND
- J1 pad 20: /BUS20 -> D3
- J1 pad 205: unconnected-(J1-Pad205) -> 3.3V
- J1 pad 206: unconnected-(J1-Pad206) -> 3.3V
- J1 pad 207: unconnected-(J1-Pad207) -> GND
- J1 pad 208: unconnected-(J1-Pad208) -> GND
- J1 pad 21: /BUS21 -> D4
- J1 pad 217: unconnected-(J1-Pad217) -> 3.3V
- J1 pad 218: unconnected-(J1-Pad218) -> 3.3V
- J1 pad 219: unconnected-(J1-Pad219) -> GND
- J1 pad 22: /BUS22 -> D5
- J1 pad 220: unconnected-(J1-Pad220) -> GND
- J1 pad 222: unconnected-(J1-Pad222) -> 3.3V
- J1 pad 223: unconnected-(J1-Pad223) -> 3.3V
- J1 pad 224: unconnected-(J1-Pad224) -> GND
- J1 pad 225: unconnected-(J1-Pad225) -> GND
- J1 pad 23: /BUS23 -> D6
- J1 pad 234: unconnected-(J1-Pad234) -> 3.3V
- J1 pad 235: unconnected-(J1-Pad235) -> 3.3V
- J1 pad 236: unconnected-(J1-Pad236) -> GND
- J1 pad 237: unconnected-(J1-Pad237) -> GND
- J1 pad 24: /BUS24 -> D7
- J1 pad 246: unconnected-(J1-Pad246) -> 3.3V
- J1 pad 247: unconnected-(J1-Pad247) -> 3.3V
- J1 pad 248: unconnected-(J1-Pad248) -> GND
- J1 pad 249: unconnected-(J1-Pad249) -> GND
- J1 pad 258: unconnected-(J1-Pad258) -> 3.3V
- J1 pad 259: unconnected-(J1-Pad259) -> 3.3V
- J1 pad 260: unconnected-(J1-Pad260) -> GND
- J1 pad 261: unconnected-(J1-Pad261) -> GND
- J1 pad 270: unconnected-(J1-Pad270) -> 3.3V
- J1 pad 271: unconnected-(J1-Pad271) -> 3.3V
- J1 pad 272: unconnected-(J1-Pad272) -> GND
- J1 pad 273: unconnected-(J1-Pad273) -> GND
- J1 pad 282: unconnected-(J1-Pad282) -> 3.3V
- J1 pad 283: unconnected-(J1-Pad283) -> 3.3V
- J1 pad 284: unconnected-(J1-Pad284) -> GND
- J1 pad 285: unconnected-(J1-Pad285) -> GND
- J1 pad 29: /BUS29 -> A0
- J1 pad 30: /BUS30 -> A1
- J1 pad 31: /BUS31 -> A2
- J1 pad 32: /BUS32 -> A3
- J1 pad 33: /BUS33 -> A4
- J1 pad 34: /BUS34 -> A5
- J1 pad 35: /BUS35 -> A6
- J1 pad 36: /BUS36 -> A7
- J1 pad 41: /BUS41 -> A8
- J1 pad 42: /BUS42 -> PROT
- J1 pad 43: /BUS43 -> A9
- J1 pad 44: /BUS44 -> INTE
- J1 pad 45: /BUS45 -> A10
- J1 pad 46: /BUS46 -> WAIT
- J1 pad 47: /BUS47 -> A11
- J1 pad 48: /BUS48 -> HLDA
- J1 pad 5: /BUS05 -> RESET
- J1 pad 53: /BUS53 -> A12
- J1 pad 54: /BUS54 -> A13
- J1 pad 55: /BUS55 -> A14
- J1 pad 56: /BUS56 -> A15
- J1 pad 57: /BUS57 -> OUT
- J1 pad 58: /BUS58 -> M1
- J1 pad 59: /BUS59 -> MEMR
- J1 pad 6: /BUS06 -> PRDY
- J1 pad 60: /BUS60 -> INP
- J1 pad 65: /BUS65 -> HLTA
- J1 pad 66: /BUS66 -> STACK
- J1 pad 67: /BUS67 -> WO
- J1 pad 68: /BUS68 -> INT
- J1 pad 69: /BUS69 -> unconnected-(J1-Pad69)
- J1 pad 7: /BUS07 -> XRDY
- J1 pad 70: /BUS70 -> unconnected-(J1-Pad70)
- J1 pad 71: /BUS71 -> unconnected-(J1-Pad71)
- J1 pad 72: /BUS72 -> unconnected-(J1-Pad72)
- J1 pad 78: unconnected-(J1-Pad78) -> 3.3V
- J1 pad 79: unconnected-(J1-Pad79) -> 3.3V
- J1 pad 8: /BUS08 -> INTA
- J1 pad 80: unconnected-(J1-Pad80) -> GND
- J1 pad 81: unconnected-(J1-Pad81) -> GND
- J1 pad 82: unconnected-(J1-Pad82) -> BEX082
- J1 pad 83: unconnected-(J1-Pad83) -> BEX083
- J1 pad 84: unconnected-(J1-Pad84) -> BEX084
- J1 pad 85: unconnected-(J1-Pad85) -> BEX085
- J1 pad 86: unconnected-(J1-Pad86) -> BEX086
- J1 pad 87: unconnected-(J1-Pad87) -> BEX087
- J1 pad 88: unconnected-(J1-Pad88) -> BEX088
- J1 pad 89: unconnected-(J1-Pad89) -> BEX089
- J1 pad 9: /BUS09 -> PANEL
- J1 pad 90: unconnected-(J1-Pad90) -> 3.3V
- J1 pad 91: unconnected-(J1-Pad91) -> 3.3V
- J1 pad 92: unconnected-(J1-Pad92) -> GND
- J1 pad 93: unconnected-(J1-Pad93) -> GND
- J1 pad 94: unconnected-(J1-Pad94) -> BEX094
- J1 pad 95: unconnected-(J1-Pad95) -> BEX095
- J1 pad 96: unconnected-(J1-Pad96) -> BEX096
- J1 pad 97: unconnected-(J1-Pad97) -> BEX097
- J1 pad 98: unconnected-(J1-Pad98) -> BEX098
- J1 pad 99: unconnected-(J1-Pad99) -> BEX099
- J2 pad 10: /BUS10 -> MWRT
- J2 pad 100: unconnected-(J2-Pad100) -> BEX100
- J2 pad 101: unconnected-(J2-Pad101) -> BEX101
- J2 pad 102: unconnected-(J2-Pad102) -> 3.3V
- J2 pad 103: unconnected-(J2-Pad103) -> 3.3V
- J2 pad 104: unconnected-(J2-Pad104) -> GND
- J2 pad 105: unconnected-(J2-Pad105) -> GND
- J2 pad 106: unconnected-(J2-Pad106) -> BEX106
- J2 pad 107: unconnected-(J2-Pad107) -> BEX107
- J2 pad 108: unconnected-(J2-Pad108) -> BEX108
- J2 pad 109: unconnected-(J2-Pad109) -> BEX109
- J2 pad 11: /BUS11 -> DBIN
- J2 pad 110: unconnected-(J2-Pad110) -> BEX110
- J2 pad 111: unconnected-(J2-Pad111) -> BEX111
- J2 pad 112: unconnected-(J2-Pad112) -> BEX112
- J2 pad 113: unconnected-(J2-Pad113) -> BEX113
- J2 pad 114: unconnected-(J2-Pad114) -> 3.3V
- J2 pad 115: unconnected-(J2-Pad115) -> 3.3V
- J2 pad 116: unconnected-(J2-Pad116) -> GND
- J2 pad 117: unconnected-(J2-Pad117) -> GND
- J2 pad 118: unconnected-(J2-Pad118) -> BEX118
- J2 pad 119: unconnected-(J2-Pad119) -> BEX119
- J2 pad 12: /BUS12 -> CLOCK
- J2 pad 120: unconnected-(J2-Pad120) -> BEX120
- J2 pad 121: unconnected-(J2-Pad121) -> BEX121
- J2 pad 122: unconnected-(J2-Pad122) -> BEX122
- J2 pad 123: unconnected-(J2-Pad123) -> BEX123
- J2 pad 124: unconnected-(J2-Pad124) -> BEX124
- J2 pad 125: unconnected-(J2-Pad125) -> BEX125
- J2 pad 126: unconnected-(J2-Pad126) -> 3.3V
- J2 pad 127: unconnected-(J2-Pad127) -> 3.3V
- J2 pad 128: unconnected-(J2-Pad128) -> GND
- J2 pad 129: unconnected-(J2-Pad129) -> GND
- J2 pad 138: unconnected-(J2-Pad138) -> 3.3V
- J2 pad 139: unconnected-(J2-Pad139) -> 3.3V
- J2 pad 140: unconnected-(J2-Pad140) -> GND
- J2 pad 141: unconnected-(J2-Pad141) -> GND
- J2 pad 145: unconnected-(J2-Pad145) -> 3.3V
- J2 pad 146: unconnected-(J2-Pad146) -> 3.3V
- J2 pad 147: unconnected-(J2-Pad147) -> GND
- J2 pad 148: unconnected-(J2-Pad148) -> GND
- J2 pad 157: unconnected-(J2-Pad157) -> 3.3V
- J2 pad 158: unconnected-(J2-Pad158) -> 3.3V
- J2 pad 159: unconnected-(J2-Pad159) -> GND
- J2 pad 160: unconnected-(J2-Pad160) -> GND
- J2 pad 169: unconnected-(J2-Pad169) -> 3.3V
- J2 pad 17: /BUS17 -> D0
- J2 pad 170: unconnected-(J2-Pad170) -> 3.3V
- J2 pad 171: unconnected-(J2-Pad171) -> GND
- J2 pad 172: unconnected-(J2-Pad172) -> GND
- J2 pad 18: /BUS18 -> D1
- J2 pad 181: unconnected-(J2-Pad181) -> 3.3V
- J2 pad 182: unconnected-(J2-Pad182) -> 3.3V
- J2 pad 183: unconnected-(J2-Pad183) -> GND
- J2 pad 184: unconnected-(J2-Pad184) -> GND
- J2 pad 19: /BUS19 -> D2
- J2 pad 193: unconnected-(J2-Pad193) -> 3.3V
- J2 pad 194: unconnected-(J2-Pad194) -> 3.3V
- J2 pad 195: unconnected-(J2-Pad195) -> GND
- J2 pad 196: unconnected-(J2-Pad196) -> GND
- J2 pad 20: /BUS20 -> D3
- J2 pad 205: unconnected-(J2-Pad205) -> 3.3V
- J2 pad 206: unconnected-(J2-Pad206) -> 3.3V
- J2 pad 207: unconnected-(J2-Pad207) -> GND
- J2 pad 208: unconnected-(J2-Pad208) -> GND
- J2 pad 21: /BUS21 -> D4
- J2 pad 217: unconnected-(J2-Pad217) -> 3.3V
- J2 pad 218: unconnected-(J2-Pad218) -> 3.3V
- J2 pad 219: unconnected-(J2-Pad219) -> GND
- J2 pad 22: /BUS22 -> D5
- J2 pad 220: unconnected-(J2-Pad220) -> GND
- J2 pad 222: unconnected-(J2-Pad222) -> 3.3V
- J2 pad 223: unconnected-(J2-Pad223) -> 3.3V
- J2 pad 224: unconnected-(J2-Pad224) -> GND
- J2 pad 225: unconnected-(J2-Pad225) -> GND
- J2 pad 23: /BUS23 -> D6
- J2 pad 234: unconnected-(J2-Pad234) -> 3.3V
- J2 pad 235: unconnected-(J2-Pad235) -> 3.3V
- J2 pad 236: unconnected-(J2-Pad236) -> GND
- J2 pad 237: unconnected-(J2-Pad237) -> GND
- J2 pad 24: /BUS24 -> D7
- J2 pad 246: unconnected-(J2-Pad246) -> 3.3V
- J2 pad 247: unconnected-(J2-Pad247) -> 3.3V
- J2 pad 248: unconnected-(J2-Pad248) -> GND
- J2 pad 249: unconnected-(J2-Pad249) -> GND
- J2 pad 258: unconnected-(J2-Pad258) -> 3.3V
- J2 pad 259: unconnected-(J2-Pad259) -> 3.3V
- J2 pad 260: unconnected-(J2-Pad260) -> GND
- J2 pad 261: unconnected-(J2-Pad261) -> GND
- J2 pad 270: unconnected-(J2-Pad270) -> 3.3V
- J2 pad 271: unconnected-(J2-Pad271) -> 3.3V
- J2 pad 272: unconnected-(J2-Pad272) -> GND
- J2 pad 273: unconnected-(J2-Pad273) -> GND
- J2 pad 282: unconnected-(J2-Pad282) -> 3.3V
- J2 pad 283: unconnected-(J2-Pad283) -> 3.3V
- J2 pad 284: unconnected-(J2-Pad284) -> GND
- J2 pad 285: unconnected-(J2-Pad285) -> GND
- J2 pad 29: /BUS29 -> A0
- J2 pad 30: /BUS30 -> A1
- J2 pad 31: /BUS31 -> A2
- J2 pad 32: /BUS32 -> A3
- J2 pad 33: /BUS33 -> A4
- J2 pad 34: /BUS34 -> A5
- J2 pad 35: /BUS35 -> A6
- J2 pad 36: /BUS36 -> A7
- J2 pad 41: /BUS41 -> A8
- J2 pad 42: /BUS42 -> PROT
- J2 pad 43: /BUS43 -> A9
- J2 pad 44: /BUS44 -> INTE
- J2 pad 45: /BUS45 -> A10
- J2 pad 46: /BUS46 -> WAIT
- J2 pad 47: /BUS47 -> A11
- J2 pad 48: /BUS48 -> HLDA
- J2 pad 5: /BUS05 -> RESET
- J2 pad 53: /BUS53 -> A12
- J2 pad 54: /BUS54 -> A13
- J2 pad 55: /BUS55 -> A14
- J2 pad 56: /BUS56 -> A15
- J2 pad 57: /BUS57 -> OUT
- J2 pad 58: /BUS58 -> M1
- J2 pad 59: /BUS59 -> MEMR
- J2 pad 6: /BUS06 -> PRDY
- J2 pad 60: /BUS60 -> INP
- J2 pad 65: /BUS65 -> HLTA
- J2 pad 66: /BUS66 -> STACK
- J2 pad 67: /BUS67 -> WO
- J2 pad 68: /BUS68 -> INT
- J2 pad 69: /BUS69 -> unconnected-(J2-Pad69)
- J2 pad 7: /BUS07 -> XRDY
- J2 pad 70: /BUS70 -> unconnected-(J2-Pad70)
- J2 pad 71: /BUS71 -> unconnected-(J2-Pad71)
- J2 pad 72: /BUS72 -> unconnected-(J2-Pad72)
- J2 pad 78: unconnected-(J2-Pad78) -> 3.3V
- J2 pad 79: unconnected-(J2-Pad79) -> 3.3V
- J2 pad 8: /BUS08 -> INTA
- J2 pad 80: unconnected-(J2-Pad80) -> GND
- J2 pad 81: unconnected-(J2-Pad81) -> GND
- J2 pad 82: unconnected-(J2-Pad82) -> BEX082
- J2 pad 83: unconnected-(J2-Pad83) -> BEX083
- J2 pad 84: unconnected-(J2-Pad84) -> BEX084
- J2 pad 85: unconnected-(J2-Pad85) -> BEX085
- J2 pad 86: unconnected-(J2-Pad86) -> BEX086
- J2 pad 87: unconnected-(J2-Pad87) -> BEX087
- J2 pad 88: unconnected-(J2-Pad88) -> BEX088
- J2 pad 89: unconnected-(J2-Pad89) -> BEX089
- J2 pad 9: /BUS09 -> PANEL
- J2 pad 90: unconnected-(J2-Pad90) -> 3.3V
- J2 pad 91: unconnected-(J2-Pad91) -> 3.3V
- J2 pad 92: unconnected-(J2-Pad92) -> GND
- J2 pad 93: unconnected-(J2-Pad93) -> GND
- J2 pad 94: unconnected-(J2-Pad94) -> BEX094
- J2 pad 95: unconnected-(J2-Pad95) -> BEX095
- J2 pad 96: unconnected-(J2-Pad96) -> BEX096
- J2 pad 97: unconnected-(J2-Pad97) -> BEX097
- J2 pad 98: unconnected-(J2-Pad98) -> BEX098
- J2 pad 99: unconnected-(J2-Pad99) -> BEX099
- J4 pad 10: /BUS10 -> MWRT
- J4 pad 100: unconnected-(J4-Pad100) -> BEX100
- J4 pad 101: unconnected-(J4-Pad101) -> BEX101
- J4 pad 102: unconnected-(J4-Pad102) -> 3.3V
- J4 pad 103: unconnected-(J4-Pad103) -> 3.3V
- J4 pad 104: unconnected-(J4-Pad104) -> GND
- J4 pad 105: unconnected-(J4-Pad105) -> GND
- J4 pad 106: unconnected-(J4-Pad106) -> BEX106
- J4 pad 107: unconnected-(J4-Pad107) -> BEX107
- J4 pad 108: unconnected-(J4-Pad108) -> BEX108
- J4 pad 109: unconnected-(J4-Pad109) -> BEX109
- J4 pad 11: /BUS11 -> DBIN
- J4 pad 110: unconnected-(J4-Pad110) -> BEX110
- J4 pad 111: unconnected-(J4-Pad111) -> BEX111
- J4 pad 112: unconnected-(J4-Pad112) -> BEX112
- J4 pad 113: unconnected-(J4-Pad113) -> BEX113
- J4 pad 114: unconnected-(J4-Pad114) -> 3.3V
- J4 pad 115: unconnected-(J4-Pad115) -> 3.3V
- J4 pad 116: unconnected-(J4-Pad116) -> GND
- J4 pad 117: unconnected-(J4-Pad117) -> GND
- J4 pad 118: unconnected-(J4-Pad118) -> BEX118
- J4 pad 119: unconnected-(J4-Pad119) -> BEX119
- J4 pad 12: /BUS12 -> CLOCK
- J4 pad 120: unconnected-(J4-Pad120) -> BEX120
- J4 pad 121: unconnected-(J4-Pad121) -> BEX121
- J4 pad 122: unconnected-(J4-Pad122) -> BEX122
- J4 pad 123: unconnected-(J4-Pad123) -> BEX123
- J4 pad 124: unconnected-(J4-Pad124) -> BEX124
- J4 pad 125: unconnected-(J4-Pad125) -> BEX125
- J4 pad 126: unconnected-(J4-Pad126) -> 3.3V
- J4 pad 127: unconnected-(J4-Pad127) -> 3.3V
- J4 pad 128: unconnected-(J4-Pad128) -> GND
- J4 pad 129: unconnected-(J4-Pad129) -> GND
- J4 pad 138: unconnected-(J4-Pad138) -> 3.3V
- J4 pad 139: unconnected-(J4-Pad139) -> 3.3V
- J4 pad 140: unconnected-(J4-Pad140) -> GND
- J4 pad 141: unconnected-(J4-Pad141) -> GND
- J4 pad 145: unconnected-(J4-Pad145) -> 3.3V
- J4 pad 146: unconnected-(J4-Pad146) -> 3.3V
- J4 pad 147: unconnected-(J4-Pad147) -> GND
- J4 pad 148: unconnected-(J4-Pad148) -> GND
- J4 pad 157: unconnected-(J4-Pad157) -> 3.3V
- J4 pad 158: unconnected-(J4-Pad158) -> 3.3V
- J4 pad 159: unconnected-(J4-Pad159) -> GND
- J4 pad 160: unconnected-(J4-Pad160) -> GND
- J4 pad 169: unconnected-(J4-Pad169) -> 3.3V
- J4 pad 17: /BUS17 -> D0
- J4 pad 170: unconnected-(J4-Pad170) -> 3.3V
- J4 pad 171: unconnected-(J4-Pad171) -> GND
- J4 pad 172: unconnected-(J4-Pad172) -> GND
- J4 pad 18: /BUS18 -> D1
- J4 pad 181: unconnected-(J4-Pad181) -> 3.3V
- J4 pad 182: unconnected-(J4-Pad182) -> 3.3V
- J4 pad 183: unconnected-(J4-Pad183) -> GND
- J4 pad 184: unconnected-(J4-Pad184) -> GND
- J4 pad 19: /BUS19 -> D2
- J4 pad 193: unconnected-(J4-Pad193) -> 3.3V
- J4 pad 194: unconnected-(J4-Pad194) -> 3.3V
- J4 pad 195: unconnected-(J4-Pad195) -> GND
- J4 pad 196: unconnected-(J4-Pad196) -> GND
- J4 pad 20: /BUS20 -> D3
- J4 pad 205: unconnected-(J4-Pad205) -> 3.3V
- J4 pad 206: unconnected-(J4-Pad206) -> 3.3V
- J4 pad 207: unconnected-(J4-Pad207) -> GND
- J4 pad 208: unconnected-(J4-Pad208) -> GND
- J4 pad 21: /BUS21 -> D4
- J4 pad 217: unconnected-(J4-Pad217) -> 3.3V
- J4 pad 218: unconnected-(J4-Pad218) -> 3.3V
- J4 pad 219: unconnected-(J4-Pad219) -> GND
- J4 pad 22: /BUS22 -> D5
- J4 pad 220: unconnected-(J4-Pad220) -> GND
- J4 pad 222: unconnected-(J4-Pad222) -> 3.3V
- J4 pad 223: unconnected-(J4-Pad223) -> 3.3V
- J4 pad 224: unconnected-(J4-Pad224) -> GND
- J4 pad 225: unconnected-(J4-Pad225) -> GND
- J4 pad 23: /BUS23 -> D6
- J4 pad 234: unconnected-(J4-Pad234) -> 3.3V
- J4 pad 235: unconnected-(J4-Pad235) -> 3.3V
- J4 pad 236: unconnected-(J4-Pad236) -> GND
- J4 pad 237: unconnected-(J4-Pad237) -> GND
- J4 pad 24: /BUS24 -> D7
- J4 pad 246: unconnected-(J4-Pad246) -> 3.3V
- J4 pad 247: unconnected-(J4-Pad247) -> 3.3V
- J4 pad 248: unconnected-(J4-Pad248) -> GND
- J4 pad 249: unconnected-(J4-Pad249) -> GND
- J4 pad 258: unconnected-(J4-Pad258) -> 3.3V
- J4 pad 259: unconnected-(J4-Pad259) -> 3.3V
- J4 pad 260: unconnected-(J4-Pad260) -> GND
- J4 pad 261: unconnected-(J4-Pad261) -> GND
- J4 pad 270: unconnected-(J4-Pad270) -> 3.3V
- J4 pad 271: unconnected-(J4-Pad271) -> 3.3V
- J4 pad 272: unconnected-(J4-Pad272) -> GND
- J4 pad 273: unconnected-(J4-Pad273) -> GND
- J4 pad 282: unconnected-(J4-Pad282) -> 3.3V
- J4 pad 283: unconnected-(J4-Pad283) -> 3.3V
- J4 pad 284: unconnected-(J4-Pad284) -> GND
- J4 pad 285: unconnected-(J4-Pad285) -> GND
- J4 pad 29: /BUS29 -> A0
- J4 pad 30: /BUS30 -> A1
- J4 pad 31: /BUS31 -> A2
- J4 pad 32: /BUS32 -> A3
- J4 pad 33: /BUS33 -> A4
- J4 pad 34: /BUS34 -> A5
- J4 pad 35: /BUS35 -> A6
- J4 pad 36: /BUS36 -> A7
- J4 pad 41: /BUS41 -> A8
- J4 pad 42: /BUS42 -> PROT
- J4 pad 43: /BUS43 -> A9
- J4 pad 44: /BUS44 -> INTE
- J4 pad 45: /BUS45 -> A10
- J4 pad 46: /BUS46 -> WAIT
- J4 pad 47: /BUS47 -> A11
- J4 pad 48: /BUS48 -> HLDA
- J4 pad 5: /BUS05 -> RESET
- J4 pad 53: /BUS53 -> A12
- J4 pad 54: /BUS54 -> A13
- J4 pad 55: /BUS55 -> A14
- J4 pad 56: /BUS56 -> A15
- J4 pad 57: /BUS57 -> OUT
- J4 pad 58: /BUS58 -> M1
- J4 pad 59: /BUS59 -> MEMR
- J4 pad 6: /BUS06 -> PRDY
- J4 pad 60: /BUS60 -> INP
- J4 pad 65: /BUS65 -> HLTA
- J4 pad 66: /BUS66 -> STACK
- J4 pad 67: /BUS67 -> WO
- J4 pad 68: /BUS68 -> INT
- J4 pad 69: /BUS69 -> unconnected-(J4-Pad69)
- J4 pad 7: /BUS07 -> XRDY
- J4 pad 70: /BUS70 -> unconnected-(J4-Pad70)
- J4 pad 71: /BUS71 -> unconnected-(J4-Pad71)
- J4 pad 72: /BUS72 -> unconnected-(J4-Pad72)
- J4 pad 78: unconnected-(J4-Pad78) -> 3.3V
- J4 pad 79: unconnected-(J4-Pad79) -> 3.3V
- J4 pad 8: /BUS08 -> INTA
- J4 pad 80: unconnected-(J4-Pad80) -> GND
- J4 pad 81: unconnected-(J4-Pad81) -> GND
- J4 pad 82: unconnected-(J4-Pad82) -> BEX082
- J4 pad 83: unconnected-(J4-Pad83) -> BEX083
- J4 pad 84: unconnected-(J4-Pad84) -> BEX084
- J4 pad 85: unconnected-(J4-Pad85) -> BEX085
- J4 pad 86: unconnected-(J4-Pad86) -> BEX086
- J4 pad 87: unconnected-(J4-Pad87) -> BEX087
- J4 pad 88: unconnected-(J4-Pad88) -> BEX088
- J4 pad 89: unconnected-(J4-Pad89) -> BEX089
- J4 pad 9: /BUS09 -> PANEL
- J4 pad 90: unconnected-(J4-Pad90) -> 3.3V
- J4 pad 91: unconnected-(J4-Pad91) -> 3.3V
- J4 pad 92: unconnected-(J4-Pad92) -> GND
- J4 pad 93: unconnected-(J4-Pad93) -> GND
- J4 pad 94: unconnected-(J4-Pad94) -> BEX094
- J4 pad 95: unconnected-(J4-Pad95) -> BEX095
- J4 pad 96: unconnected-(J4-Pad96) -> BEX096
- J4 pad 97: unconnected-(J4-Pad97) -> BEX097
- J4 pad 98: unconnected-(J4-Pad98) -> BEX098
- J4 pad 99: unconnected-(J4-Pad99) -> BEX099
- J6 pad 1: unconnected-(J6-Pad1) -> 3.3V
- J6 pad 10: unconnected-(J6-Pad10) -> A1
- J6 pad 11: unconnected-(J6-Pad11) -> D1
- J6 pad 12: unconnected-(J6-Pad12) -> D0
- J6 pad 13: unconnected-(J6-Pad13) -> 3.3V
- J6 pad 14: unconnected-(J6-Pad14) -> GND
- J6 pad 19: unconnected-(J6-Pad19) -> 3.3V
- J6 pad 2: unconnected-(J6-Pad2) -> GND
- J6 pad 20: unconnected-(J6-Pad20) -> GND
- J6 pad 21: unconnected-(J6-Pad21) -> RESET
- J6 pad 22: unconnected-(J6-Pad22) -> PRDY
- J6 pad 23: unconnected-(J6-Pad23) -> XRDY
- J6 pad 24: unconnected-(J6-Pad24) -> INTA
- J6 pad 25: unconnected-(J6-Pad25) -> 3.3V
- J6 pad 26: unconnected-(J6-Pad26) -> GND
- J6 pad 27: unconnected-(J6-Pad27) -> PANEL
- J6 pad 28: unconnected-(J6-Pad28) -> MWRT
- J6 pad 29: unconnected-(J6-Pad29) -> DBIN
- J6 pad 3: unconnected-(J6-Pad3) -> A3
- J6 pad 30: unconnected-(J6-Pad30) -> CLOCK
- J6 pad 31: unconnected-(J6-Pad31) -> 3.3V
- J6 pad 32: unconnected-(J6-Pad32) -> GND
- J6 pad 33: unconnected-(J6-Pad33) -> D7
- J6 pad 34: unconnected-(J6-Pad34) -> D6
- J6 pad 35: unconnected-(J6-Pad35) -> A6
- J6 pad 36: unconnected-(J6-Pad36) -> A7
- J6 pad 37: unconnected-(J6-Pad37) -> 3.3V
- J6 pad 38: unconnected-(J6-Pad38) -> GND
- J6 pad 4: unconnected-(J6-Pad4) -> D3
- J6 pad 42: unconnected-(J6-Pad42) -> GND
- J6 pad 43: unconnected-(J6-Pad43) -> 3.3V
- J6 pad 44: unconnected-(J6-Pad44) -> D5
- J6 pad 45: unconnected-(J6-Pad45) -> A5
- J6 pad 46: unconnected-(J6-Pad46) -> D4
- J6 pad 47: unconnected-(J6-Pad47) -> A4
- J6 pad 48: unconnected-(J6-Pad48) -> GND
- J6 pad 49: unconnected-(J6-Pad49) -> 3.3V
- J6 pad 5: unconnected-(J6-Pad5) -> A2
- J6 pad 50: unconnected-(J6-Pad50) -> PROT
- J6 pad 51: unconnected-(J6-Pad51) -> INTE
- J6 pad 52: unconnected-(J6-Pad52) -> WAIT
- J6 pad 53: unconnected-(J6-Pad53) -> HLDA
- J6 pad 54: unconnected-(J6-Pad54) -> GND
- J6 pad 55: unconnected-(J6-Pad55) -> 3.3V
- J6 pad 56: unconnected-(J6-Pad56) -> A12
- J6 pad 57: unconnected-(J6-Pad57) -> A13
- J6 pad 58: unconnected-(J6-Pad58) -> OUT
- J6 pad 59: unconnected-(J6-Pad59) -> M1
- J6 pad 6: unconnected-(J6-Pad6) -> D2
- J6 pad 60: unconnected-(J6-Pad60) -> GND
- J6 pad 61: unconnected-(J6-Pad61) -> 3.3V
- J6 pad 62: unconnected-(J6-Pad62) -> A14
- J6 pad 63: unconnected-(J6-Pad63) -> MEMR
- J6 pad 64: unconnected-(J6-Pad64) -> INP
- J6 pad 65: unconnected-(J6-Pad65) -> A15
- J6 pad 66: unconnected-(J6-Pad66) -> GND
- J6 pad 67: unconnected-(J6-Pad67) -> 3.3V
- J6 pad 68: unconnected-(J6-Pad68) -> HLTA
- J6 pad 69: unconnected-(J6-Pad69) -> STACK
- J6 pad 7: unconnected-(J6-Pad7) -> 3.3V
- J6 pad 70: unconnected-(J6-Pad70) -> A11
- J6 pad 71: unconnected-(J6-Pad71) -> WO
- J6 pad 72: unconnected-(J6-Pad72) -> GND
- J6 pad 73: unconnected-(J6-Pad73) -> 3.3V
- J6 pad 74: unconnected-(J6-Pad74) -> A10
- J6 pad 75: unconnected-(J6-Pad75) -> INT
- J6 pad 76: unconnected-(J6-Pad76) -> A9
- J6 pad 77: unconnected-(J6-Pad77) -> A8
- J6 pad 78: unconnected-(J6-Pad78) -> GND
- J6 pad 79: unconnected-(J6-Pad79) -> 3.3V
- J6 pad 8: unconnected-(J6-Pad8) -> GND
- J6 pad 9: unconnected-(J6-Pad9) -> A0
- L1 pad 2: 3.3V IN -> 3.3V
- R1 pad 1: Net-(J3-CC2) -> Net-(J5-CC2)
- R2 pad 1: Net-(J3-CC1) -> Net-(J5-CC1)
- R3 pad 2: 3.3V IN -> 3.3V
- S1 pad 1: 3.3V -> 5V
- S1 pad 2: 3.3V IN -> VBUS
- U1 pad 5: VBUS -> 5V
Routing:
- net INT: track 0.00 -> 194.5 mm, vias 0 -> 5
- net WO: track 0.00 -> 193.2 mm, vias 0 -> 5
- net STACK: track 0.00 -> 192.3 mm, vias 0 -> 5
- net HLTA: track 0.00 -> 191.4 mm, vias 0 -> 5
- net VBUS: track 1.90 -> 193.0 mm
- net 3.3V IN: track 190.4 -> 0.00 mm, vias 3 -> 0
- net INP: track 0.00 -> 186.9 mm, vias 0 -> 5
- net MEMR: track 0.00 -> 186.0 mm, vias 0 -> 5
- net M1: track 0.00 -> 185.2 mm, vias 0 -> 5
- net OUT: track 0.00 -> 184.4 mm, vias 0 -> 5
- net A15: track 0.00 -> 183.5 mm, vias 0 -> 5
- net A14: track 0.00 -> 182.6 mm, vias 0 -> 5
- net A13: track 0.00 -> 181.8 mm, vias 0 -> 6
- net A12: track 0.00 -> 180.9 mm, vias 0 -> 5
- net HLDA: track 0.00 -> 176.6 mm, vias 0 -> 5
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- removed copper zone on F.Cu, net 3.3V IN
- removed copper zone on F.Cu, net GND
- removed copper zone on F.Cu, net Net-(D1-K)
Other:
- board size 160 x 220 mm -> 220 x 160 mm

Commit message: Back Panel Done
Parts:
- removed C1, C2: 10u, Capacitor_SMD:C_0402_1005Metric_Pad0.74x0.62mm_HandSolder
- removed D3: D_Schottky, Diode_SMD:D_0402_1005Metric_Pad0.77x0.64mm_HandSolder
- added Cout_1: 10u, Capacitor_SMD:C_0402_1005Metric_Pad0.74x0.62mm_HandSolder, F.Cu at (115.5, 98.8)
- added Cout_2: 10u, Capacitor_SMD:C_0402_1005Metric_Pad0.74x0.62mm_HandSolder, F.Cu at (117.3, 98.8)
- Cln_1, Cln_2: footprint Capacitor_SMD:C_0402_1005Metric_Pad0.74x0.62mm_HandSolder -> Capacitor_SMD:C_0603_1608Metric_Pad1.08x0.95mm_HandSolder
- D1: footprint Diode_SMD:D_0402_1005Metric_Pad0.77x0.64mm_HandSolder -> Library:DO-214BA_MCH-L
- L1: footprint Inductor_SMD:L_0402_1005Metric_Pad0.77x0.64mm_HandSolder -> Library:DR73-150-R
- moved R5 91.8 mm to (149.1, 109.4)
- moved D2 54.5 mm to (142.6, 109.5), turned to 180 degrees
- moved L1 52.3 mm to (123.5, 104.0), turned to 180 degrees
- moved D1 44.0 mm to (123.2, 96.7), turned to 180 degrees
- moved J2 36.5 mm to (228.0, 93.7)
- moved J4 36.5 mm to (228.0, 163.6)
- moved J6 36.5 mm to (131.7, 178.9)
- moved J3 36.5 mm to (228.0, 128.6)
- moved J5 36.5 mm to (316.7, 75.3)
- moved R1 36.5 mm to (310.6, 74.1)
- moved R2 36.5 mm to (310.6, 76.0)
- moved J1 36.5 mm to (228.0, 198.6)
- moved S1 36.5 mm to (110.5, 70.3)
- moved R4 36.1 mm to (148.7, 68.5)
- moved Cln_2 35.9 mm to (123.2, 92.0), turned to 180 degrees
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Routing:
- net 3.3V: track 0.00 -> 56.6 mm, vias 0 -> 3
- net GND: track 305.2 -> 356.2 mm, vias 209 -> 242
- net VBUS: track 193.0 -> 215.4 mm
- net 5V: track 0.00 -> 13.5 mm
- net Net-(U1-V_{FB}): track 0.00 -> 12.1 mm
- net Net-(D4-K): track 0.00 -> 7.29 mm
- net Net-(D2-K): track 0.00 -> 5.09 mm
- net Net-(DB1-K): track 0.00 -> 4.81 mm
- net Net-(R3-Pad1): track 0.00 -> 4.65 mm, vias 0 -> 1
- net D1: vias 6 -> 5
- net A1: vias 6 -> 5
- net PROT: vias 6 -> 5
- net A13: vias 6 -> 5
- net Net-(D1-K): vias 0 -> 1
- added copper zone on F.Cu, net 5V
- added copper zone on F.Cu, net GND
- added copper zone on F.Cu, net Net-(D1-K)
Other:
- board text added: "Brian Lu"
- board text added: "Caleb Shinkle"
- board text added: "ECE 47700: Spring 2025"
- board text added: "Nathan Huang"
- board text added: "Seth Deegan"
- board text added: "TEAM 15: AlphaCassiopeiae"

Commit message: Change
Other:
- board text added: "Card"
Changed lines of the file:
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@@
 			(layer "F.SilkS"
 				(type "Top Silk Screen")
+				(color "White")
 			)
 			(layer "F.Paste"
@@
 			(layer "F.Mask"
 				(type "Top Solder Mask")
+				(color "Black")
 				(thickness 0.01)
 			)
@@
 			(layer "B.Mask"
 				(type "Bottom Solder Mask")
+				(color "Black")
 				(thickness 0.01)
 			)
@@
 			(layer "B.SilkS"
 				(type "Bottom Silk Screen")
+				(color "White")
 			)
 			(copper_finish "None")
@@
 		)
 		(property "Value" "10k"
-			(at 0 1.17 360)
+			(at 0 1.17 0)
 			(layer "F.Fab")
 			(hide yes)
@@
 		)
 		(fp_text user "${REFERENCE}"
-			(at 0 0 360)
+			(at 0 0 0)
 			(layer "F.Fab")
 			(effects
@@
 		(at 228 163.616666)
 		(property "Reference" "J4"
-			(at -76.85 -8.241666 360)
+			(at -76.85 -8.241666 0)
 			(layer "F.SilkS")
 			(effects
@@
 		)
 		(property "Value" "10145891-0320J13LF"
-			(at -76.425 -5.841666 360)
+			(at -76.425 -5.841666 0)
 			(layer "F.Fab")
 			(effects
@@
 		)
 		(property "Footprint" "Library:AMPHENOL_10145891-0320J13LF"
-			(at 0 0 360)
+			(at 0 0 0)
 			(layer "F.Fab")
 			(hide yes)
@@
 		)
 		(property "Datasheet" "https://cdn.amphenol-cs.com/media/wysiwyg/files/documentation/datasheet/ssio/ssio_ddr4.pdf"
-			(at 0 0 360)
+			(at 0 0 0)
 			(layer "F.Fab")
 			(hide yes)
@@
 		)
 		(property "Description" ""
-			(at 0 0 360)
+			(at 0 0 0)
 			(layer "F.Fab")
 			(hide yes)
@@
 		(at 228 128.633333)
 		(property "Reference" "J3"
-			(at -76.275 -8.608333 360)
+			(at -76.275 -8.608333 0)
 			(layer "F.SilkS")
 			(effects
@@
 		)
 		(property "Value" "10145891-0320J13LF"
-			(at -76.55 -6.433333 360)
+			(at -76.55 -6.433333 0)
 			(layer "F.Fab")
 			(effects
@@
 		)
 		(property "Footprint" "Library:AMPHENOL_10145891-0320J13LF"
-			(at 0 0 360)
+			(at 0 0 0)
 			(layer "F.Fab")
 			(hide yes)
@@
 		)
 		(property "Datasheet" "https://cdn.amphenol-cs.com/media/wysiwyg/files/documentation/datasheet/ssio/ssio_ddr4.pdf"
-			(at 0 0 360)
+			(at 0 0 0)
 			(layer "F.Fab")
 			(hide yes)
@@
 		)
 		(property "Description" ""
-			(at 0 0 360)
+			(at 0 0 0)
 			(layer "F.Fab")
 			(hide yes)
@@
 		)
 		(property "Value" "31.6k"
-			(at 0 1.17 360)
+			(at 0 1.17 0)
 			(layer "F.Fab")
 			(hide yes)
@@
 		)
 		(fp_text user "${REFERENCE}"
-			(at 0 0 360)
+			(at 0 0 0)
 			(layer "F.Fab")
 			(effects
@@
 		(tags "LED handsolder")
 		(property "Reference" "D4"
-			(at 0.015 -2.2 360)
+			(at 0.015 -2.2 0)
 			(layer "F.SilkS")
 			(effects
@@
 		)
 		(property "Value" "HEARTBEAT"
-			(at 0 1.43 360)
+			(at 0 1.43 0)
 			(layer "F.Fab")
 			(effects
@@
 		)
 		(fp_text user "${REFERENCE}"
-			(at 0 0 360)
+			(at 0 0 0)
 			(layer "F.Fab")
 			(effects
@@
 		)
 		(property "Footprint" "Library:DO-214BA_MCH-L"
-			(at 0 0 360)
+			(at 0 0 0)
 			(layer "F.Fab")
 			(hide yes)
@@
 		)
 		(property "Datasheet" ""
-			(at 0 0 360)
+			(at 0 0 0)
 			(layer "F.Fab")
 			(hide yes)
@@
 		)
 		(property "Description" "Schottky diode"
-			(at 0 0 360)
+			(at 0 0 0)
 			(layer "F.Fab")
 			(hide yes)
@@
 		)
 		(property "Value" "100n"
-			(at 0 1.16 360)
+			(at 0 1.16 0)
 			(layer "F.Fab")
 			(hide yes)
@@
 		)
 		(fp_text user "${REFERENCE}"
-			(at 0 0 360)
+			(at 0 0 0)
 			(layer "F.Fab")
 			(effects
@@
 		(tags "capacitor handsolder")
 		(property "Reference" "Cln_1"
-			(at 5.05 0.1 360)
+			(at 5.05 0.1 0)
 			(layer "F.SilkS")
 			(effects
@@
 		)
 		(property "Value" "10u"
-			(at 0 1.43 360)
+			(at 0 1.43 0)
 			(layer "F.Fab")
 			(hide yes)
@@
 		)
 		(fp_text user "${REFERENCE}"
-			(at 0 0 360)
+			(at 0 0 0)
 			(layer "F.Fab")
 			(effects
@@
 		)
 		(property "Value" "1N4148"
-			(at 0 1.17 360)
+			(at 0 1.17 0)
 			(layer "F.Fab")
 			(hide yes)
@@
 		)
 		(fp_text user "${REFERENCE}"
-			(at 0 0 360)
+			(at 0 0 0)
 			(layer "F.Fab")
 			(effects
@@
 		(tags "resistor")
 		(property "Reference" "R5"
-			(at 0 -1.17 360)
+			(at 0 -1.17 0)
 			(layer "F.SilkS")
 			(effects
@@
 		)
 		(property "Value" "150"
-			(at 0 1.17 360)
+			(at 0 1.17 0)
 			(layer "F.Fab")
 			(effects
@@
 		)
 		(fp_text user "${REFERENCE}"
-			(at 0 0 360)
+			(at 0 0 0)
 			(layer "F.Fab")
 			(effects
@@
 		(at 228 93.65)
 		(property "Reference" "J2"
-			(at -77.625 -7.4 360)
+			(at -77.625 -7.4 0)
 			(layer "F.SilkS")
 			(effects
@@
 		)
 		(property "Value" "10145891-0320J13LF"
-			(at -77.775 -4.95 360)
+			(at -77.775 -4.95 0)
 			(layer "F.Fab")
 			(effects
@@
 		)
 		(property "Footprint" "Library:AMPHENOL_10145891-0320J13LF"
-			(at 0 0 360)
+			(at 0 0 0)
 			(layer "F.Fab")
 			(hide yes)
@@
 		)
 		(property "Datasheet" "https://cdn.amphenol-cs.com/media/wysiwyg/files/documentation/datasheet/ssio/ssio_ddr4.pdf"
-			(at 0 0 360)
+			(at 0 0 0)
 			(layer "F.Fab")
 			(hide yes)
@@
 		)
 		(property "Description" ""
-			(at 0 0 360)
+			(at 0 0 0)
 			(layer "F.Fab")
 			(hide yes)
@@
 		(tags "resistor")
 		(property "Reference" "R4"
-			(at 0.1 1.4 360)
+			(at 0.1 1.4 0)
 			(layer "F.SilkS")
 			(effects
@@
 		)
 		(property "Value" "150"
-			(at -0.05 -1.55 360)
+			(at -0.05 -1.55 0)
 			(layer "F.Fab")
 			(effects
@@
 		)
 		(fp_text user "${REFERENCE}"
-			(at 0 0 360)
+			(at 0 0 0)
 			(layer "F.Fab")
 			(effects
@@
 		(at 228 198.6)
 		(property "Reference" "J1"
-			(at -78.025 7.35 360)
+			(at -78.025 7.35 0)
 			(layer "F.SilkS")
 			(effects
@@
 		)
 		(property "Value" "10145891-0320J13LF"
-			(at -78.075 5.35 360)
+			(at -78.075 5.35 0)
 			(layer "F.Fab")
 			(effects
@@
 		)
 		(property "Footprint" "Library:AMPHENOL_10145891-0320J13LF"
-			(at 0 0 360)
+			(at 0 0 0)
 			(layer "F.Fab")
 			(hide yes)
@@
 		)
 		(property "Datasheet" "https://cdn.amphenol-cs.com/media/wysiwyg/files/documentation/datasheet/ssio/ssio_ddr4.pdf"
-			(at 0 0 360)
+			(at 0 0 0)
 			(layer "F.Fab")
 			(hide yes)
@@
 		)
 		(property "Description" ""
-			(at 0 0 360)
+			(at 0 0 0)
 			(layer "F.Fab")
 			(hide yes)
@@
 		)
 		(property "Price" "3.64"
-			(at 0 0 360)
+			(at 0 0 0)
 			(layer "F.SilkS")
 			(hide yes)
@@
 		)
 		(property "Link" "https://www.digikey.com/en/products/detail/amphenol-cs-fci/10145891-0320J13LF/10233357"
-			(at 0 0 360)
+			(at 0 0 0)
 			(layer "F.SilkS")
 			(hide yes)
@@
 		)
 		(property "Drawing" "https://mm.digikey.com/Volume0/opasdata/d220001/medias/docus/6180/10145891.pdf"
-			(at 0 0 360)
+			(at 0 0 0)
 			(layer "F.SilkS")
 			(hide yes)
@@
 		)
 		(property "Footprint" "Library:DR73-150-R"
-			(at 0 0 360)
+			(at 0 0 0)
 			(layer "F.Fab")
 			(hide yes)
@@
 		)
 		(property "Datasheet" ""
-			(at 0 0 360)
+			(at 0 0 0)
 			(layer "F.Fab")
 			(hide yes)
@@
 		)
 		(property "Description" "Inductor"
-			(at 0 0 360)
+			(at 0 0 0)
 			(layer "F.Fab")
 			(hide yes)
@@
 		(tags "capacitor handsolder")
 		(property "Reference" "Cln_2"
-			(at 5.05 -0.05 360)
+			(at 5.05 -0.05 0)
 			(layer "F.SilkS")
 			(effects
@@
 		)
 		(property "Value" "10u"
-			(at 0 1.43 360)
+			(at 0 1.43 0)
 			(layer "F.Fab")
 			(hide yes)
@@
 		)
 		(fp_text user "${REFERENCE}"
-			(at 0 0 360)
+			(at 0 0 0)
 			(layer "F.Fab")
 			(effects
@@
 		(tags "SOT TO_SOT_SMD")
 		(property "Reference" "U1"
-			(at -0.0375 3.05 360)
+			(at -0.0375 3.05 0)
 			(layer "F.SilkS")
 			(effects
@@
 		)
 		(property "Value" "MCP16331x-xCH"
-			(at -3.1375 7.1 360)
+			(at -3.1375 7.1 0)
 			(layer "F.Fab")
 			(effects
@@
 		)
 		(property "Footprint" "Package_TO_SOT_SMD:SOT-23-6"
-			(at 0 0 360)
+			(at 0 0 0)
 			(layer "F.Fab")
 			(hide yes)
@@
 		)
 		(property "Datasheet" "http://ww1.microchip.com/downloads/en/DeviceDoc/20005308C.pdf"
-			(at 0 0 360)
+			(at 0 0 0)
 			(layer "F.Fab")
 			(hide yes)
@@
 		)
 		(property "Description" "High-Voltage Input Integrated Switch Step-Down Regulator, VDD +4.4V to 50V, Out +2.0V to +24V, SOT-23"
-			(at 0 0 360)
+			(at 0 0 0)
 			(layer "F.Fab")
 			(hide yes)
@@
 		)
 		(fp_text user "${REFERENCE}"
-			(at 0 0 360)
+			(at 0 0 0)
 			(layer "F.Fab")
 			(effects
@@
 		(tags "LED handsolder")
 		(property "Reference" "D2"
-			(at 0 -1.43 360)
+			(at 0 -1.43 0)
 			(layer "F.SilkS")
 			(effects
@@
 		)
 		(property "Value" "HEARTBEAT"
-			(at 0 1.43 360)
+			(at 0 1.43 0)
 			(layer "F.Fab")
 			(effects
@@
 		)
 		(fp_text user "${REFERENCE}"
-			(at 0 0 360)
+			(at 0 0 0)
 			(layer "F.Fab")
 			(effects
@@
 		(layer "B.SilkS")
 		(effects
+			(font
+				(size 5 5)
+				(thickness 0.3)
+				(bold yes)
+			)
+			(justify left bottom mirror)
+		)
+	)
+	(gr_text "Card"
+		(at 311.05 206.8 270)
+		(layer "B.SilkS")
+		(effects
